File: hardware_v1/eurocard.sch (EAGLE design)
At the start: 35 parts, among them IC1 TPS22958, K1 PIN20X2, P1 MAB64Q, U1 EEPROM24, U2 MCP2515-I/SO, U3 MCP2551-I/SN, U4 MCP2551-I/SN, X1 8MHz

Commit message: hardware_v1: add missing title to TPS22958 section
Other:
- note added: "Raspberry Pi Power Control"
Changed lines of the file:
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@@
 <text x="137.16" y="210.82" size="1.778" layer="91">L-CAN address this board</text>
 <text x="2.54" y="43.18" size="1.778" layer="91">120 ohm bus term</text>
+<text x="175.26" y="33.02" size="1.778" layer="91">Raspberry Pi Power Control</text>
 </plain>
 <instances>

Commit message: hardware_v1: update schematic
Parts:
- removed IC1: TPS22958, worlickwerx:TPS22958
- removed U$1: TEENSY_3.1-3.2_ALL_PINS, Teensy_3_and_LC_Series_Boards_v1.4:TEENSY_3.1-3.2_ALL_PINS
- added R10, R11, R13: 10k, resistor:R-EU_M0805
- added R12: 0.1, resistor:R-EU_M0805
- added U5: TEENSY_3.1-3.2_ALL_PINS, Teensy_3_and_LC_Series_Boards_v1.4:TEENSY_3.1-3.2_ALL_PINS
- added U6: TPS22958, worlickwerx:TPS22958
- added U7: INA169, SparkFun-AnalogIC:INA169
Connections:
- removed net +5VSUPPLY: 2.5A.2, C6.1, C7.1, C9.1, IC1.VBIAS, IC1.VIN, IC1.VIN2, U$1.VIN, U4.VDD
- new net N$15: C11.1, R12.2, U6.VOUT, U6.VOUT2, U7.VIN+
- new net N$18: U5.3.3V, U7.V+
- new net PWR-MEAS: R13.2, U5.21/A7/PWM, U7.OUT
- new net VIN: 2.5A.2, C6.1, C7.1, C9.1, U4.VDD, U5.VIN, U6.VBIAS, U6.VIN, U6.VIN2
- net +5V: now also R12.1, U7.VIN-; no longer C11.1, IC1.VOUT, IC1.VOUT2
- net CAN-ACT: now also U5.15/A1/T; no longer U$1.15/A1/T
- net CAN-RX: now also U5.4/CAN-RX/PWM; no longer U$1.4/CAN-RX/PWM
- net CAN-TX: now also U5.3/CAN-TX/PWM; no longer U$1.3/CAN-TX/PWM
- net CONS-RX: now also U5.1/TX1/T; no longer U$1.1/TX1/T
- net CONS-TX: now also U5.0/RX1/T; no longer U$1.0/RX1/T
- net GND: now also R10.1, R11.1, R13.1, U5.GND, U6.GND, U7.GND; no longer IC1.GND, U$1.GND
- net IDENTIFY: now also U5.14/A0; no longer U$1.14/A0
- net MOD-A0: now also U5.9/RX2/PWM; no longer U$1.9/RX2/PWM
- net MOD-A1: now also U5.8/TX3; no longer U$1.8/TX3
- net MOD-A2: now also U5.7/RX3; no longer U$1.7/RX3
- net MOD-A3: now also U5.6/PWM; no longer U$1.6/PWM
- net N$14: now also U6.CT; no longer IC1.CT
- net NODE-A0: now also U5.16/A2/T; no longer U$1.16/A2/T
- net NODE-A1: now also U5.17/A3/T; no longer U$1.17/A3/T
- net NODE-A2: now also U5.18/A4/T/SDA0; no longer U$1.18/A4/T/SDA0
- net NODE-A3: now also U5.19/A5/T/SCL0; no longer U$1.19/A5/T/SCL0
- net PI-RESET: now also U5.22/A8/T/PWM; no longer U$1.22/A8/T/PWM
- net PWR-ON: now also R10.2, U5.23/A9/T/PWM, U6.ON; no longer IC1.ON, U$1.23/A9/T/PWM
- net PWR-SENSE: now also R11.2, U5.2; no longer U$1.2
- net PWR-SHUTDOWN: now also U5.20/A6/PWM; no longer U$1.20/A6/PWM
Other:
- note added: "+5V regulated from bus"
- note added: "1V/A"
- note added: "2W 1% shunt"
- note added: "CAN interface for Raspberry Pi"
- note added: "Compute Board V1"
- note added: "ID EEPROM"
- note added: "Raspberry Pi"
- note added: "green L-CAN activity"
- note removed: "120 ohm bus term"
- note removed: "CAN interface + transceiver for Raspberry Pi"
- note removed: "ID EEPROM - device tree overlay etc"
- note removed: "Jim Garlick"
- note removed: "green TEENSY CAN activity"
- moved on the sheet: C10, C11, C7, C8, C9

Commit message: hardware_v1: move module address pins on DIN connector
The four module address pins on B26 thru B29 were
grounded on my second ebay DIN backplane.  Move them to
A8 through A11 which are clear on both backplanes.

Note: the second backplane also had SMT VME termination
resistors soldered on board which had to be removed
for these pins plus the two L-CAN pins.

A 120 ohm resistor was added to terminate the L-CAN
at both ends of both backplanes (not shown on schematic).
Connections:
- net GND: no longer P1-A14.S
- net MOD-A0: now also P1-A11.S
- net MOD-A1: now also P1-A10.S
- net MOD-A3: now also P1-A8.S
Other:
- note added: "X-CAN address"
- note removed: "X-CAN address from module controller"
Changed lines of the file:
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@@
 <text x="233.68" y="210.82" size="1.778" layer="94">amber identify</text>
 <text x="307.34" y="116.84" size="1.778" layer="94">CAN interface for Raspberry Pi</text>
-<text x="76.2" y="22.86" size="1.778" layer="94">X-CAN address from module controller</text>
-<text x="76.2" y="20.32" size="1.778" layer="94">(open collector)</text>
+<text x="7.62" y="68.58" size="1.778" layer="94">X-CAN address</text>
+<text x="7.62" y="66.04" size="1.778" layer="94">(open collector)</text>
 <text x="137.16" y="210.82" size="1.778" layer="94">L-CAN address this board</text>
 <text x="172.72" y="132.08" size="1.778" layer="94">Raspberry Pi Power Control</text>
@@
 <pinref part="GND13" gate="1" pin="GND"/>
 <wire x1="68.58" y1="20.32" x2="68.58" y2="17.78" width="0.1524" layer="91"/>
-<wire x1="68.58" y1="66.04" x2="68.58" y2="20.32" width="0.1524" layer="91"/>
+<wire x1="68.58" y1="99.06" x2="68.58" y2="20.32" width="0.1524" layer="91"/>
 <junction x="68.58" y="20.32"/>
-<wire x1="68.58" y1="99.06" x2="68.58" y2="66.04" width="0.1524" layer="91"/>
-<junction x="68.58" y="66.04"/>
 <wire x1="35.56" y1="99.06" x2="68.58" y2="99.06" width="0.1524" layer="91"/>
-<wire x1="35.56" y1="66.04" x2="68.58" y2="66.04" width="0.1524" layer="91"/>
 </segment>
 <segment>
@@
 <wire x1="30.48" y1="20.32" x2="30.48" y2="17.78" width="0.1524" layer="91"/>
 <pinref part="GND14" gate="1" pin="GND"/>
-<pinref part="P1" gate="-A14" pin="S"/>
-<wire x1="33.02" y1="66.04" x2="30.48" y2="66.04" width="0.1524" layer="91"/>
-<wire x1="30.48" y1="66.04" x2="30.48" y2="20.32" width="0.1524" layer="91"/>
+<wire x1="30.48" y1="99.06" x2="30.48" y2="20.32" width="0.1524" layer="91"/>
 <junction x="30.48" y="20.32"/>
 <pinref part="P1" gate="-A1" pin="S"/>
 <wire x1="33.02" y1="99.06" x2="30.48" y2="99.06" width="0.1524" layer="91"/>
-<wire x1="30.48" y1="99.06" x2="30.48" y2="66.04" width="0.1524" layer="91"/>
-<junction x="30.48" y="66.04"/>
 </segment>
 <segment>
@@
 </segment>
 <segment>
-<wire x1="55.88" y1="35.56" x2="88.9" y2="35.56" width="0.1524" layer="91"/>
-<label x="78.74" y="35.56" size="1.778" layer="95"/>
-</segment>
-<segment>
 <pinref part="U5" gate="G$1" pin="6/PWM"/>
 <wire x1="187.96" y1="81.28" x2="157.48" y2="81.28" width="0.1524" layer="91"/>
 <label x="157.48" y="81.28" size="1.778" layer="95"/>
+</segment>
+<segment>
+<pinref part="P1" gate="-A8" pin="S"/>
+<wire x1="33.02" y1="81.28" x2="12.7" y2="81.28" width="0.1524" layer="91"/>
+<label x="12.7" y="81.28" size="1.778" layer="95"/>
 </segment>
 </net>
@@
 </segment>
 <segment>
-<wire x1="55.88" y1="30.48" x2="88.9" y2="30.48" width="0.1524" layer="91"/>
-<label x="78.74" y="30.48" size="1.778" layer="95"/>
-</segment>
-<segment>
 <pinref part="U5" gate="G$1" pin="8/TX3"/>
 <wire x1="187.96" y1="76.2" x2="157.48" y2="76.2" width="0.1524" layer="91"/>
 <label x="157.48" y="76.2" size="1.778" layer="95"/>
 </segment>
+<segment>
+<pinref part="P1" gate="-A10" pin="S"/>
+<wire x1="33.02" y1="76.2" x2="12.7" y2="76.2" width="0.1524" layer="91"/>
+<label x="12.7" y="76.2" size="1.778" layer="95"/>
+</segment>
 </net>
 <net name="MOD-A0" class="0">
@@
 </segment>
 <segment>
-<wire x1="55.88" y1="27.94" x2="88.9" y2="27.94" width="0.1524" layer="91"/>
-<label x="78.74" y="27.94" size="1.778" layer="95"/>
-</segment>
-<segment>
 <pinref part="U5" gate="G$1" pin="9/RX2/PWM"/>
 <wire x1="187.96" y1="73.66" x2="157.48" y2="73.66" width="0.1524" layer="91"/>
 <label x="157.48" y="73.66" size="1.778" layer="95"/>
+</segment>
+<segment>
+<pinref part="P1" gate="-A11" pin="S"/>
+<wire x1="33.02" y1="73.66" x2="12.7" y2="73.66" width="0.1524" layer="91"/>
+<label x="12.7" y="73.66" size="1.778" layer="95"/>
 </segment>
 </net>
@@
 </segment>
 <segment>
-<wire x1="55.88" y1="33.02" x2="88.9" y2="33.02" width="0.1524" layer="91"/>
-<label x="78.74" y="33.02" size="1.778" layer="95"/>
-</segment>
-<segment>
 <pinref part="U5" gate="G$1" pin="7/RX3"/>
 <wire x1="187.96" y1="78.74" x2="157.48" y2="78.74" width="0.1524" layer="91"/>
 <label x="157.48" y="78.74" size="1.778" layer="95"/>
+</segment>
+<segment>
+<wire x1="35.56" y1="78.74" x2="12.7" y2="78.74" width="0.1524" layer="91"/>
+<label x="12.7" y="78.74" size="1.778" layer="95"/>
 </segment>
 </net>
@@
 </segment>
 </net>
-<net name="N$12" class="0">
-<segment>
-<wire x1="35.56" y1="60.96" x2="53.34" y2="60.96" width="0.1524" layer="91"/>
-</segment>
-</net>
-<net name="N$13" class="0">
-<segment>
-<wire x1="35.56" y1="22.86" x2="53.34" y2="22.86" width="0.1524" layer="91"/>
-</segment>
-</net>
