File: hardware_v2/daughter.brd (EAGLE design)
At the start: 78 x 56 mm, 11 parts, among them K1 PIN20X2, U1 EEPROM24, U2 MCP2515-I/SO, U3 MCP2551-I/SN, X1 MABC48B2

Commit message: hardware_v2: add TPS27081A load switch
Parts:
- removed R4: 10k, resistor:M0805
- removed U2: MCP2515-I/SO, Microchip_By_element14_Batch_1:SOIC127P1034X264-18N
- removed U3: MCP2551-I/SN, Microchip_By_element14_Batch_1:SOIC127P600X175-8N
- added C4: 1uF, resistor:C1206
- added C5: 100nF, resistor:C1206
- added R5, R6: 10K, resistor:M1206
- added U4: TPS27081A, worlickwerx:SOT95P280X145-6N
- moved CFG 8.38 mm to (97.4, 36.0), turned to 0 degrees
Connections:
- net N$1 renamed ID-SC
- net N$2 renamed ID-SD
- removed net CANINT: K1.32, U2.12
- removed net CE0: K1.24, U2.16
- removed net MISO: K1.21, U2.15
- removed net MOSI: K1.19, U2.14
- removed net N$4: U3.2
- removed net N$5: U2.1, U3.1
- removed net N$6: U2.2, U3.4
- removed net N$7: R4.1, U2.17
- removed net SCK: K1.23, U2.13
- new net CAN-CS0: K1.24
- new net CAN-INT: K1.32
- new net CAN-MISO: K1.21
- new net CAN-MOSI: K1.19
- new net CAN-SCK: K1.23
- new net N$1: R6.1, U4.6
- new net PWR-ON: R5.2, U4.5
- new net PWR-SENSE: K1.37
- new net PWR-SHUTDOWN: K1.38
- net +3V3: no longer R4.2, U2.18
- net +5V: now also C5.1, U4.2, U4.3; no longer U3.3
- net BUS5V: now also C4.1, R6.2, U4.4
- net CAN-H: no longer U3.7
- net CAN-L: no longer U3.6
- net GND: now also C4.2, C5.2, R5.1, U4.1; no longer U2.9
Routing:
- net GND: track 0.00 -> 134.5 mm
- net BUS5V: track 0.00 -> 38.5 mm
- net +5V: track 2.56 -> 36.5 mm
- net PWR-ON: track 0.00 -> 10.8 mm, vias 0 -> 1
- net +3V3: track 75.5 -> 71.2 mm
- net N$1: track 0.00 -> 3.40 mm
- net ID-SD: track 26.3 -> 26.8 mm
- net ID-SC: track 30.2 -> 30.7 mm
- removed copper zone on layer 1, net GND
Other:
- board size 78 x 56 mm -> 78.5 x 56 mm

Commit message: hardware_v2: add stm32
Parts:
- added C6: 100nF, resistor:C0805K
- added R10, R11, R12, R13, R4, R7, R8, R9: 10K, resistor:M0805
- added R14: 10k, resistor:M0805
- added U$1: STM32F103_TQFP48_7X7, dan:LQFP48_7X7
- added U2: MCP2551-I/SN, Microchip_By_element14_Batch_1:SOIC127P600X175-8N
- moved R1 22.6 mm to (85.0, 50.8), turned to 180 degrees
- moved R2 18.4 mm to (88.7, 50.9)
- moved R3 15.6 mm to (87.6, 42.5)
- moved C5 14.5 mm to (54.5, 51.0), turned to 0 degrees
- moved C1 13.5 mm to (95.0, 42.5)
- moved U1 13.1 mm to (92.7, 46.8)
- moved CFG 7.83 mm to (90.4, 39.5), turned to 90 degrees
- moved C4 7.07 mm to (62.0, 43.5), turned to 0 degrees
- moved R5 7.02 mm to (67.0, 46.5)
- moved R6 7.02 mm to (63.5, 48.0)
- moved U4 7.02 mm to (59.0, 48.0)
Connections:
- removed net BUS3V3: X1.C3
- removed net CAN-CS0: K1.24
- removed net CAN-H: X1.C5
- removed net CAN-INT: K1.32
- removed net CAN-L: X1.B5
- removed net CAN-MISO: K1.21
- removed net CAN-MOSI: K1.19
- removed net CAN-SCK: K1.23
- new net CONS-RX: K1.10, U$1.30
- new net CONS-TX: K1.8, U$1.31
- new net LCAN-H: U2.7
- new net LCAN-L: U2.6
- new net LCAN-RX: U$1.32, U2.4
- new net LCAN-TX: U$1.33, U2.1
- new net MOD-A0: R13.2, X1.B14
- new net MOD-A1: R10.2, X1.C14
- new net MOD-A2: R11.2, X1.B15
- new net MOD-A3: R12.2, X1.C15
- new net N$10: R12.1, U$1.17
- new net N$16: R14.2, U2.8
- new net N$2: R4.1, U$1.10
- new net N$4: R7.1, U$1.11, U2.2
- new net N$5: R8.1, U$1.12
- new net N$6: R9.1, U$1.13
- new net N$7: R13.1, U$1.14
- new net N$8: R10.1, U$1.15
- new net N$9: R11.1, U$1.16
- new net NODE-A0: R4.2, X1.B12
- new net NODE-A1: R7.2, X1.C12
- new net NODE-A2: R8.2, X1.B13
- new net NODE-A3: R9.2, X1.C13
- new net VIN: C6.1, U2.3
- net GND: now also C6.2, K1.11, K1.13, K1.15, K1.19, K1.21, K1.23, K1.29, K1.31, K1.33, K1.35, R14.1, X1.A2, X1.B2, X1.C2
- net PWR-ON: now also U$1.26
- net PWR-SENSE: now also U$1.28
- net PWR-SHUTDOWN: now also U$1.27
Routing:
- net GND: track 134.5 -> 105.9 mm
- net +3V3: track 71.2 -> 44.1 mm
- net ID-SD: track 26.8 -> 7.70 mm
- net ID-SC: track 30.7 -> 13.8 mm
- net +5V: track 36.5 -> 23.3 mm
- net CONS-TX: track 0.00 -> 12.8 mm
- net CONS-RX: track 0.00 -> 11.5 mm
- net BUS5V: track 38.5 -> 32.6 mm
- net N$3: track 10.8 -> 12.1 mm
- net PWR-ON: track 10.8 -> 11.4 mm

Commit message: hardware_v2: build in STM32
Parts:
- removed CFG: (no value), FLYFISH:PIN_W_2
- removed U1: EEPROM24, FLYFISH:SOIC8
- added C2: 10uF, resistor:C0805K
- added C3, C7, C8: 100nF, resistor:C0805K
- added C9: 22pF, resistor:C1206
- added IC1: LM1117IMPX-3.3, lm1117:SOT223
- added Q1: 8.00MHz, crystal:SM49
- added R15, R16: 10K, resistor:M0805
- C1: value 100nF -> 22pF; device resistor:C0805K -> resistor:C1206
- R3: value 1k -> 10K
- moved C1 36.4 mm to (59.4, 34.5), turned to 180 degrees
- moved C6 23.8 mm to (78.9, 34.7), turned to 0 degrees
- moved R3 23.4 mm to (64.9, 37.1)
- moved U2 10.1 mm to (72.6, 37.6)
- moved R4 7.50 mm to (46.7, 24.1)
- moved R11 7.19 mm to (46.7, 16.5)
- moved R8 6.84 mm to (46.7, 21.6)
- moved R13 6.77 mm to (46.7, 19.1)
- moved U$1 6.71 mm to (73.4, 26.3)
- moved R1 6.16 mm to (91.1, 49.9)
- moved R12 4.19 mm to (51.1, 15.2)
- moved R2 3.78 mm to (91.1, 47.9), turned to 180 degrees
- moved R7 3.51 mm to (51.1, 22.9)
- moved R10 2.92 mm to (51.1, 17.8)
- moved R9 2.45 mm to (51.1, 20.3)
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Connections:
- removed net VIN: C6.1, U2.3
- new net N$11: R16.2, U$1.20
- new net N$12: U2.2
- new net NRST: R15.2, U$1.7
- new net STBY3V3: C3.1, C7.1, C8.1, IC1.2, IC1.TAB, R15.1, U$1.1, U$1.24, U$1.36, U$1.48, U$1.9
- new net SWCLK: U$1.37, X1.A4
- new net SWDIO: U$1.34, X1.A3
- new net SWO: U$1.39, X1.A5
- new net XTALA: C1.1, Q1.1, U$1.5
- new net XTALB: C9.1, Q1.2, U$1.6
- new net XTALC: U$1.3
- new net XTALD: U$1.4
- net +3V3: no longer C1.1, R3.2, U1.8
- net BUS5V: now also C2.1, C6.1, IC1.3, U2.3
- net GND: now also C2.2, C3.2, C7.2, C8.2, C9.2, IC1.1, R16.1, R3.1, U$1.23, U$1.35, U$1.47, U$1.8; no longer CFG.2, K1.11, K1.13, K1.15, K1.19, K1.21, K1.23, K1.29, K1.31, K1.33, K1.35, K1.9, U1.1, U1.2, U1.3, U1.4
- net ID-SC: now also R2.1; no longer R1.1, U1.6
- net ID-SD: now also R1.1; no longer R2.1, U1.5
- net LCAN-H: now also X1.C5
- net LCAN-L: now also X1.C4
- net N$3: now also R3.2, U$1.44; no longer CFG.1, R3.1, U1.7
- net N$4: no longer U2.2
Routing:
- net GND: track 105.9 -> 237.5 mm
- net CONS-TX: track 12.8 -> 84.9 mm
- net CONS-RX: track 11.5 -> 83.5 mm
- net PWR-SHUTDOWN: track 0.00 -> 57.3 mm
- net PWR-SENSE: track 0.00 -> 53.4 mm
- net STBY3V3: track 0.00 -> 46.5 mm, vias 0 -> 4
- net +3V3: track 44.1 -> 0.13 mm
- net LCAN-L: track 0.00 -> 42.5 mm
- net BUS5V: track 32.6 -> 73.4 mm
- net LCAN-TX: track 0.00 -> 39.3 mm
- net LCAN-H: track 0.00 -> 39.1 mm
- net LCAN-RX: track 0.00 -> 35.8 mm
- net N$9: track 0.00 -> 30.2 mm
- net N$10: track 0.00 -> 27.4 mm
- net N$7: track 0.00 -> 26.5 mm
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
Commit message: hardware_v2: iteration after prelim board milling
Try the 8mhz and 32khz oscillators off-baord, e.g.
shared across the bus.  Experiment with drivers,
conditioning, termination later.

BOOT0 and BOOT1 are tied to ground via 10K resistors.
NRST is tied high via 10K resistor.

Wire the two STM32 slave I2C busses: pi ID EEPROM
emulation and general pi signaling.

IDENTIFY, LCAN-ACT, ALIVE, and +5V power LEDs
are populated but not connected yet.  Possibly the
active LEDs will be folded in with SPI-driven
MAX7212 LED array.
Parts:
- removed C8: 100nF, resistor:C0805K
- removed C9: 22pF, resistor:C1206
- removed IC1: LM1117IMPX-3.3, lm1117:SOT223
- removed Q1: 8.00MHz, crystal:SM49
- removed R13, R15, R16: 10K, resistor:M0805
- removed R14: 10k, resistor:M0805
- added LED1, LED2, LED3, LED4: (no value), led:CHIP-LED0805
- added U$2: MF-SMDF050, fuse:MF-SMDF050
- added U3: LM1117IMPX-3.3, lm1117:SOT223
- C1: value 22pF -> 100nF
- C2: value 10uF -> 100nF; device resistor:C0805K -> resistor:C1206
- C3, C6, C7: device resistor:C0805K -> resistor:C1206
- R1, R2: value 3k9 -> 3K9; device resistor:M0805 -> resistor:M1206
- R10, R11, R12: value 10K -> 220; device resistor:M0805 -> resistor:M1206
- R3, R4, R7, R8: device resistor:M0805 -> resistor:M1206
- R9: value 10K -> 330; device resistor:M0805 -> resistor:M1206
- moved R11 64.5 mm to (106.9, 39.6), turned to 90 degrees
- moved R9 63.2 mm to (106.9, 49.8), turned to 90 degrees
- moved R10 62.0 mm to (106.9, 44.7), turned to 90 degrees
- moved R12 59.1 mm to (106.9, 34.5), turned to 90 degrees
- moved R8 45.7 mm to (88.9, 39.2), turned to 0 degrees
- moved R3 25.6 mm to (72.8, 12.8)
- moved C1 24.1 mm to (83.5, 34.8), turned to 90 degrees
- moved C7 19.6 mm to (60.7, 27.0), turned to 90 degrees
- moved R7 17.9 mm to (65.4, 33.5)
- moved U2 16.5 mm to (88.9, 34.8)
- moved R4 11.4 mm to (57.8, 27.0), turned to 270 degrees
- moved R1 5.70 mm to (85.4, 50.8), turned to 270 degrees
- moved R2 4.25 mm to (88.0, 50.8), turned to 270 degrees
- moved C3 3.71 mm to (80.4, 19.9)
- moved C6 1.51 mm to (79.4, 33.2), turned to 270 degrees
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- renumbered U$1 to U1
Connections:
- removed net N$10: R12.1, U1.17
- removed net N$11: R16.2, U1.20
- removed net N$12: U2.2
- removed net N$2: R4.1, U1.10
- removed net XTALA: C1.1, Q1.1, U1.5
- removed net XTALB: C9.1, Q1.2, U1.6
- removed net XTALC: U1.3
- removed net XTALD: U1.4
- new net ALIVE: R12.2, U1.25
- new net IDENTIFY: R11.2, U1.46
- new net LCAN-ACT: R10.2, U1.41
- new net OSC-HSE: U1.5, X1.C10
- new net OSC-LSE: U1.3, X1.C9
- new net SCL: K1.5, U1.42
- new net SDA: K1.3, U1.43
- net +5V: now also R9.2
- net BUS5V: now also C1.1, U$2.2, U3.3; no longer C6.1, IC1.3, X1.A1, X1.B1, X1.C1
- net GND: now also LED1.C, LED2.C, LED3.C, LED4.C, R7.2, R8.1, U2.2, U3.1; no longer C8.2, C9.2, IC1.1, R14.1, R16.1, X1.A2, X1.B2, X1.C2
- net ID-SC: now also R1.1, U1.21; no longer R2.1
- net ID-SD: now also R2.1, U1.22; no longer R1.1
- net MOD-A0: now also U1.14; no longer R13.2
- net MOD-A1: now also U1.15; no longer R10.2
- net MOD-A2: now also U1.16; no longer R11.2
- net MOD-A3: now also U1.17; no longer R12.2
- net N$16: now also R8.2; no longer R14.2
- net N$3: now also R7.1; no longer R3.2
- net N$4: now also U$2.1, X1.A1, X1.B1, X1.C1; no longer R7.1, U1.11
- net N$5: now also LED4.A, R12.1; no longer R8.1, U1.12
- net N$6: now also R3.2, U1.20; no longer R9.1, U1.13
- net N$7: now also LED3.A, R11.1; no longer R13.1, U1.14
- net N$8: now also LED2.A; no longer U1.15
- net N$9: now also LED1.A, R9.1; no longer R11.1, U1.16
- net NODE-A0: now also U1.10; no longer R4.2
- net NODE-A1: now also U1.11; no longer R7.2
- net NODE-A2: now also U1.12; no longer R8.2
- net NODE-A3: now also U1.13; no longer R9.2
- net NRST: now also R4.1; no longer R15.2
- net STBY3V3: now also C6.1, R4.2, U3.2, U3.TAB; no longer C8.1, IC1.2, IC1.TAB, R15.1
- net SWCLK: now also X1.C7; no longer X1.A4
- net SWDIO: now also X1.C6; no longer X1.A3
- net SWO: now also X1.C8; no longer X1.A5
Routing:
- net ID-SC: track 0.00 -> 100.2 mm
- net ID-SD: track 0.00 -> 95.4 mm
- net STBY3V3: track 46.5 -> 112.4 mm, vias 4 -> 5
- net SWDIO: track 4.86 -> 53.9 mm, vias 1 -> 0
- net GND: track 237.5 -> 281.5 mm, vias 0 -> 6
- net SWCLK: track 1.78 -> 42.9 mm, vias 1 -> 0
- net SDA: track 0.00 -> 40.8 mm, vias 0 -> 2
- net SWO: track 1.77 -> 42.2 mm, vias 1 -> 0
- net SCL: track 0.00 -> 37.6 mm, vias 0 -> 2
- net MOD-A2: track 5.68 -> 37.6 mm
- net BUS5V: track 73.4 -> 105.2 mm
- net PWR-ON: track 24.1 -> 54.8 mm
- net MOD-A3: track 6.90 -> 36.1 mm
- net OSC-HSE: track 0.00 -> 28.7 mm
- net MOD-A0: track 5.68 -> 33.9 mm
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- added copper zone on layer 16, net GND
