File: hardware_v2/daughter.sch (EAGLE design)
At the start: 11 parts, among them K1 PIN20X2, U1 EEPROM24, U2 MCP2515-I/SO, U3 MCP2551-I/SN, X1 MABC48B2

Commit message: hardware_v2: add TPS27081A load switch
Parts:
- removed R4: 10k, resistor:R-EU_M0805
- removed U2: MCP2515-I/SO, Microchip_By_element14_Batch_1:MCP2515-I/SO
- removed U3: MCP2551-I/SN, Microchip_By_element14_Batch_1:MCP2551-I/SN
- added C4: 1uF, resistor:C-EUC1206
- added C5: 100nF, resistor:C-EUC1206
- added R5, R6: 10K, resistor:R-EU_M1206
- added U4: TPS27081A, worlickwerx:TPS27081A
Connections:
- net N$1 renamed ID-SC
- net N$2 renamed ID-SD
- removed net CANINT: K1.32, U2.~INT
- removed net CE0: K1.24, U2.~CS
- removed net MISO: K1.21, U2.SO
- removed net MOSI: K1.19, U2.SI
- removed net N$4: U3.VSS
- removed net N$5: U2.TXCAN, U3.TXD
- removed net N$6: U2.RXCAN, U3.RXD
- removed net N$7: R4.1, U2.~RESET
- removed net SCK: K1.23, U2.SCK
- new net CAN-CS0: K1.24
- new net CAN-INT: K1.32
- new net CAN-MISO: K1.21
- new net CAN-MOSI: K1.19
- new net CAN-SCK: K1.23
- new net N$1: R6.1, U4.R1/C1
- new net PWR-ON: R5.2, U4.ON/OFF
- new net PWR-SENSE: K1.37
- new net PWR-SHUTDOWN: K1.38
- net +3V3: no longer R4.2, U2.VDD
- net +5V: now also C5.1, U4.VOUT1, U4.VOUT2; no longer U3.VDD
- net BUS5V: now also C4.1, R6.2, U4.VIN
- net CAN-H: no longer U3.CANH
- net CAN-L: no longer U3.CANL
- net GND: now also C4.2, C5.2, R5.1, U4.R2; no longer U2.VSS
Other:
- note added: "Compute Board V2"
- note added: "Raspberry Pi"
- note removed: "Jim Garlick"
- moved on the sheet: C1, CFG, K1, R1, R2, R3, U1

Commit message: hardware_v2: add stm32
Parts:
- added C6: 100nF, resistor:C-EUC0805K
- added R10, R11, R12, R13, R4, R7, R8, R9: 10K, resistor:R-EU_M0805
- added R14: 10k, resistor:R-EU_M0805
- added U$1: STM32F103_TQFP48_7X7, dan:STM32F103_TQFP48_7X7
- added U2: MCP2551-I/SN, Microchip_By_element14_Batch_1:MCP2551-I/SN
Connections:
- removed net BUS3V3: X1-C3.S
- removed net CAN-CS0: K1.24
- removed net CAN-H: X1-C5.S
- removed net CAN-INT: K1.32
- removed net CAN-L: X1-B5.S
- removed net CAN-MISO: K1.21
- removed net CAN-MOSI: K1.19
- removed net CAN-SCK: K1.23
- new net CONS-RX: K1.10, U$1.PA9
- new net CONS-TX: K1.8, U$1.PA10
- new net LCAN-H: U2.CANH
- new net LCAN-L: U2.CANL
- new net LCAN-RX: U$1.PA11, U2.RXD
- new net LCAN-TX: U$1.PA12, U2.TXD
- new net MOD-A0: R13.2, X1-B14.S
- new net MOD-A1: R10.2, X1-C14.S
- new net MOD-A2: R11.2, X1-B15.S
- new net MOD-A3: R12.2, X1-C15.S
- new net N$10: R12.1, U$1.PA7
- new net N$16: R14.2, U2.RS
- new net N$2: R4.1, U$1.PA0-WKUP
- new net N$4: R7.1, U$1.PA1, U2.VSS
- new net N$5: R8.1, U$1.PA2
- new net N$6: R9.1, U$1.PA3
- new net N$7: R13.1, U$1.PA4
- new net N$8: R10.1, U$1.PA5
- new net N$9: R11.1, U$1.PA6
- new net NODE-A0: R4.2, X1-B12.S
- new net NODE-A1: R7.2, X1-C12.S
- new net NODE-A2: R8.2, X1-B13.S
- new net NODE-A3: R9.2, X1-C13.S
- new net VIN: C6.1, U2.VDD
- net GND: now also C6.2, K1.11, K1.13, K1.15, K1.19, K1.21, K1.23, K1.29, K1.31, K1.33, K1.35, R14.1, X1-A2.S, X1-B2.S, X1-C2.S
- net PWR-ON: now also U$1.PB13
- net PWR-SENSE: now also U$1.PB15
- net PWR-SHUTDOWN: now also U$1.PB14
Other:
- note added: "CAN transceiver for L-CAN"
- moved on the sheet: K1, R6

Commit message: hardware_v2: build in STM32
Parts:
- removed CFG: (no value), FLYFISH:PIN2_100
- removed U1: EEPROM24, FLYFISH:EEPROM24
- added C2: 10uF, resistor:C-EUC0805K
- added C3, C7, C8: 100nF, resistor:C-EUC0805K
- added C9: 22pF, resistor:C-EUC1206
- added IC1: LM1117IMPX-3.3, lm1117:LM1117IMPX-3.3
- added Q1: 8.00MHz, crystal:CRYSTALSM49
- added R15, R16: 10K, resistor:R-EU_M0805
- C1: value 100nF -> 22pF; device resistor:C-EUC0805K -> resistor:C-EUC1206; DIELECTRIC X7R -> (none)
- R3: value 1k -> 10K
Connections:
- removed net VIN: C6.1, U2.VDD
- new net N$11: R16.2, U$1.PB2
- new net N$12: U2.VSS
- new net NRST: R15.2, U$1.NRST
- new net STBY3V3: C3.1, C7.1, C8.1, IC1.OUT, IC1.OUT1, R15.1, U$1.VBAT, U$1.VDDA, U$1.VDD_1, U$1.VDD_2, U$1.VDD_3
- new net SWCLK: U$1.PA14, X1-A4.S
- new net SWDIO: U$1.PA13, X1-A3.S
- new net SWO: U$1.PB3, X1-A5.S
- new net XTALA: C1.1, Q1.1, U$1.PD0-OSC_IN
- new net XTALB: C9.1, Q1.2, U$1.PD1-OSC_OUT
- new net XTALC: U$1.PC14-OSC32_IN
- new net XTALD: U$1.PC15-OSC32-OUT
- net +3V3: no longer C1.1, R3.2, U1.VCC
- net BUS5V: now also C2.1, C6.1, IC1.IN, U2.VDD
- net GND: now also C2.2, C3.2, C7.2, C8.2, C9.2, IC1.GND, R16.1, R3.1, U$1.VSSA, U$1.VSS_1, U$1.VSS_2, U$1.VSS_3; no longer CFG.2, K1.11, K1.13, K1.15, K1.19, K1.21, K1.23, K1.29, K1.31, K1.33, K1.35, K1.9, U1.A0, U1.A1, U1.A2, U1.GND
- net ID-SC: now also R2.1; no longer R1.1, U1.SCL
- net ID-SD: now also R1.1; no longer R2.1, U1.SDA
- net LCAN-H: now also X1-C5.S
- net LCAN-L: now also X1-C4.S
- net N$3: now also R3.2, U$1.BOOT0; no longer CFG.1, R3.1, U1.WP
- net N$4: no longer U2.VSS
Other:
- note added: "L-CAN transceiver"
- note removed: "CAN transceiver for L-CAN"
- moved on the sheet: C1, C4, C5, C6, K1, R1, R10, R11, R12, R13, R14, R2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

Commit message: hardware_v2: iteration after prelim board milling
Try the 8mhz and 32khz oscillators off-baord, e.g.
shared across the bus.  Experiment with drivers,
conditioning, termination later.

BOOT0 and BOOT1 are tied to ground via 10K resistors.
NRST is tied high via 10K resistor.

Wire the two STM32 slave I2C busses: pi ID EEPROM
emulation and general pi signaling.

IDENTIFY, LCAN-ACT, ALIVE, and +5V power LEDs
are populated but not connected yet.  Possibly the
active LEDs will be folded in with SPI-driven
MAX7212 LED array.
Parts:
- removed C8: 100nF, resistor:C-EUC0805K
- removed C9: 22pF, resistor:C-EUC1206
- removed IC1: LM1117IMPX-3.3, lm1117:LM1117IMPX-3.3
- removed Q1: 8.00MHz, crystal:CRYSTALSM49
- removed R13, R15, R16: 10K, resistor:R-EU_M0805
- removed R14: 10k, resistor:R-EU_M0805
- added LED1, LED2, LED3, LED4: (no value), led:LEDCHIP-LED0805
- added U$2: MF-SMDF050, fuse:MF-SMDF050
- added U3: LM1117IMPX-3.3, lm1117:LM1117IMPX-3.3
- C1: value 22pF -> 100nF
- C2: value 10uF -> 100nF; device resistor:C-EUC0805K -> resistor:C-EUC1206; DIELECTRIC X7R -> (none)
- C3, C6, C7: device resistor:C-EUC0805K -> resistor:C-EUC1206; DIELECTRIC X7R -> (none)
- R1, R2: value 3k9 -> 3K9; device resistor:R-EU_M0805 -> resistor:R-EU_M1206; TOLERANCE 5% -> (none)
- R10, R11, R12: value 10K -> 220; device resistor:R-EU_M0805 -> resistor:R-EU_M1206; TOLERANCE 5% -> (none)
- R3, R4, R7, R8: device resistor:R-EU_M0805 -> resistor:R-EU_M1206; TOLERANCE 5% -> (none)
- R9: value 10K -> 330; device resistor:R-EU_M0805 -> resistor:R-EU_M1206; TOLERANCE 5% -> (none)
- renumbered U$1 to U1
Connections:
- removed net N$10: R12.1, U1.PA7
- removed net N$11: R16.2, U1.PB2
- removed net N$12: U2.VSS
- removed net N$2: R4.1, U1.PA0-WKUP
- removed net XTALA: C1.1, Q1.1, U1.PD0-OSC_IN
- removed net XTALB: C9.1, Q1.2, U1.PD1-OSC_OUT
- removed net XTALC: U1.PC14-OSC32_IN
- removed net XTALD: U1.PC15-OSC32-OUT
- new net ALIVE: R12.2, U1.PB12
- new net IDENTIFY: R11.2, U1.PB9
- new net LCAN-ACT: R10.2, U1.PB5
- new net OSC-HSE: U1.PD0-OSC_IN, X1-C10.S
- new net OSC-LSE: U1.PC14-OSC32_IN, X1-C9.S
- new net SCL: K1.5, U1.PB6
- new net SDA: K1.3, U1.PB7
- net +5V: now also R9.2
- net BUS5V: now also C1.1, U$2.2, U3.IN; no longer C6.1, IC1.IN, X1-A1.S, X1-B1.S, X1-C1.S
- net GND: now also LED1.C, LED2.C, LED3.C, LED4.C, R7.2, R8.1, U2.VSS, U3.GND; no longer C8.2, C9.2, IC1.GND, R14.1, R16.1, X1-A2.S, X1-B2.S, X1-C2.S
- net ID-SC: now also R1.1, U1.PB10; no longer R2.1
- net ID-SD: now also R2.1, U1.PB11; no longer R1.1
- net MOD-A0: now also U1.PA4; no longer R13.2
- net MOD-A1: now also U1.PA5; no longer R10.2
- net MOD-A2: now also U1.PA6; no longer R11.2
- net MOD-A3: now also U1.PA7; no longer R12.2
- net N$16: now also R8.2; no longer R14.2
- net N$3: now also R7.1; no longer R3.2
- net N$4: now also U$2.1, X1-A1.S, X1-B1.S, X1-C1.S; no longer R7.1, U1.PA1
- net N$5: now also LED4.A, R12.1; no longer R8.1, U1.PA2
- net N$6: now also R3.2, U1.PB2; no longer R9.1, U1.PA3
- net N$7: now also LED3.A, R11.1; no longer R13.1, U1.PA4
- net N$8: now also LED2.A; no longer U1.PA5
- net N$9: now also LED1.A, R9.1; no longer R11.1, U1.PA6
- net NODE-A0: now also U1.PA0-WKUP; no longer R4.2
- net NODE-A1: now also U1.PA1; no longer R7.2
- net NODE-A2: now also U1.PA2; no longer R8.2
- net NODE-A3: now also U1.PA3; no longer R9.2
- net NRST: now also R4.1; no longer R15.2
- net STBY3V3: now also C6.1, R4.2, U3.OUT, U3.OUT1; no longer C8.1, IC1.OUT, IC1.OUT1, R15.1
- net SWCLK: now also X1-C7.S; no longer X1-A4.S
- net SWDIO: now also X1-C6.S; no longer X1-A3.S
- net SWO: now also X1-C8.S; no longer X1-A5.S
Other:
- note added: "2.5A PTC"
- note added: "BLU"
- note added: "GRN"
- note added: "RED"
- note added: "STM32F103C8T6"
- note added: "YEL"
- moved on the sheet: C1, C2, C3, C6, C7, R1, R10, R11, R12, R2, R3, R4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
