File: hardware/pi-carrier/eurocard.kicad_pcb (KiCad board)
At the start: 2 copper layers, 159.9 x 99.9 mm, 72 parts, among them J1 molliebus, J2 Conn_01x03_Male, J3 Conn_01x03_Male, J4 Conn_02x20_Odd_Even, J5 Raspberry_Pi_2_3, J6 Conn_02x20_Odd_Even, J7 Conn_01x02, J8 Conn_02x08_Counter_Clockwise, U1 SN74LVC1G07DBVR, U10 LTP747, U11 TCAN332, U12 MCP2515-xSO, U13 CAT24C128, U2 TCAN332, U3 LM1117-3.3, U4 74AUP1G74, U5 TPS27081ADDCR, U6 STM32F103C8Tx, U7 INA169NA_3K, U8 SN74AHCT125N, U9 MAX7219, Y1 8MHz, Y2 8MHz

Commit message: pi-carrier: connect MCP2515 INT to GPIO12 (pin32)
Connections:
- U12 pad 12: Net-(U12-Pad12) -> /PI_GPIO12
Routing:
- net /PI_GPIO12: track 73.5 -> 139.9 mm, vias 1 -> 3

Commit message: pi-carrier: omit fully utilized GPIOs from expansion
Problem: Pi GPIO12 and PI_SPI1_CE2 are both assigned to CAN adapter,
so exposing them on expansion header only asks for trouble.

Disconnect those pins.
Connections:
- J4 pad 32: /PI_GPIO12 -> Net-(J4-Pad32)
- J4 pad 36: /PI_SPI1_CE2 -> Net-(J4-Pad36)
Routing:
- net /PI_SPI1_CE2: track 145.3 -> 146.1 mm
- net /PI_GPIO12: track 139.9 -> 140.6 mm

Commit message: pi-carrier: update pcb from schematic
Connections:
- net /PB14 renamed Net-(U6-Pad27)

Commit message: pi-carrier: replace 1x3 symbols
Problem: 1x3 pinheader symbols are hard to spot

Replace 1x3 schematic symbols with ones that have a filled body.

Refresh PCB.
Parts:
- J2, J3: value Conn_01x03_Male -> Conn_01x03
- moved J3 14.3 mm to (176.9, 50.5)
- moved J2 14.2 mm to (162.5, 50.4)
Connections:
- J2 pad 2: /BOOT1 -> Net-(J2-Pad2)
- J3 pad 2: Net-(J3-Pad2) -> /BOOT1
- U4 pad 7: Net-(J3-Pad2) -> Net-(J2-Pad2)
Routing:
- net Net-(J3-Pad2): track 7.43 -> 0.00 mm
- net Net-(J2-Pad2): track 0.00 -> 7.43 mm

Commit message: pi-carrier: move SWD to header
Problem: SWD pins are not really appropriate to have on the bus.

Move SWD to a 4-pin header.
Reroute pcb.
Parts:
- added J9: Conn_01x04, Connector_PinHeader_2.54mm:PinHeader_1x04_P2.54mm_Vertical, F.Cu at (167.0, 81.9)
- moved C16 0.15 mm to (187.0, 74.8)
Connections:
- J1 pad a15: /SWO -> Net-(J1-Pada15)
- J1 pad a16: /SWDIO -> Net-(J1-Pada16)
- J1 pad a17: /SWCLK -> Net-(J1-Pada17)
Routing:
- net /SWO: track 33.8 -> 38.6 mm, vias 0 -> 2
- net /SWCLK: track 39.8 -> 44.5 mm, vias 1 -> 2
- net GND: track 130.3 -> 135.0 mm
- net /SWDIO: track 32.4 -> 36.4 mm, vias 0 -> 2
Other:
- board text added: "gnd"
- board text added: "swclk"
- board text added: "swdio"
- board text added: "swo"
- board text removed: "SWCLK"
- board text removed: "SWDIO"
- board text removed: "SWO"

Commit message: pi-carrier: fix EEPROM write protect
Problem: EEPROM write protect is wired wrong.

Make WP a jumperable pull-up to 3V3.  Data sheet says it is pulled
down to GND internally.

Reroute PCB and label "Write Protect" instead of "Write Enable".
Parts:
- moved J7 0.72 mm to (100.2, 122.9)
Connections:
- J7 pad 2: GND -> Net-(J7-Pad2)
- U13 pad 7: Net-(J7-Pad1) -> Net-(J7-Pad2)
Routing:
- net Net-(J7-Pad1): track 18.6 -> 12.7 mm
- net Net-(J7-Pad2): track 0.00 -> 5.22 mm
Other:
- board text added: "write protect"
- board text removed: "write enable"

Commit message: pi-carrier: use PI_SPI1_CE0 on CAN
Instead of CE2, use PI_SPI1_CE0, to tidy things up.
Reroute PCB.
Connections:
- net /PI_GPIO12 renamed /PI_SPI1_INT
- J4 pad 12: /PI_SPI1_CE0 -> Net-(J4-Pad12)
- J4 pad 36: Net-(J4-Pad36) -> /PI_SPI1_CE2
- U12 pad 16: /PI_SPI1_CE2 -> /PI_SPI1_CE0
Routing:
- net /PI_SPI1_CE2: track 146.1 -> 76.7 mm, vias 3 -> 1
- net /PI_SPI1_CE0: track 102.7 -> 126.4 mm

Commit message: pi-carrier: rename PI_SPIx_CEn lines
Name the SPI CEx lines, where x > 0, to their PI_GPIO counterparts
since these are more likely to be used as GPIO.

Reroute PCB.
Connections:
- net /PI_SPI1_CE1 renamed /PI_GPIO17
- net /PI_SPI1_CE2 renamed /PI_GPIO16
- net /PI_SPI4_CE1 renamed /PI_GPIO25
