File: hardware/pi-carrier/eurocard.kicad_pcb (KiCad board)
At the start: 2 copper layers, 159.9 x 99.9 mm, 73 parts, among them J1 molliebus, J2 Conn_01x03, J3 Conn_01x03, J4 Conn_02x20_Odd_Even, J5 Raspberry_Pi_2_3, J6 Conn_02x20_Odd_Even, J7 Conn_01x02, J8 Conn_02x08_Counter_Clockwise, J9 Conn_01x04, U1 SN74LVC1G07DBVR, U10 LTP747, U11 TCAN332, U12 MCP2515-xSO, U13 CAT24C128, U2 TCAN332, U3 LM1117-3.3, U4 74AUP1G74, U5 TPS27081ADDCR, U6 STM32F103C8Tx, U7 INA169NA_3K, U8 SN74AHCT125N, U9 MAX7219, Y1 8MHz, Y2 8MHz

Commit message: pi-carrier: move SWD connector to top of board
Parts:
- moved J9 27.3 mm to (166.6, 54.6)
- moved R16 2.47 mm to (177.7, 54.2), turned to 90 degrees
Routing:
- net /SWCLK: track 44.5 -> 76.8 mm, vias 2 -> 3
- net /SWO: track 38.6 -> 67.8 mm, vias 2 -> 3
- net /SWDIO: track 36.4 -> 65.4 mm, vias 2 -> 3
- net Net-(R16-Pad1): track 33.8 -> 31.5 mm
- net /BOOT1: track 4.07 -> 5.67 mm
Other:
- board text added: "SWCLK"
- board text added: "SWDIO"
- board text added: "SWO"
- board text removed: "gnd"
- board text removed: "swclk"
- board text removed: "swdio"
- board text removed: "swo"

Commit message: pi-carrier: drop DIN pin number labels
Other:
- board text removed: "20"
- board text removed: "30"

Commit message: pi-carrier: add expansion mounting holes
Add two M2.5 mounting holes to secure expansion card.
Parts:
- added REF**: MountingHole_2.7mm_M2.5_DIN965, MountingHole:MountingHole_2.7mm_M2.5_DIN965, F.Cu at (149.1, 81.4)
- added REF**: MountingHole_2.7mm_M2.5_DIN965, MountingHole:MountingHole_2.7mm_M2.5_DIN965, F.Cu at (199.9, 138.8)
- moved R8 1.02 mm to (145.8, 78.1)
- moved R9 1.02 mm to (145.8, 78.1)
Routing:
- net /PI_5V: track 78.1 -> 75.3 mm
- net /PI_SCL: track 118.2 -> 119.8 mm
- net /PWR_MEASURE_V: track 67.0 -> 66.2 mm

Commit message: pi-carrier: remove leftover trace
Routing:
- net Net-(J4-Pad13): track 9.53 -> 0.00 mm, vias 1 -> 0

Commit message: pi-carrier: label exp header pads for usb
Move GPIO17 to other side of expansion header to make room.
Label two header pins as for USB D+, D-.
Connections will be made with bodge wire.
Connections:
- net Net-(J4-Pad13) renamed /PI_USB_D-
- J4 pad 11: /PI_GPIO17 -> /PI_USB_D+
- J4 pad 12: Net-(J4-Pad12) -> /PI_GPIO17
Routing:
- net /PI_GPIO17: track 115.7 -> 111.4 mm
Other:
- board text added: "USB_D+"
- board text added: "USB_D-"

Commit message: pi-carrier: tweak silk screen
Add SWD label to SWD header, and move pin defs to bottom.
Add pi-carrier v2, (c), CERN lic, OSHW logo.
Parts:
- added REF**: OSHW-Logo2_7.3x6mm_SilkScreen, Symbol:OSHW-Logo2_7.3x6mm_SilkScreen, F.Cu at (86.3, 50.4)
Other:
- board text added: "(c) 2020 WorlickWerx"
- board text added: "CERN-OHL-1.2"
- board text added: "SWD"
- board text added: "pi-carrier v2"

Commit message: pi-carrier: add bypass cap on INA169
Datasheet says optional, but better safe than sorry.
Parts:
- added C22: 100nF, Capacitor_SMD:C_0805_2012Metric_Pad1.18x1.45mm_HandSolder, B.Cu at (150.6, 73.3)
Routing:
- net GND: track 135.0 -> 138.5 mm
- net +3V3: track 202.9 -> 205.6 mm

Commit message: pi-carrier: add PTC silk label
Other:
- board text added: "3A PTC"
