File: hardware/pi-carrier/eurocard.kicad_pcb (KiCad board)
At the start: 2 copper layers, 159.9 x 99.9 mm, 83 parts, among them J1 DIN41612_C96_male_ra_molliebus, J2 Debug, J3 console, J4 Conn_02x20_Odd_Even, J5 Conn_02x20_raspberry_pi4B, J9 Conn_02x05_Odd_Even, U1 74LVC1G07, U10 Lite-on LTP747KR, U11 TCAN332DR, U12 MCP2518FD, U2 TCAN332DR, U3 LM1117IMPX-3.3, U4 74LVC2G04, U5 74LVC2G38, U6 STM32F103C8T6, U8 SN74AHCT125PWR, U9 MAX7219CWG, X1 ASE-40.000MHz-LC, X2 ASE-8.000MHz-LC, Y1 ABS07-32.768KHZ-6-T

Commit message: pi-carrier: add heart symbol above blinky led
Problem: the blinky LED really needs a little heart symbol.

Oh joy, unicode is accepted.
Other:
- board text added: "♥"
Changed lines of the file:
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@@
     (effects (font (size 1 1) (thickness 0.15)))
+  )
+  (gr_text "♥" (at 199.1488 63.8024) (layer "F.SilkS")
+    (effects (font (face "FreeSerif") (size 1.5 1.5) (thickness 0.3) bold) (justify left bottom))
+    (render_cache "♥" 0
+      (polygon
+        (pts
+          (xy 200.421183 62.745428)          (xy 200.42063 62.763429)          (xy 200.418973 62.781526)          (xy 200.416211 62.799722)
+          (xy 200.412344 62.818014)          (xy 200.407372 62.836404)          (xy 200.401296 62.854891)          (xy 200.394115 62.873475)
+          (xy 200.385828 62.892157)          (xy 200.376438 62.910936)          (xy 200.365942 62.929812)          (xy 200.354341 62.948786)
+          (xy 200.341636 62.967857)          (xy 200.327826 62.987025)          (xy 200.312911 63.006291)          (xy 200.296891 63.025654)
+          (xy 200.279766 63.045114)          (xy 200.269153 63.057221)          (xy 200.25728 63.070279)          (xy 200.244149 63.084286)
+          (xy 200.233473 63.095416)          (xy 200.222089 63.10708)          (xy 200.209997 63.119278)          (xy 200.197197 63.132011)
+          (xy 200.183688 63.145279)          (xy 200.16947 63.159081)          (xy 200.159599 63.168579)          (xy 200.145002 63.182608)
+          (xy 200.131301 63.195846)          (xy 200.118495 63.208291)          (xy 200.106584 63.219944)          (xy 200.095569 63.230805)
+          (xy 200.082274 63.244055)          (xy 200.07057 63.255896)          (xy 200.058179 63.268717)          (xy 200.050056 63.277389)
+          (xy 200.035795 63.293794)          (xy 200.021588 63.31086)          (xy 200.007436 63.328587)          (xy 199.993338 63.346975)
+          (xy 199.979294 63.366025)          (xy 199.965305 63.385736)          (xy 199.951371 63.406107)          (xy 199.93749 63.42714)
+          (xy 199.923664 63.448835)          (xy 199.909893 63.47119)          (xy 199.896175 63.494207)          (xy 199.882513 63.517884)
+          (xy 199.868904 63.542223)          (xy 199.85535 63.567223)          (xy 199.841851 63.592884)          (xy 199.835121 63.605963)
+          (xy 199.828405 63.619207)          (xy 199.821669 63.605586)          (xy 199.814926 63.592155)          (xy 199.808174 63.578913)
+          (xy 199.801414 63.565861)          (xy 199.787872 63.540326)          (xy 199.774298 63.515549)          (xy 199.760692 63.49153)
+          (xy 199.747055 63.468271)          (xy 199.733387 63.445769)          (xy 199.719687 63.424026)          (xy 199.705955 63.403042)
+          (xy 199.692192 63.382816)          (xy 199.678398 63.363349)          (xy 199.664572 63.34464)          (xy 199.650714 63.326689)
+          (xy 199.636825 63.309497)          (xy 199.622905 63.293064)          (xy 199.608953 63.277389)          (xy 199.597785 63.265747)
+          (xy 199.587112 63.254836)          (xy 199.574893 63.242506)          (xy 199.561129 63.228756)          (xy 199.549791 63.217511)
+          (xy 199.537584 63.205469)          (xy 199.524507 63.192627)          (xy 199.510562 63.178987)          (xy 199.495746 63.164549)
+          (xy 199.480868 63.149962)          (xy 199.466595 63.135878)          (xy 199.452927 63.122296)          (xy 199.439864 63.109216)
+          (xy 199.427407 63.096639)          (xy 199.415556 63.084564)          (xy 199.404309 63.072991)          (xy 199.393668 63.061921)
+          (xy 199.380422 63.047942)          (xy 199.368252 63.034856)          (xy 199.356688 63.021655)          (xy 199.345262 63.007516)
+          (xy 199.333974 62.992438)          (xy 199.322823 62.976421)          (xy 199.314549 62.963792)          (xy 199.306353 62.950635)
+          (xy 199.298235 62.93695)          (xy 199.290193 62.922737)          (xy 199.282229 62.907996)          (xy 199.279592 62.902965)
+          (xy 199.272062 62.88776)          (xy 199.265273 62.872645)          (xy 199.259225 62.857621)          (xy 199.253917 62.842686)
+          (xy 199.24935 62.827842)          (xy 199.245524 62.813088)          (xy 199.242438 62.798424)          (xy 199.240093 62.783851)
+          (xy 199.238118 62.764559)          (xy 199.23746 62.745428)          (xy 199.237671 62.728157)          (xy 199.238307 62.71115)
+          (xy 199.239366 62.694406)          (xy 199.240849 62.677925)          (xy 199.242755 62.661708)          (xy 199.245085 62.645754)
+          (xy 199.247838 62.630063)          (xy 199.251015 62.614636)          (xy 199.254788 62.599375)          (xy 199.259144 62.584182)
+          (xy 199.264084 62.569058)          (xy 199.269608 62.554003)          (xy 199.275716 62.539016)          (xy 199.282408 62.524098)
+          (xy 199.289684 62.509249)          (xy 199.297543 62.494469)          (xy 199.306193 62.480003)          (xy 199.315839 62.466281)
+          (xy 199.32648 62.453304)          (xy 199.338118 62.441071)          (xy 199.350752 62.429582)          (xy 199.364382 62.418837)
+          (xy 199.379008 62.408837)          (xy 199.39463 62.39958)          (xy 199.411128 62.391165)          (xy 199.428381 62.383872)
+          (xy 199.44639 62.377701)          (xy 199.465155 62.372652)          (xy 199.479724 62.369602)          (xy 199.494719 62.367183)
+          (xy 199.510138 62.365395)          (xy 199.525983 62.364238)          (xy 199.542253 62.363712)          (xy 199.54777 62.363677)
+          (xy 199.567455 62.364047)          (xy 199.586485 62.365159)          (xy 199.604859 62.367012)          (xy 199.622577 62.369607)
+          (xy 199.63964 62.372943)          (xy 199.656048 62.37702)          (xy 199.6718 62.381839)          (xy 199.686897 62.387399)
+          (xy 199.701338 62.3937)          (xy 199.715124 62.400742)          (xy 199.728255 62.408526)          (xy 199.74073 62.417051)
+          (xy 199.752549 62.426318)          (xy 199.763713 62.436325)          (xy 199.774222 62.447075)          (xy 199.784075 62.458565)
+          (xy 199.793422 62.470989)          (xy 199.803189 62.48422)          (xy 199.811896 62.496203)          (xy 199.820912 62.508778)
+          (xy 199.830237 62.521946)          (xy 199.838895 62.509406)          (xy 199.841961 62.505093)          (xy 199.850677 62.492667)
+          (xy 199.859252 62.480726)          (xy 199.859913 62.479814)          (xy 199.868424 62.467664)          (xy 199.874567 62.458565)
+          (xy 199.884429 62.447075)          (xy 199.894963 62.436325)          (xy 199.90617 62.426318)          (xy 199.91805 62.417051)
+          (xy 199.930602 62.408526)          (xy 199.943827 62.400742)          (xy 199.957725 62.3937)          (xy 199.972295 62.387399)
+          (xy 199.987538 62.381839)          (xy 200.003453 62.37702)          (xy 200.020041 62.372943)          (xy 200.037302 62.369607)
+          (xy 200.055235 62.367012)          (xy 200.073841 62.365159)          (xy 200.093119 62.364047)          (xy 200.11307 62.363677)
+          (xy 200.129482 62.363982)          (xy 200.145468 62.3649)          (xy 200.161029 62.36643)          (xy 200.176165 62.368571)
+          (xy 200.190876 62.371324)          (xy 200.205162 62.374689)          (xy 200.223549 62.380127)          (xy 200.24118 62.386653)
+          (xy 200.258056 62.394267)          (xy 200.266211 62.398481)          (xy 200.281815 62.407577)          (xy 200.29639 62.417463)
+          (xy 200.309934 62.428139)          (xy 200.322447 62.439606)          (xy 200.333931 62.451862)          (xy 200.344384 62.464908)
+          (xy 200.353806 62.478744)          (xy 200.362198 62.493369)          (xy 200.369794 62.508408)          (xy 200.37683 62.52348)
+          (xy 200.383304 62.538587)          (xy 200.389217 62.553728)          (xy 200.39457 62.568904)          (xy 200.399361 62.584113)
+          (xy 200.403591 62.599358)          (xy 200.407261 62.614636)          (xy 200.410524 62.630063)          (xy 200.413352 62.645754)
+          (xy 200.415744 62.661708)          (xy 200.417702 62.677925)          (xy 200.419225 62.694406)          (xy 200.420312 62.71115)
+          (xy 200.420965 62.728157)
+        )
+      )
+    )
   )
   (gr_text "Barrier" (at 196.304 96.289) (layer "F.SilkS")

Commit message: pi-carrier: update version to 3.2
Problem: we need another minor rev of the pi-carrier.

Bump version to 3.2.
Other:
- board text added: "pi-carrier v3.2"
- board text removed: "pi-carrier v3.1"
Changed lines of the file:
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@@
     (effects (font (size 1 1) (thickness 0.15)))
   )
-  (gr_text "pi-carrier v3.1" (at 107.15 49.68) (layer "F.SilkS")
+  (gr_text "pi-carrier v3.2" (at 107.15 49.68) (layer "F.SilkS")
     (effects (font (size 2 2) (thickness 0.3)))
   )

Commit message: pi-carrier: remove pi5 power mode
Problem: there is no need to have a special pi5 power mode
now that we have the pi5_adapter with a load switch.

Restore PA6 test point and drop DNP resistors for selecting
pi5 power mode.
Parts:
- removed R2: 10K, Resistor_SMD:R_0603_1608Metric
- removed R3: 0, Resistor_SMD:R_0603_1608Metric
- added TP19: PA6, TestPoint:TestPoint_Pad_1.0x1.0mm, B.Cu at (150.2, 61.2)
- J3: value console -> Console
Connections:
- U6 pad 16: /~{PI5_ENA} -> Net-(U6-PA6)
Routing:
- net /~{PI5_ENA}: track 73.9 -> 0.00 mm, vias 3 -> 0
- net Net-(U6-PA6): track 0.00 -> 73.6 mm, vias 0 -> 3
- net /PI_3V3: track 224.9 -> 211.3 mm
- net /RUN_PG: track 86.0 -> 75.2 mm
Other:
- board text removed: "PI5_BTN"
- board text removed: "place for Pi 5"

Commit message: pi-carrier: ensure TP Reference is plotted on silk
Problem: testpoint silk labels did not show up on the v3.1
board.

I thought I was being clever and replaced the Value field of
"TestPoint" with a descriptive name, and placed it on the silk
layer, but KiCad 7 did not plot Value fields in the fabrication
outputs.

After receiving the boards, I noted that the Gerber Viewer tool
did not show those fields on the silk layer.  Maybe it is a KiCad
bug or maybe I did something wrong.

Set Value back to "TestPoint" in all TP footprints, uncheck "visible".

Place the Reference field on the silk layer, check "visible".

Now the silk labels are the reference desgnators (e.g. "TP17")
rather than the descriptive names, but this is probably more
appropriate and expected anyway.
Parts:
- TP1: value 5V -> TestPoint
- TP10: value ~{RST} -> TestPoint
- TP11: value GND -> TestPoint
- TP12: value CAN+ -> TestPoint
- TP13: value CAN- -> TestPoint
- TP14: value PI3V3 -> TestPoint
- TP15: value NSS -> TestPoint
- TP16: value SCK -> TestPoint
- TP17: value MOSI -> TestPoint
- TP18: value PB4 -> TestPoint
- TP19: value PA6 -> TestPoint
- TP2: value 3V3 -> TestPoint
- TP20: value PA7 -> TestPoint
- TP21: value PA11 -> TestPoint
- TP22: value PA12 -> TestPoint
- TP25: value RUN_PG -> TestPoint
- TP26: value GLOBAL_EN -> TestPoint
- TP3: value STBY -> TestPoint
- TP4: value CELL -> TestPoint
- TP5: value 8MHz -> TestPoint
- TP6: value VBAT -> TestPoint
- TP7: value 40MHz -> TestPoint
- TP8: value SDA -> TestPoint
- TP9: value SCL -> TestPoint

Commit message: pi-carrier: fix console label
Problem: console label did not show up on silk

Same problem as with the test points in the last commit, and same fix.
Add a separate descriptive silk label.
Other:
- board text added: "Pi Console"
Changed lines of the file:
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@@
         (effects (font (size 1 1) (thickness 0.15)))
     )
-    (fp_text value "Console" (at 0 3.98) (layer "F.SilkS")
+    (fp_text value "Console" (at 0 3.98) (layer "F.SilkS") hide
         (effects (font (size 1 1) (thickness 0.15)))
     )
-    (fp_text user "${REFERENCE}" (at 0 0) (layer "F.Fab")
+    (fp_text user "${REFERENCE}" (at 0 0) (layer "F.Fab") hide
         (effects (font (size 1 1) (thickness 0.15)))
     )
@@
     (effects (font (size 1 1) (thickness 0.15)))
   )
+  (gr_text "Pi Console" (at 161.0996 96.6446) (layer "F.SilkS")
+    (effects (font (size 1 1) (thickness 0.15)) (justify left bottom))
+  )
   (gr_text "3V3@800mA" (at 181.88 59.17) (layer "F.SilkS")

Commit message: pi-carrier: drop 3-pin debug connector
Problem: meh, extra 3-pin debug connector is not too helpful.

Drop it.
Parts:
- removed J2: Debug, Connector_JST:JST_SH_BM03B-SRSS-TB_1x03-1MP_P1.00mm_Vertical
- F1: value PTC 3A 6V -> PTC 3A
Routing:
- net /SWCLK: track 193.4 -> 180.9 mm, vias 4 -> 3
- net /SWDIO: track 305.7 -> 294.3 mm, vias 5 -> 4
- net GND: track 121.5 -> 119.4 mm, vias 109 -> 108

Commit message: pi-carrier: add 3-pin power connector
Problem: RUN_PG and GLOBAL_EN should be via a connector
rather than solderd in.

Replace the testpoints on the back of the board with a 3-pin
JST connector on the front of the board.
Parts:
- removed TP25, TP26: TestPoint, TestPoint:TestPoint_Pad_1.0x1.0mm
- added J2: Console, Connector_JST:JST_SH_SM03B-SRSS-TB_1x03-1MP_P1.00mm_Horizontal, F.Cu at (180.5, 65.2)
- moved TP19 44.1 mm to (169.8, 100.7)
Routing:
- net Net-(U6-PA6): track 73.6 -> 6.52 mm, vias 3 -> 1
- net /RUN_PG: track 75.2 -> 51.6 mm, vias 3 -> 2
- net /GLOBAL_EN: track 73.0 -> 50.6 mm, vias 3 -> 2
- net /BUTTON1: track 71.6 -> 72.4 mm
Other:
- board text added: "GLOBAL_EN"
- board text added: "RUN_PG"

Commit message: pi-carrier: make room for M.2
- remove J4 HAT connector and mounting holes
- relocate components to make space for M.2
- move heartbeat LED and debug J9 near STM32
- drop GPIO console connection, just use JST connector
- reroute traces
Parts:
- removed J4: Conn_02x20_Odd_Even, 00_eurocard:Rasp_pi_hat_socket
- removed R4, R6: 0, Resistor_SMD:R_0603_1608Metric
- added REF**: OSHW-Logo_5.7x6mm_SilkScreen, Symbol:OSHW-Logo_5.7x6mm_SilkScreen, F.Cu at (199.8, 140.6)
- moved D1 66.5 mm to (200.1, 124.0), turned to 90 degrees
- moved C20 61.0 mm to (197.9, 124.0), turned to 90 degrees
- moved TP4 56.8 mm to (195.8, 130.9)
- moved BT1 55.6 mm to (183.1, 130.9)
- moved TP6 53.9 mm to (192.8, 124.7)
- moved J3 50.0 mm to (174.5, 50.9), turned to -90 degrees
- moved D3 48.4 mm to (188.7, 112.0)
- moved R15 48.2 mm to (184.7, 112.0)
- moved J9 39.0 mm to (196.6, 103.6), turned to 0 degrees
- moved TP3 34.1 mm to (166.9, 113.6)
- moved C17 29.9 mm to (183.6, 62.5)
- moved TP13 24.0 mm to (198.3, 66.0)
- moved TP7 20.8 mm to (180.1, 75.7)
- moved X1 20.4 mm to (177.3, 71.2)
- moved U12 20.3 mm to (183.7, 68.3)
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Connections:
- J5 pad 10: /GPIO15 -> unconnected-(J5-GPIO15/RXD-Pad10)
- J5 pad 11: /GPIO17 -> unconnected-(J5-GPIO17-Pad11)
- J5 pad 15: /GPIO22 -> unconnected-(J5-GPIO22-Pad15)
- J5 pad 16: /GPIO23 -> unconnected-(J5-GPIO23-Pad16)
- J5 pad 18: /GPIO24 -> unconnected-(J5-GPIO24-Pad18)
- J5 pad 19: /GPIO10 -> unconnected-(J5-MOSI0/GPIO10-Pad19)
- J5 pad 21: /GPIO9 -> unconnected-(J5-MISO0/GPIO9-Pad21)
- J5 pad 22: /GPIO25 -> unconnected-(J5-GPIO25-Pad22)
- J5 pad 23: /GPIO11 -> unconnected-(J5-SCLK0/GPIO11-Pad23)
- J5 pad 24: /GPIO8 -> unconnected-(J5-~{CE0}/GPIO8-Pad24)
- J5 pad 26: /GPIO7 -> unconnected-(J5-~{CE1}/GPIO7-Pad26)
- J5 pad 27: /ID_SD -> unconnected-(J5-ID_SD/GPIO0-Pad27)
- J5 pad 28: /ID_SC -> unconnected-(J5-ID_SC/GPIO1-Pad28)
- J5 pad 7: /GPIO4 -> unconnected-(J5-GCLK0/GPIO4-Pad7)
- J5 pad 8: /GPIO14 -> unconnected-(J5-GPIO14/TXD-Pad8)
Routing:
- net /ID_SC: track 126.8 -> 0.00 mm
- net /ID_SD: track 123.2 -> 0.00 mm
- net /GPIO7: track 119.4 -> 0.00 mm
- net /GPIO8: track 113.3 -> 0.00 mm
- net /GPIO11: track 109.7 -> 0.00 mm
- net /GPIO25: track 106.1 -> 0.00 mm
- net /GPIO9: track 102.4 -> 0.00 mm
- net /GPIO15: track 99.3 -> 0.00 mm, vias 1 -> 0
- net /GPIO10: track 96.2 -> 0.00 mm
- net /GPIO24: track 92.4 -> 0.00 mm
- net /GPIO14: track 90.9 -> 0.00 mm, vias 1 -> 0
- net +BATT: track 138.8 -> 52.1 mm, vias 7 -> 5
- net /GPIO23: track 85.0 -> 0.00 mm
- net /GPIO22: track 81.4 -> 0.00 mm
- net /GPIO17: track 67.9 -> 0.00 mm
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Other:
- board text added: "CONSOLE_RX"
- board text added: "CONSOLE_TX"
- board text removed: "3V3@800mA"
- board text removed: "5V@3A"
- board text removed: "Pi Console"
- board text removed: "Real Time Clock Power"
- board text removed: "place for console on GPIO"
