File: hardware/pi-carrier/eurocard.kicad_sch (KiCad schematic)
At the start: 69 parts, among them J1 DIN41612_C96_male_ra_molliebus, J2 Conn_01x03, J3 Conn_01x03, J4 Conn_02x20_Odd_Even, J5 Conn_02x20_raspberry_pi4B, J6 Conn_02x20_Odd_Even, J7 Conn_01x02, J8 8x10 prototype area, J9 Conn_01x04, U1 SN74LVC1G07DBVR, U10 Lite-on LTP747KR, U11 TCAN332DR, U12 MCP2515-I/SO, U13 CAT24C128WI, U2 TCAN332DR, U3 LM1117IMPX-3.3, U4 SN74AUP1G74DCUR, U5 TPS27081ADDCR, U6 STM32F103C8T6, U7 INA169NA, U8 SN74AHCT125PWR, U9 MAX7219CWG, X1 Abracon ASE-16.000MHz-LC, X2 Abracon ASE-8.000MHz-LC

Commit message: pi-carrier: drop pi ID EEPROM and pullups
Problem: pi ID EEPROM is not used, and the other I2C pullups
are in the wrong place.

Delete them.
Parts:
- removed C21: 100nF 16V, Capacitor_SMD:C_0805_2012Metric_Pad1.18x1.45mm_HandSolder, symbol Device:C
- removed J7: Conn_01x02, Connector_PinHeader_2.54mm:PinHeader_1x02_P2.54mm_Vertical, symbol Connector_Generic:Conn_01x02
- removed R12, R13: DNP, Resistor_SMD:R_0805_2012Metric_Pad1.20x1.40mm_HandSolder, symbol Device:R
- removed R19, R20: 4.7K, Resistor_SMD:R_0805_2012Metric_Pad1.20x1.40mm_HandSolder, symbol Device:R
- removed R21: 10K, Resistor_SMD:R_0805_2012Metric_Pad1.20x1.40mm_HandSolder, symbol Device:R
- removed U13: CAT24C128WI, Package_SO:SOIC-8_3.9x4.9mm_P1.27mm, symbol Memory_EEPROM:CAT24C128
Connections:
- removed net ID_SC: J4.3 (Pin_3), J4.5 (Pin_5), J5.27 (ID_SD/GPIO0), J5.28 (ID_SC/GPIO1), J5.3 (SDA/GPIO2), J5.5 (SCL/GPIO3), U6.21 (PB10), U6.22 (PB11)
- new net PI_SCL: J4.5 (Pin_5), J5.5 (SCL/GPIO3), U6.21 (PB10)
- new net PI_SDA: J4.3 (Pin_3), J5.3 (SDA/GPIO2), U6.22 (PB11)
- no-connect marks 37 -> 39

Commit message: pi-carrier: add STM32 I2C pullups
Problem: I2C requires pullups powered by the STM32 power not
pi 3V3 as before.

Add back I2C pullups in the STM32 section of the schematic.
Recreate annotations.
Parts:
- added R12, R13: 4.7K, Resistor_SMD:R_0805_2012Metric_Pad1.20x1.40mm_HandSolder, symbol Device:R
Connections:
- net +3V3: now also R12.1, R13.1
- net PI_SCL: now also R13.2
- net PI_SDA: now also R12.2
Changed lines of the file:
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@@
   (junction (at 66.04 157.48) (diameter 0) (color 0 0 0 0)
   )
+  (junction (at 152.4 153.67) (diameter 0) (color 0 0 0 0)
+  )
   (junction (at 66.04 152.4) (diameter 0) (color 0 0 0 0)
   )
@@
     (stroke (width 0) (type default) (color 0 0 0 0))
   )
+  (wire (pts (xy 133.35 156.21) (xy 144.78 156.21))
+    (stroke (width 0) (type default) (color 0 0 0 0))
+  )
   (wire (pts (xy 102.87 69.85) (xy 109.22 69.85))
     (stroke (width 0) (type default) (color 0 0 0 0))
@@
     (stroke (width 0) (type default) (color 0 0 0 0))
   )
+  (wire (pts (xy 152.4 153.67) (xy 152.4 156.21))
+    (stroke (width 0) (type default) (color 0 0 0 0))
+  )
   (wire (pts (xy 127 154.94) (xy 129.54 154.94))
     (stroke (width 0) (type default) (color 0 0 0 0))
@@
     (stroke (width 0) (type default) (color 0 0 0 0))
   )
+  (wire (pts (xy 133.35 153.67) (xy 144.78 153.67))
+    (stroke (width 0) (type default) (color 0 0 0 0))
+  )
   (wire (pts (xy 254 104.14) (xy 259.08 104.14))
     (stroke (width 0) (type default) (color 0 0 0 0))
@@
     (stroke (width 0) (type default) (color 0 0 0 0))
   )
+  (wire (pts (xy 152.4 152.4) (xy 152.4 153.67))
+    (stroke (width 0) (type default) (color 0 0 0 0))
+  )
   (wire (pts (xy 102.87 77.47) (xy 104.14 77.47))
     (stroke (width 0) (type default) (color 0 0 0 0))
@@
     (effects (font (size 1.27 1.27)) (justify right bottom))
   )
+  (label "PI_SDA" (at 133.35 153.67 0)
+    (effects (font (size 1.27 1.27)) (justify left bottom))
+  )
   (label "PI_USB_D-" (at 228.6 104.14 0)
     (effects (font (size 1.27 1.27)) (justify left bottom))
@@
     (effects (font (size 1.27 1.27)) (justify right bottom))
   )
+  (label "PI_SCL" (at 133.35 156.21 0)
+    (effects (font (size 1.27 1.27)) (justify left bottom))
+  )
   (label "GA3" (at 53.34 140.97 180)
     (effects (font (size 1.27 1.27)) (justify right bottom))
@@
     (pin "2")
   )
+  (symbol (lib_id "Device:R") (at 148.59 153.67 270) (unit 1)
+    (in_bom yes) (on_board yes)
+    (property "Reference" "R12" (id 0) (at 156.21 153.67 90)
+      (effects (font (size 1.27 1.27)) (justify right))
+    )
+    (property "Value" "4.7K" (id 1) (at 151.13 153.67 90)
+      (effects (font (size 1.27 1.27)) (justify right))
+    )
+    (property "Footprint" "Resistor_SMD:R_0805_2012Metric_Pad1.20x1.40mm_HandSolder" (id 2) (at 148.59 151.892 90)
+      (effects (font (size 1.27 1.27)) hide)
+    )
+    (property "Datasheet" "~" (id 3) (at 148.59 153.67 0)
+      (effects (font (size 1.27 1.27)) hide)
+    )
+    (pin "1")
+    (pin "2")
+  )
+  (symbol (lib_id "Device:R") (at 148.59 156.21 270) (unit 1)
+    (in_bom yes) (on_board yes)
+    (property "Reference" "R13" (id 0) (at 156.21 156.21 90)
+      (effects (font (size 1.27 1.27)) (justify right))
+    )
+    (property "Value" "4.7K" (id 1) (at 151.13 156.21 90)
+      (effects (font (size 1.27 1.27)) (justify right))
+    )
+    (property "Footprint" "Resistor_SMD:R_0805_2012Metric_Pad1.20x1.40mm_HandSolder" (id 2) (at 148.59 154.432 90)
+      (effects (font (size 1.27 1.27)) hide)
+    )
+    (property "Datasheet" "~" (id 3) (at 148.59 156.21 0)
+      (effects (font (size 1.27 1.27)) hide)
+    )
+    (pin "1")
+    (pin "2")
+  )
   (symbol (lib_id "Device:LED_Dual_AAKK") (at 248.92 25.4 0) (unit 1)
     (in_bom yes) (on_board yes) (fields_autoplaced)
@@
     (pin "4")
   )
+  (symbol (lib_id "power:+3V3") (at 152.4 152.4 0) (unit 1)
+    (in_bom yes) (on_board yes)
+    (property "Reference" "#PWR054" (id 0) (at 152.4 156.21 0)
+      (effects (font (size 1.27 1.27)) hide)
+    )
+    (property "Value" "+3V3" (id 1) (at 148.59 149.86 0))
+    (property "Footprint" "" (id 2) (at 152.4 152.4 0)
+      (effects (font (size 1.27 1.27)) hide)
+    )
+    (property "Datasheet" "" (id 3) (at 152.4 152.4 0)
+      (effects (font (size 1.27 1.27)) hide)
+    )
+    (pin "1")
+  )
   (sheet_instances
     (path "/" (page "1"))
@@
       (reference "#PWR053") (unit 1) (value "GND") (footprint "")
     )
+    (path "/bc1fec57-f0df-46a2-8f1d-85e3fb1ddd36"
+      (reference "#PWR054") (unit 1) (value "+3V3") (footprint "")
+    )
     (path "/00000000-0000-0000-0000-00005fe3b2f2"
       (reference "#PWR055") (unit 1) (value "GND") (footprint "")
@@
       (reference "R11") (unit 1) (value "10K") (footprint "Resistor_SMD:R_0805_2012Metric_Pad1.20x1.40mm_HandSolder")
     )
+    (path "/60dcce00-cc14-440d-98ef-fede0f250f80"
+      (reference "R12") (unit 1) (value "4.7K") (footprint "Resistor_SMD:R_0805_2012Metric_Pad1.20x1.40mm_HandSolder")
+    )
+    (path "/7da67589-58cc-4e37-88bc-efd345dfa100"
+      (reference "R13") (unit 1) (value "4.7K") (footprint "Resistor_SMD:R_0805_2012Metric_Pad1.20x1.40mm_HandSolder")
+    )
     (path "/00000000-0000-0000-0000-00005fdf5fc8"

Commit message: pi-carrier: drop power measurement shunt
Problem: power measurement drops too much V on the pi supply.

Remove power shunt and associated measurement circuitry.
Parts:
- removed C22: 100nF 16V, Capacitor_SMD:C_0805_2012Metric_Pad1.18x1.45mm_HandSolder, symbol Device:C
- removed R10: 10K, Resistor_SMD:R_0805_2012Metric_Pad1.20x1.40mm_HandSolder, symbol Device:R
- removed R6: 0.1 (1%) 2W, Resistor_SMD:R_2512_6332Metric_Pad1.40x3.35mm_HandSolder, symbol Device:R
- removed R8, R9: 10K (0.1%), Resistor_SMD:R_0805_2012Metric_Pad1.20x1.40mm_HandSolder, symbol Device:R
- removed U7: INA169NA, Package_TO_SOT_SMD:SOT-23-5_HandSoldering, symbol 00_eurocard:INA169NA_3K
Connections:
- net PI_5V: now also R7.2, U5.2 (VOUT), U5.3 (VOUT)
- net PWR_MEASURE_I: no longer names the net of U6.18 (PB0)
- net PWR_MEASURE_V: no longer names the net of U6.19 (PB1)
- no-connect marks 39 -> 41

Commit message: pi-carrier: remove power LED
Problem: Red power LED was too bright and is redundant with
pi power LED.

Drop extra LED.
Parts:
- removed D1: LED_RED, LED_SMD:LED_0805_2012Metric_Pad1.15x1.40mm_HandSolder, symbol Device:LED
- removed R7: 510, Resistor_SMD:R_0805_2012Metric_Pad1.20x1.40mm_HandSolder, symbol Device:R
Changed lines of the file:
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@@
   (junction (at 45.72 166.37) (diameter 0) (color 0 0 0 0)
   )
-  (junction (at 121.92 48.26) (diameter 0) (color 0 0 0 0)
-  )
   (junction (at 90.17 35.56) (diameter 0) (color 0 0 0 0)
   )
@@
     (stroke (width 0) (type default) (color 0 0 0 0))
   )
-  (wire (pts (xy 121.92 48.26) (xy 134.62 48.26))
-    (stroke (width 0) (type default) (color 0 0 0 0))
-  )
   (wire (pts (xy 87.63 40.64) (xy 87.63 46.99))
     (stroke (width 0) (type default) (color 0 0 0 0))
@@
     (stroke (width 0) (type default) (color 0 0 0 0))
   )
-  (wire (pts (xy 102.87 48.26) (xy 121.92 48.26))
+  (wire (pts (xy 102.87 48.26) (xy 134.62 48.26))
     (stroke (width 0) (type default) (color 0 0 0 0))
   )
@@
     (stroke (width 0) (type default) (color 0 0 0 0))
   )
-  (wire (pts (xy 101.6 57.15) (xy 101.6 58.42))
-    (stroke (width 0) (type default) (color 0 0 0 0))
-  )
   (wire (pts (xy 69.85 34.29) (xy 69.85 44.45))
     (stroke (width 0) (type default) (color 0 0 0 0))
@@
     (stroke (width 0) (type default) (color 0 0 0 0))
   )
-  (wire (pts (xy 120.65 57.15) (xy 121.92 57.15))
-    (stroke (width 0) (type default) (color 0 0 0 0))
-  )
   (wire (pts (xy 175.26 63.5) (xy 175.26 71.12))
     (stroke (width 0) (type default) (color 0 0 0 0))
@@
     (stroke (width 0) (type default) (color 0 0 0 0))
   )
-  (wire (pts (xy 110.49 57.15) (xy 113.03 57.15))
-    (stroke (width 0) (type default) (color 0 0 0 0))
-  )
   (wire (pts (xy 123.19 175.26) (xy 134.62 175.26))
     (stroke (width 0) (type default) (color 0 0 0 0))
@@
     (stroke (width 0) (type default) (color 0 0 0 0))
   )
-  (wire (pts (xy 101.6 57.15) (xy 102.87 57.15))
-    (stroke (width 0) (type default) (color 0 0 0 0))
-  )
   (wire (pts (xy 44.45 69.85) (xy 53.34 69.85))
     (stroke (width 0) (type default) (color 0 0 0 0))
@@
     (stroke (width 0) (type default) (color 0 0 0 0))
   )
-  (wire (pts (xy 121.92 48.26) (xy 121.92 57.15))
-    (stroke (width 0) (type default) (color 0 0 0 0))
-  )
   (wire (pts (xy 66.04 130.81) (xy 59.69 130.81))
     (stroke (width 0) (type default) (color 0 0 0 0))
@@
     (pin "1")
   )
-  (symbol (lib_id "Device:R") (at 116.84 57.15 90) (unit 1)
-    (in_bom yes) (on_board yes)
-    (property "Reference" "R7" (id 0) (at 115.57 54.61 90)
-      (effects (font (size 1.27 1.27)) (justify right))
-    )
-    (property "Value" "510" (id 1) (at 115.57 57.15 90)
-      (effects (font (size 1.27 1.27)) (justify right))
-    )
-    (property "Footprint" "Resistor_SMD:R_0805_2012Metric_Pad1.20x1.40mm_HandSolder" (id 2) (at 116.84 58.928 90)
-      (effects (font (size 1.27 1.27)) hide)
-    )
-    (property "Datasheet" "~" (id 3) (at 116.84 57.15 0)
-      (effects (font (size 1.27 1.27)) hide)
-    )
-    (pin "1")
-    (pin "2")
-  )
-  (symbol (lib_id "Device:LED") (at 106.68 57.15 0) (mirror x) (unit 1)
-    (in_bom yes) (on_board yes)
-    (property "Reference" "D1" (id 0) (at 106.68 54.61 0))
-    (property "Value" "LED_RED" (id 1) (at 106.68 59.69 0))
-    (property "Footprint" "LED_SMD:LED_0805_2012Metric_Pad1.15x1.40mm_HandSolder" (id 2) (at 106.68 57.15 0)
-      (effects (font (size 1.27 1.27)) hide)
-    )
-    (property "Datasheet" "~" (id 3) (at 106.68 57.15 0)
-      (effects (font (size 1.27 1.27)) hide)
-    )
-    (property "MPN" "APT2012SURCK" (id 4) (at 106.68 57.15 0)
-      (effects (font (size 1.27 1.27)) hide)
-    )
-    (property "Manufacturer" "Kingbright" (id 5) (at 106.68 57.15 0)
-      (effects (font (size 1.27 1.27)) hide)
-    )
-    (property "digkey.com" "754-1133-2-ND" (id 6) (at 106.68 57.15 0)
-      (effects (font (size 1.27 1.27)) hide)
-    )
-    (pin "1")
-    (pin "2")
-  )
-  (symbol (lib_id "power:GND") (at 101.6 58.42 0) (unit 1)
-    (in_bom yes) (on_board yes)
-    (property "Reference" "#PWR026" (id 0) (at 101.6 64.77 0)
-      (effects (font (size 1.27 1.27)) hide)
-    )
-    (property "Value" "GND" (id 1) (at 99.06 58.42 0))
-    (property "Footprint" "" (id 2) (at 101.6 58.42 0)
-      (effects (font (size 1.27 1.27)) hide)
-    )
-    (property "Datasheet" "" (id 3) (at 101.6 58.42 0)
-      (effects (font (size 1.27 1.27)) hide)
-    )
-    (pin "1")
-  )
   (symbol (lib_id "power:GND") (at 175.26 71.12 0) (unit 1)
     (in_bom yes) (on_board yes)
@@
       (reference "#PWR025") (unit 1) (value "GND") (footprint "")
     )
-    (path "/00000000-0000-0000-0000-00005ed2ccf1"
-      (reference "#PWR026") (unit 1) (value "GND") (footprint "")
-    )
     (path "/00000000-0000-0000-0000-00005ee4cbdd"
       (reference "#PWR027") (unit 1) (value "+5V") (footprint "")
@@
       (reference "C19") (unit 1) (value "100nF 16V") (footprint "Capacitor_SMD:C_0805_2012Metric_Pad1.18x1.45mm_HandSolder")
     )
-    (path "/00000000-0000-0000-0000-00005ed1cb4e"
-      (reference "D1") (unit 1) (value "LED_RED") (footprint "LED_SMD:LED_0805_2012Metric_Pad1.15x1.40mm_HandSolder")
-    )
     (path "/84c3fabc-e977-49be-994f-37fed9bce5e7"
       (reference "D2") (unit 1) (value "LED_Dual_AAKK") (footprint "LED_THT:LED_BL-FL7680RGB")
@@
       (reference "R5") (unit 1) (value "10K") (footprint "Resistor_SMD:R_0805_2012Metric_Pad1.20x1.40mm_HandSolder")
     )
-    (path "/00000000-0000-0000-0000-00005ed1b5ec"
-      (reference "R7") (unit 1) (value "510") (footprint "Resistor_SMD:R_0805_2012Metric_Pad1.20x1.40mm_HandSolder")
-    )
     (path "/00000000-0000-0000-0000-00005eaf7f56"

Commit message: pi-carrier: remove load switch
Problem: switching PI_5V with load switch drops power supply
too much.

Just power the pi power inputs all the time and use the pi's
own PMIC to control power.
Parts:
- removed C6: 1uF 16V, Capacitor_SMD:C_0805_2012Metric_Pad1.18x1.45mm_HandSolder, symbol Device:C
- removed R4: 10K, Resistor_SMD:R_0805_2012Metric_Pad1.20x1.40mm_HandSolder, symbol Device:R
- removed U5: TPS27081ADDCR, Package_TO_SOT_SMD:SOT-23-6_Handsoldering, symbol 00_eurocard:TPS27081ADDCR
- added J7: Conn_01x03, Connector_PinHeader_2.54mm:PinHeader_1x03_P2.54mm_Vertical, symbol Connector_Generic:Conn_01x03
Connections:
- net +5V: now also J5.2 (5V), J5.4 (5V)
- net GND: now also J7.2 (Pin_2)
- net PI_5V: no longer J5.2 (5V), J5.4 (5V)
- net GLOBAL_EN: now reaches U6.27 (PB14)
- net GLOBAL_EN: now also J7.1 (Pin_1)
- net RUN_PG: now reaches U6.29 (PA8)
- net RUN_PG: now also J7.3 (Pin_3)
- no-connect marks 41 -> 39
