File: hardware/pi-carrier/eurocard.kicad_sch (KiCad schematic)
At the start: 53 parts, among them J1 DIN41612_C96_male_ra_molliebus, J2 Conn_01x03, J3 Conn_01x03, J4 Conn_02x20_Odd_Even, J5 Conn_02x20_raspberry_pi4B, J6 Conn_02x20_Odd_Even, J7 Conn_01x03, J8 8x10 prototype area, J9 Conn_01x04, U1 SN74LVC1G07DBVR, U10 Lite-on LTP747KR, U11 TCAN332DR, U12 MCP2515-I/SO, U2 TCAN332DR, U3 LM1117IMPX-3.3, U4 SN74AUP1G74DCUR, U6 STM32F103C8T6, U8 SN74AHCT125PWR, U9 MAX7219CWG, X1 Abracon ASE-16.000MHz-LC, X2 Abracon ASE-8.000MHz-LC

Commit message: pi-carrier: connect SWD to pi
Problem: STM32 must be programmed with an external programmer.

OpenOCD can be used to program the STM32.  Connect SWDIO and SWCLK
to two pi GPIO pins.

Fix some minor ERC problems.
Connections:
- net PI_GPIO13: no longer J5.33 (PWM1/GPIO13)
- net PI_GPIO16: no longer J5.36 (GPIO16)
- net SWCLK: now also J5.33 (PWM1/GPIO13)
- net SWDIO: now also J5.36 (GPIO16)
- net PERSONALITY: no longer names the net of U6.40 (PB4)
- net PI_USB_D+: no longer names the net of J4.11 (Pin_11)
- net PI_USB_D-: no longer names the net of J4.13 (Pin_13)
Other:
- moved on the sheet: J9
Changed lines of the file:
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@@
   )
   (no_connect (at 20.32 168.91))
-  (no_connect (at 228.6 104.14))
   (no_connect (at 20.32 158.75))
   (no_connect (at 92.71 177.8))
@@
   (no_connect (at 213.36 109.22))
   (no_connect (at 213.36 106.68))
-  (no_connect (at 228.6 101.6))
   (no_connect (at 149.86 175.26))
   (no_connect (at 92.71 172.72))
@@
   (no_connect (at 121.92 77.47))
   (no_connect (at 223.52 68.58))
-  (no_connect (at 93.98 120.65))
+  (no_connect (at 109.22 120.65))
   (no_connect (at 254 121.92))
   (no_connect (at 44.45 92.71))
@@
   (no_connect (at 109.22 95.25))
   (no_connect (at 254 96.52))
+  (no_connect (at 241.3 101.6))
+  (no_connect (at 241.3 104.14))
   (no_connect (at 142.24 138.43))
   (no_connect (at 123.19 172.72))
@@
     (stroke (width 0) (type default) (color 0 0 0 0))
   )
-  (wire (pts (xy 102.87 69.85) (xy 109.22 69.85))
+  (wire (pts (xy 101.6 66.04) (xy 107.95 66.04))
     (stroke (width 0) (type default) (color 0 0 0 0))
   )
@@
     (stroke (width 0) (type default) (color 0 0 0 0))
   )
+  (wire (pts (xy 101.6 68.58) (xy 107.95 68.58))
+    (stroke (width 0) (type default) (color 0 0 0 0))
+  )
   (wire (pts (xy 223.52 53.34) (xy 237.49 53.34))
     (stroke (width 0) (type default) (color 0 0 0 0))
@@
     (stroke (width 0) (type default) (color 0 0 0 0))
   )
-  (wire (pts (xy 109.22 120.65) (xy 93.98 120.65))
-    (stroke (width 0) (type default) (color 0 0 0 0))
-  )
   (wire (pts (xy 63.5 173.99) (xy 58.42 173.99))
     (stroke (width 0) (type default) (color 0 0 0 0))
@@
     (stroke (width 0) (type default) (color 0 0 0 0))
   )
-  (wire (pts (xy 241.3 101.6) (xy 228.6 101.6))
-    (stroke (width 0) (type default) (color 0 0 0 0))
-  )
   (polyline (pts (xy 156.21 63.5) (xy 156.21 161.29))
     (stroke (width 0) (type default) (color 0 0 0 0))
@@
     (stroke (width 0) (type default) (color 0 0 0 0))
   )
-  (wire (pts (xy 102.87 72.39) (xy 109.22 72.39))
-    (stroke (width 0) (type default) (color 0 0 0 0))
-  )
   (wire (pts (xy 175.26 53.34) (xy 175.26 63.5))
     (stroke (width 0) (type default) (color 0 0 0 0))
@@
     (stroke (width 0) (type default) (color 0 0 0 0))
   )
+  (wire (pts (xy 101.6 71.12) (xy 107.95 71.12))
+    (stroke (width 0) (type default) (color 0 0 0 0))
+  )
   (polyline (pts (xy 262.89 81.28) (xy 262.89 13.97))
     (stroke (width 0) (type default) (color 0 0 0 0))
@@
     (stroke (width 0) (type default) (color 0 0 0 0))
   )
-  (wire (pts (xy 102.87 77.47) (xy 104.14 77.47))
+  (wire (pts (xy 101.6 73.66) (xy 102.87 73.66))
     (stroke (width 0) (type default) (color 0 0 0 0))
   )
@@
     (stroke (width 0) (type default) (color 0 0 0 0))
   )
-  (wire (pts (xy 104.14 77.47) (xy 104.14 78.74))
+  (wire (pts (xy 102.87 73.66) (xy 102.87 74.93))
     (stroke (width 0) (type default) (color 0 0 0 0))
   )
@@
     (stroke (width 0) (type default) (color 0 0 0 0))
   )
-  (wire (pts (xy 102.87 74.93) (xy 109.22 74.93))
-    (stroke (width 0) (type default) (color 0 0 0 0))
-  )
   (wire (pts (xy 44.45 87.63) (xy 53.34 87.63))
     (stroke (width 0) (type default) (color 0 0 0 0))
@@
     (stroke (width 0) (type default) (color 0 0 0 0))
   )
-  (wire (pts (xy 241.3 104.14) (xy 228.6 104.14))
-    (stroke (width 0) (type default) (color 0 0 0 0))
-  )
   (wire (pts (xy 80.01 144.78) (xy 81.28 144.78))
     (stroke (width 0) (type default) (color 0 0 0 0))
@@
     (effects (font (size 1.27 1.27)) (justify left bottom))
   )
-  (label "PI_USB_D-" (at 228.6 104.14 0)
-    (effects (font (size 1.27 1.27)) (justify left bottom))
-  )
   (label "PI_SPI1_INT" (at 81.28 182.88 0)
     (effects (font (size 1.27 1.27)) (justify left bottom))
@@
     (effects (font (size 1.27 1.27)) (justify left bottom))
   )
-  (label "SWCLK" (at 109.22 74.93 180)
+  (label "SWCLK" (at 107.95 71.12 180)
     (effects (font (size 1.27 1.27)) (justify right bottom))
   )
@@
     (effects (font (size 1.27 1.27)) (justify left bottom))
   )
-  (label "SWO" (at 109.22 69.85 180)
+  (label "SWO" (at 107.95 66.04 180)
     (effects (font (size 1.27 1.27)) (justify right bottom))
   )
-  (label "PI_GPIO13" (at 227.33 149.86 180)
-    (effects (font (size 1.27 1.27)) (justify right bottom))
+  (label "SWDIO" (at 158.75 114.3 0)
+    (effects (font (size 1.27 1.27)) (justify left bottom))
   )
   (label "RSV17" (at 46.99 26.67 180)
@@
     (effects (font (size 1.27 1.27)) (justify left bottom))
   )
-  (label "PI_USB_D+" (at 228.6 101.6 0)
-    (effects (font (size 1.27 1.27)) (justify left bottom))
-  )
   (label "USER21" (at 12.7 123.19 0)
     (effects (font (size 1.27 1.27)) (justify left bottom))
@@
     (effects (font (size 1.27 1.27)) (justify right bottom))
   )
+  (label "SWCLK" (at 227.33 149.86 180)
+    (effects (font (size 1.27 1.27)) (justify right bottom))
+  )
   (label "PI_SCL" (at 133.35 156.21 0)
     (effects (font (size 1.27 1.27)) (justify left bottom))
@@
     (effects (font (size 1.27 1.27)) (justify right bottom))
   )
-  (label "PERSONALITY" (at 93.98 120.65 0)
-    (effects (font (size 1.27 1.27)) (justify left bottom))
-  )
   (label "USER23" (at 19.05 41.91 0)
     (effects (font (size 1.27 1.27)) (justify left bottom))
@@
     (effects (font (size 1.27 1.27)) (justify left bottom))
   )
-  (label "PI_GPIO16" (at 158.75 114.3 0)
-    (effects (font (size 1.27 1.27)) (justify left bottom))
-  )
   (label "RSV20" (at 46.99 34.29 180)
     (effects (font (size 1.27 1.27)) (justify right bottom))
@@
     (effects (font (size 1.27 1.27)) (justify left bottom))
   )
-  (label "BOOT0" (at 93.98 87.63 0)
-    (effects (font (size 1.27 1.27)) (justify left bottom))
-  )
   (label "USER16" (at 12.7 135.89 0)
     (effects (font (size 1.27 1.27)) (justify left bottom))
@@
     (effects (font (size 1.27 1.27)) (justify left bottom))
   )
-  (label "SWDIO" (at 109.22 72.39 180)
+  (label "SWDIO" (at 107.95 68.58 180)
     (effects (font (size 1.27 1.27)) (justify right bottom))
   )
@@
     (pin "3")
   )
-  (symbol (lib_id "Connector_Generic:Conn_01x04") (at 97.79 74.93 180) (unit 1)
+  (symbol (lib_id "Connector_Generic:Conn_01x04") (at 96.52 71.12 180) (unit 1)
     (in_bom yes) (on_board yes)
-    (property "Reference" "J9" (id 0) (at 100.33 78.74 0))
-    (property "Value" "Conn_01x04" (id 1) (at 99.8728 66.4464 0)
+    (property "Reference" "J9" (id 0) (at 99.06 74.93 0))
+    (property "Value" "Conn_01x04" (id 1) (at 98.6028 62.6364 0)
       (effects (font (size 1.27 1.27)) hide)
     )
-    (property "Footprint" "Connector_PinHeader_2.54mm:PinHeader_1x04_P2.54mm_Vertical" (id 2) (at 97.79 74.93 0)
+    (property "Footprint" "Connector_PinHeader_2.54mm:PinHeader_1x04_P2.54mm_Vertical" (id 2) (at 96.52 71.12 0)
       (effects (font (size 1.27 1.27)) hide)
     )
-    (property "Datasheet" "~" (id 3) (at 97.79 74.93 0)
+    (property "Datasheet" "~" (id 3) (at 96.52 71.12 0)
       (effects (font (size 1.27 1.27)) hide)
     )
-    (property "MPN" "PRPC004SAAN-RC" (id 4) (at 97.79 74.93 0)
+    (property "MPN" "PRPC004SAAN-RC" (id 4) (at 96.52 71.12 0)
       (effects (font (size 1.27 1.27)) hide)
     )
-    (property "Manufacturer" "Sullins Connector Solutions" (id 5) (at 97.79 74.93 0)
+    (property "Manufacturer" "Sullins Connector Solutions" (id 5) (at 96.52 71.12 0)
       (effects (font (size 1.27 1.27)) hide)
     )
-    (property "digkey.com" "S1011EC-04-DN" (id 6) (at 97.79 74.93 0)
+    (property "digkey.com" "S1011EC-04-DN" (id 6) (at 96.52 71.12 0)
       (effects (font (size 1.27 1.27)) hide)
     )
@@
     (pin "2")
   )
-  (symbol (lib_id "power:GND") (at 104.14 78.74 0) (unit 1)
+  (symbol (lib_id "power:GND") (at 102.87 74.93 0) (unit 1)
     (in_bom yes) (on_board yes)
-    (property "Reference" "#PWR055" (id 0) (at 104.14 85.09 0)
+    (property "Reference" "#PWR055" (id 0) (at 102.87 81.28 0)
       (effects (font (size 1.27 1.27)) hide)
     )
-    (property "Value" "GND" (id 1) (at 106.68 78.74 0))
-    (property "Footprint" "" (id 2) (at 104.14 78.74 0)
+    (property "Value" "GND" (id 1) (at 105.41 74.93 0))
+    (property "Footprint" "" (id 2) (at 102.87 74.93 0)
       (effects (font (size 1.27 1.27)) hide)
     )
-    (property "Datasheet" "" (id 3) (at 104.14 78.74 0)
+    (property "Datasheet" "" (id 3) (at 102.87 74.93 0)
       (effects (font (size 1.27 1.27)) hide)
     )
@@
   (symbol (lib_id "power:+5V") (at 187.96 91.44 0) (unit 1)
     (in_bom yes) (on_board yes)
-    (property "Reference" "#PWR?" (id 0) (at 187.96 95.25 0)
+    (property "Reference" "#PWR0112" (id 0) (at 187.96 95.25 0)
       (effects (font (size 1.27 1.27)) hide)
     )
@@
       (reference "#PWR0111") (unit 1) (value "+3V3") (footprint "")
     )
+    (path "/de7a585a-8b2b-4829-991d-a6a551151af8"
+      (reference "#PWR0112") (unit 1) (value "+5V") (footprint "")
+    )
     (path "/00000000-0000-0000-0000-0000626cb5b5"
       (reference "#PWR0114") (unit 1) (value "GND") (footprint "")
@@
       (reference "#PWR0134") (unit 1) (value "GND") (footprint "")
     )
-    (path "/de7a585a-8b2b-4829-991d-a6a551151af8"
-      (reference "#PWR?") (unit 1) (value "+5V") (footprint "")
-    )
     (path "/5b3c9143-4a88-4586-a41d-71dcd6e39798"

Commit message: pi-carrier: reassign GA0, GA1
Problem: STM34 OSC32 pins are used for GA0, GA1, so the RTC
cannot be clocked from the 32KHz clock source.

Reloacte GA0, GA1 to different GPIOs.
Connections:
- net GA0: now also U6.10 (PA0); no longer U6.4 (PC15)
- net GA1: now also U6.11 (PA1); no longer U6.3 (PC14)
- net PA0: no longer U6.10 (PA0)
- net PA1: no longer U6.11 (PA1)
- no-connect marks 39 -> 41
Changed lines of the file:
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@@
   (no_connect (at 213.36 109.22))
   (no_connect (at 213.36 106.68))
+  (no_connect (at 109.22 105.41))
+  (no_connect (at 109.22 102.87))
   (no_connect (at 149.86 175.26))
   (no_connect (at 92.71 172.72))
@@
     (stroke (width 0) (type default) (color 0 0 0 0))
   )
-  (wire (pts (xy 109.22 105.41) (xy 93.98 105.41))
-    (stroke (width 0) (type default) (color 0 0 0 0))
-  )
   (wire (pts (xy 109.22 118.11) (xy 93.98 118.11))
     (stroke (width 0) (type default) (color 0 0 0 0))
@@
   )
   (wire (pts (xy 20.32 97.79) (xy 12.7 97.79))
-    (stroke (width 0) (type default) (color 0 0 0 0))
-  )
-  (wire (pts (xy 109.22 102.87) (xy 93.98 102.87))
     (stroke (width 0) (type default) (color 0 0 0 0))
   )
@@
     (effects (font (size 1.27 1.27)) (justify left bottom))
   )
-  (label "PA0" (at 154.94 110.49 180)
-    (effects (font (size 1.27 1.27)) (justify right bottom))
-  )
   (label "CAN-" (at 53.34 158.75 180)
     (effects (font (size 1.27 1.27)) (justify right bottom))
@@
     (effects (font (size 1.27 1.27)) (justify right bottom))
   )
-  (label "GA0" (at 93.98 105.41 0)
-    (effects (font (size 1.27 1.27)) (justify left bottom))
+  (label "GA0" (at 154.94 110.49 180)
+    (effects (font (size 1.27 1.27)) (justify right bottom))
   )
   (label "PI_3V3" (at 153.67 175.26 270)
@@
     (effects (font (size 1.27 1.27)) (justify right bottom))
   )
-  (label "GA1" (at 93.98 102.87 0)
-    (effects (font (size 1.27 1.27)) (justify left bottom))
+  (label "GA1" (at 154.94 113.03 180)
+    (effects (font (size 1.27 1.27)) (justify right bottom))
   )
   (label "USER14" (at 12.7 140.97 0)
@@
     (effects (font (size 1.27 1.27)) (justify left bottom))
   )
-  (label "PA1" (at 154.94 113.03 180)
-    (effects (font (size 1.27 1.27)) (justify right bottom))
-  )
   (label "PI_SPI0_MISO" (at 227.33 137.16 180)

Commit message: pi-carrier: get rid of proto area
Problem: STM32 pins broken out in proto area are almost all
used now.

Get rid of proto area.
Parts:
- removed J8: 8x10 prototype area, 00_eurocard:protopad, symbol Connector_Generic:Conn_02x08_Counter_Clockwise
Connections:
- net PA2: no longer names the net of U6.12 (PA2)
- net PA3: no longer names the net of U6.13 (PA3)
- no-connect marks 41 -> 43
Other:
- note removed: "Proto area"
