File: hardware/pi-carrier/eurocard.kicad_sch (KiCad schematic)
At the start: 60 parts, among them J1 DIN41612_C96_male_ra_molliebus, J4 Conn_02x20_Odd_Even, J5 Conn_02x20_raspberry_pi4B, J7 button1, J8 button1, J9 Conn_02x05_Odd_Even, U1 SN74LVC1G07DBVR, U10 Lite-on LTP747KR, U11 TCAN332DR, U12 MCP2518FD, U2 TCAN332DR, U3 LM1117IMPX-3.3, U6 STM32F103C8T6, U8 SN74AHCT125PWR, U9 MAX7219CWG, X1 ASE-40.000MHz-LC, X2 ASE-8.000MHz-LC, Y1 ABS25-32.768KHZ-T

Commit message: pi-carrier: change 32.768khz xtal footprint
Problem: rtc xtal is too big

Go with Abracon ABS07-32.768KHZ-T (in stock at digikey).
Parts:
- Y1: value ABS25-32.768KHZ-T -> ABS07; footprint Crystal:Crystal_SMD_Abracon_ABS25-4Pin_8.0x3.8mm -> Crystal:Crystal_SMD_3215-2Pin_3.2x1.5mm
Changed lines of the file:
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@@
       (effects (font (size 1.27 1.27)) (justify right))
     )
-    (property "Value" "ABS25-32.768KHZ-T" (id 1) (at 86.868 91.186 90)
+    (property "Value" "ABS07" (id 1) (at 86.868 91.186 90)
       (effects (font (size 1.27 1.27)) (justify right))
     )
-    (property "Footprint" "Crystal:Crystal_SMD_Abracon_ABS25-4Pin_8.0x3.8mm" (id 2) (at 83.693 91.186 0)
+    (property "Footprint" "Crystal:Crystal_SMD_3215-2Pin_3.2x1.5mm" (id 2) (at 83.693 91.186 0)
       (effects (font (size 1.27 1.27)) hide)
     )
@@
     )
     (path "/4a56290b-e44d-4245-8f59-6421930de3a9"
-      (reference "Y1") (unit 1) (value "ABS25-32.768KHZ-T") (footprint "Crystal:Crystal_SMD_Abracon_ABS25-4Pin_8.0x3.8mm")
-    )
-  )
+      (reference "Y1") (unit 1) (value "ABS07") (footprint "Crystal:Crystal_SMD_3215-2Pin_3.2x1.5mm")
+    )
+  )

Commit message: pi-carrier: label some test points
Parts:
- added TP11: GND, TestPoint:TestPoint_Pad_1.0x1.0mm, symbol Connector:TestPoint
- TP1: value TestPoint -> 5V
- TP10: value TestPoint -> ~{RST}
- TP14: value TestPoint -> PI3V3
- TP2: value TestPoint -> 3V3
- TP3: value TestPoint -> 5VSB
- TP4: value TestPoint -> BATT
- TP5: value TestPoint -> 8MHz
- TP6: value TestPoint -> VBAT
- TP7: value TestPoint -> 40MHz
Connections:
- net GND: now also TP11.1
Other:
- note added: "5V polyfuse and 800mA 3V3 LDO"
- note removed: "5V polyfuse and 3V3 LDO"
Changed lines of the file:
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@@
   (junction (at 65.786 135.89) (diameter 0) (color 0 0 0 0)
   )
+  (junction (at 48.26 194.31) (diameter 0) (color 0 0 0 0)
+  )
   (junction (at 77.089 185.674) (diameter 0) (color 0 0 0 0)
   )
@@
     (stroke (width 0) (type default) (color 0 0 0 0))
   )
+  (wire (pts (xy 49.784 194.31) (xy 48.26 194.31))
+    (stroke (width 0) (type default) (color 0 0 0 0))
+  )
   (wire (pts (xy 223.52 33.02) (xy 255.27 33.02))
     (stroke (width 0) (type default) (color 0 0 0 0))
@@
     (stroke (width 0) (type default) (color 0 0 0 0))
   )
+  (wire (pts (xy 48.26 194.564) (xy 48.26 194.31))
+    (stroke (width 0) (type default) (color 0 0 0 0))
+  )
   (wire (pts (xy 123.19 179.07) (xy 135.255 179.07))
     (stroke (width 0) (type default) (color 0 0 0 0))
@@
     (stroke (width 0) (type default) (color 0 0 0 0))
   )
-  (text "5V polyfuse and 3V3 LDO" (at 20.574 201.93 0)
+  (text "5V polyfuse and 800mA 3V3 LDO" (at 17.399 202.057 0)
     (effects (font (size 1.4 1.4)) (justify left bottom))
   )
@@
       (effects (font (size 1.524 1.524)) (justify left))
     )
-    (property "Value" "SN74LVC1G07DBVR" (id 1) (at 124.46 25.4 0)
+    (property "Value" "SN74LVC1G07DBVR" (id 1) (at 114.808 24.765 0)
       (effects (font (size 0.9906 0.9906)) (justify left))
     )
@@
       (effects (font (size 1.27 1.27)) (justify left))
     )
-    (property "Value" "22uF 16V" (id 1) (at 42.926 193.294 0)
+    (property "Value" "22uF 16V" (id 1) (at 42.926 193.04 0)
       (effects (font (size 1.27 1.27)) (justify left))
     )
@@
       (effects (font (size 1.27 1.27)) (justify left))
     )
-    (property "Value" "TestPoint" (id 1) (at 83.3121 38.1 0)
+    (property "Value" "BATT" (id 1) (at 83.3121 38.1 0)
       (effects (font (size 1.27 1.27)) (justify left) hide)
     )
@@
       (effects (font (size 1.27 1.27)) (justify left))
     )
-    (property "Value" "TestPoint" (id 1) (at 132.715 184.6579 0)
+    (property "Value" "40MHz" (id 1) (at 132.715 184.6579 0)
       (effects (font (size 1.27 1.27)) (justify left) hide)
     )
@@
       (effects (font (size 1.27 1.27)) (justify left))
     )
-    (property "Value" "TestPoint" (id 1) (at 152.146 27.1779 0)
+    (property "Value" "~{RST}" (id 1) (at 152.146 27.1779 0)
       (effects (font (size 1.27 1.27)) (justify left) hide)
     )
@@
       (effects (font (size 1.27 1.27)) (justify left))
     )
-    (property "Value" "TestPoint" (id 1) (at 86.3601 71.628 0)
+    (property "Value" "8MHz" (id 1) (at 86.3601 71.628 0)
       (effects (font (size 1.27 1.27)) (justify left) hide)
     )
@@
     (pin "9")
   )
+  (symbol (lib_id "Connector:TestPoint") (at 49.784 194.31 270) (unit 1)
+    (in_bom yes) (on_board yes)
+    (property "Reference" "TP11" (id 0) (at 50.292 196.215 90)
+      (effects (font (size 1.27 1.27)) (justify left))
+    )
+    (property "Value" "GND" (id 1) (at 51.8161 196.85 0)
+      (effects (font (size 1.27 1.27)) (justify left) hide)
+    )
+    (property "Footprint" "TestPoint:TestPoint_Pad_1.0x1.0mm" (id 2) (at 49.784 199.39 0)
+      (effects (font (size 1.27 1.27)) hide)
+    )
+    (property "Datasheet" "~" (id 3) (at 49.784 199.39 0)
+      (effects (font (size 1.27 1.27)) hide)
+    )
+    (pin "1")
+  )
   (symbol (lib_id "Device:Crystal") (at 83.693 91.186 90) (unit 1)
     (in_bom yes) (on_board yes)
@@
       (effects (font (size 1.27 1.27)) (justify left))
     )
-    (property "Value" "TestPoint" (id 1) (at 203.073 91.9479 0)
+    (property "Value" "PI3V3" (id 1) (at 203.073 91.9479 0)
       (effects (font (size 1.27 1.27)) (justify left) hide)
     )
@@
       (effects (font (size 1.27 1.27)) (justify left))
     )
-    (property "Value" "TestPoint" (id 1) (at 79.2479 19.05 0)
+    (property "Value" "5VSB" (id 1) (at 79.2479 19.05 0)
       (effects (font (size 1.27 1.27)) (justify left) hide)
     )
@@
       (effects (font (size 1.27 1.27)) (justify left))
     )
-    (property "Value" "TestPoint" (id 1) (at 29.972 184.6579 0)
+    (property "Value" "5V" (id 1) (at 29.972 184.6579 0)
       (effects (font (size 1.27 1.27)) (justify left) hide)
     )
@@
       (effects (font (size 1.27 1.27)) (justify left))
     )
-    (property "Value" "TestPoint" (id 1) (at 101.092 28.4479 0)
+    (property "Value" "VBAT" (id 1) (at 101.092 28.4479 0)
       (effects (font (size 1.27 1.27)) (justify left) hide)
     )
@@
       (effects (font (size 1.27 1.27)) (justify left))
     )
-    (property "Value" "TestPoint" (id 1) (at 53.213 184.6579 0)
+    (property "Value" "3V3" (id 1) (at 53.213 184.6579 0)
       (effects (font (size 1.27 1.27)) (justify left) hide)
     )
@@
     )
     (path "/742cedd8-f59c-488a-90ba-ace1820f1544"
-      (reference "TP1") (unit 1) (value "TestPoint") (footprint "TestPoint:TestPoint_Pad_1.0x1.0mm")
+      (reference "TP1") (unit 1) (value "5V") (footprint "TestPoint:TestPoint_Pad_1.0x1.0mm")
     )
     (path "/fb7e9a73-660b-4b63-8b2d-48f26d03301c"
-      (reference "TP2") (unit 1) (value "TestPoint") (footprint "TestPoint:TestPoint_Pad_1.0x1.0mm")
+      (reference "TP2") (unit 1) (value "3V3") (footprint "TestPoint:TestPoint_Pad_1.0x1.0mm")
     )
     (path "/668d5884-c2f6-4856-b7cc-cb82034eb83b"
-      (reference "TP3") (unit 1) (value "TestPoint") (footprint "TestPoint:TestPoint_Pad_1.0x1.0mm")
+      (reference "TP3") (unit 1) (value "5VSB") (footprint "TestPoint:TestPoint_Pad_1.0x1.0mm")
     )
     (path "/1382e30f-e7c4-4888-9d15-af05cd61516f"
-      (reference "TP4") (unit 1) (value "TestPoint") (footprint "TestPoint:TestPoint_Pad_1.0x1.0mm")
+      (reference "TP4") (unit 1) (value "BATT") (footprint "TestPoint:TestPoint_Pad_1.0x1.0mm")
     )
     (path "/25f1ed64-1aca-4ace-a240-819442d64a2f"
-      (reference "TP5") (unit 1) (value "TestPoint") (footprint "TestPoint:TestPoint_Pad_1.0x1.0mm")
+      (reference "TP5") (unit 1) (value "8MHz") (footprint "TestPoint:TestPoint_Pad_1.0x1.0mm")
     )
     (path "/8896d593-d9f6-44e2-ae50-6a530075fd69"
-      (reference "TP6") (unit 1) (value "TestPoint") (footprint "TestPoint:TestPoint_Pad_1.0x1.0mm")
+      (reference "TP6") (unit 1) (value "VBAT") (footprint "TestPoint:TestPoint_Pad_1.0x1.0mm")
     )
     (path "/201081ef-0f25-4232-9497-fa1d74654379"
-      (reference "TP7") (unit 1) (value "TestPoint") (footprint "TestPoint:TestPoint_Pad_1.0x1.0mm")
+      (reference "TP7") (unit 1) (value "40MHz") (footprint "TestPoint:TestPoint_Pad_1.0x1.0mm")
     )
     (path "/1838f5b3-ada5-4ad1-9e7a-41b590633da3"
@@
     )
     (path "/20371431-6fbf-4ca4-9bfc-33b5b1c4838f"
-      (reference "TP10") (unit 1) (value "TestPoint") (footprint "TestPoint:TestPoint_Pad_1.0x1.0mm")
+      (reference "TP10") (unit 1) (value "~{RST}") (footprint "TestPoint:TestPoint_Pad_1.0x1.0mm")
+    )
+    (path "/3419fbe9-0846-41f3-8285-8e12eaf7e98d"
+      (reference "TP11") (unit 1) (value "GND") (footprint "TestPoint:TestPoint_Pad_1.0x1.0mm")
     )
     (path "/612988bd-f0e1-4325-995c-c88a8701fa16"
-      (reference "TP14") (unit 1) (value "TestPoint") (footprint "TestPoint:TestPoint_Pad_1.0x1.0mm")
+      (reference "TP14") (unit 1) (value "PI3V3") (footprint "TestPoint:TestPoint_Pad_1.0x1.0mm")
     )
     (path "/00000000-0000-0000-0000-00005e488a75"

Commit message: pi-carrier: add USB OTG connector to schematic
Problem: Molliebus reserves some pins for the pi USB 2 port,
to implement a low-speed ethernet gadget that would allow nodes
to have networking without anything plugged in externally.

Add a JST connector with USB_D- and USB_D+ pins routed to the bus.
A USB-C to JST connector would allow the pi 4B to hook into this.
Parts:
- added J2: usb, Connector_JST:JST_SH_SM03B-SRSS-TB_1x03-1MP_P1.00mm_Horizontal, symbol Connector_Generic_MountingPin:Conn_01x03_MountingPin
Connections:
- net GND: now also J1.a21 (USB_GND), J2.3 (Pin_3), J2.MP (MountPin)
- net SCL: now also TP9.1
- net SDA: now also TP8.1
- net USB_D-: now reaches J1.a19 (USB_D-)
- net USB_D-: now also J2.1 (Pin_1)
- net USB_D+: now reaches J1.a20 (USB_D+)
- net USB_D+: now also J2.2 (Pin_2)
- no-connect marks 61 -> 58
Other:
- note added: "USB OTG"
- moved on the sheet: C10, C12, C13, C15, C16, C6, D3, R12, R13, R14, R15, R16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

Commit message: pi-carrier: add more test points
Problem: some key probing points are still inaccessible.

Expand test points.  Change "value" field to match function.
Parts:
- added TP12: CAN+, TestPoint:TestPoint_Pad_1.0x1.0mm, symbol Connector:TestPoint
- added TP13: CAN-, TestPoint:TestPoint_Pad_1.0x1.0mm, symbol Connector:TestPoint
- added TP15: NSS, TestPoint:TestPoint_Pad_1.0x1.0mm, symbol Connector:TestPoint
- added TP16: SCK, TestPoint:TestPoint_Pad_1.0x1.0mm, symbol Connector:TestPoint
- added TP17: MOSI, TestPoint:TestPoint_Pad_1.0x1.0mm, symbol Connector:TestPoint
- TP3: value 5VSB -> SB
- TP4: value BATT -> CELL
- TP8: value TestPoint -> SDA
- TP9: value TestPoint -> SCL
Connections:
- net CAN+: now also TP12.1
- net CAN-: now also TP13.1
- net MOSI: now also TP17.1
- net NSS: now also TP15.1
- net SCK: now also TP16.1
Other:
- note added: "Reset"
- note removed: "reset generation (power on or bus 5V)"

Commit message: pi-carrier: adjust 32.768kHz xtal circuit
Problem: the stm32f103c8 data sheet provides some information
on LSE xtal selection load capacitance in sec 5.3.6.  It includes
the statement that one should never use a resonator with a load
capacitance of 12.5pF which is exactly what we have.

Switch to a part that has 6pF load capacitance, just mimicing the
example provided:  Cl = 6pF Cstray = 2pF => Cl1 = Cl2 = 8pF.
Adjust caps accordingly.
Parts:
- C13, C6: value 20pf -> 8pf
- Y1: value ABS07 -> ABS07-32.768KHZ-6-T
Changed lines of the file:
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@@
       (effects (font (size 1.27 1.27)) (justify left))
     )
-    (property "Value" "20pf" (id 1) (at 80.137 101.346 90)
+    (property "Value" "8pf" (id 1) (at 80.137 101.346 90)
       (effects (font (size 1.27 1.27)) (justify left))
     )
@@
       (effects (font (size 1.27 1.27)) (justify right))
     )
-    (property "Value" "ABS07" (id 1) (at 86.487 98.806 90)
+    (property "Value" "ABS07-32.768KHZ-6-T" (id 1) (at 78.74 103.8352 90)
       (effects (font (size 1.27 1.27)) (justify right))
     )
@@
       (effects (font (size 1.27 1.27)) (justify left))
     )
-    (property "Value" "20pf" (id 1) (at 80.137 93.726 90)
+    (property "Value" "8pf" (id 1) (at 80.137 93.726 90)
       (effects (font (size 1.27 1.27)) (justify left))
     )
@@
     )
     (path "/d722c931-abc0-4448-bdf4-321f37863a97"
-      (reference "C6") (unit 1) (value "20pf") (footprint "Capacitor_SMD:C_0603_1608Metric")
+      (reference "C6") (unit 1) (value "8pf") (footprint "Capacitor_SMD:C_0603_1608Metric")
     )
     (path "/00000000-0000-0000-0000-00005ee4c209"
@@
     )
     (path "/2c4e9f3e-b7f0-4d93-8152-df5a959ae4a3"
-      (reference "C13") (unit 1) (value "20pf") (footprint "Capacitor_SMD:C_0603_1608Metric")
+      (reference "C13") (unit 1) (value "8pf") (footprint "Capacitor_SMD:C_0603_1608Metric")
     )
     (path "/00000000-0000-0000-0000-00005f7ef160"
@@
     )
     (path "/4a56290b-e44d-4245-8f59-6421930de3a9"
-      (reference "Y1") (unit 1) (value "ABS07") (footprint "Crystal:Crystal_SMD_3215-2Pin_3.2x1.5mm")
-    )
-  )
+      (reference "Y1") (unit 1) (value "ABS07-32.768KHZ-6-T") (footprint "Crystal:Crystal_SMD_3215-2Pin_3.2x1.5mm")
+    )
+  )

Commit message: pi-carrier: fix R12, R13 connection to +3V3
Connections:
- net +3V3: now also R12.1, R13.1
Other:
- moved on the sheet: R12, TP8, TP9
Changed lines of the file:
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@@
   (junction (at 65.405 135.89) (diameter 0) (color 0 0 0 0)
   )
-  (junction (at 148.209 69.215) (diameter 0) (color 0 0 0 0)
-  )
   (junction (at 261.62 27.94) (diameter 0) (color 0 0 0 0)
   )
@@
   (junction (at 125.857 69.596) (diameter 0) (color 0 0 0 0)
   )
+  (junction (at 148.082 70.104) (diameter 0) (color 0 0 0 0)
+  )
   (junction (at 98.552 30.48) (diameter 0) (color 0 0 0 0)
   )
   (junction (at 144.78 29.21) (diameter 0) (color 0 0 0 0)
   )
-  (junction (at 139.319 69.088) (diameter 0) (color 0 0 0 0)
-  )
   (junction (at 46.355 140.462) (diameter 0) (color 0 0 0 0)
   )
   (junction (at 71.247 193.294) (diameter 0) (color 0 0 0 0)
   )
-  (junction (at 139.319 69.215) (diameter 0) (color 0 0 0 0)
-  )
   (junction (at 187.96 165.1) (diameter 0) (color 0 0 0 0)
   )
@@
   (junction (at 81.28 21.59) (diameter 0) (color 0 0 0 0)
   )
+  (junction (at 138.938 70.104) (diameter 0) (color 0 0 0 0)
+  )
   (junction (at 83.947 76.708) (diameter 0) (color 0 0 0 0)
   )
@@
   (junction (at 237.49 154.94) (diameter 0) (color 0 0 0 0)
   )
-  (junction (at 148.209 74.295) (diameter 0) (color 0 0 0 0)
+  (junction (at 148.082 74.422) (diameter 0) (color 0 0 0 0)
   )
   (junction (at 95.25 30.48) (diameter 0) (color 0 0 0 0)
@@
     (stroke (width 0) (type default) (color 0 0 0 0))
   )
-  (wire (pts (xy 153.289 74.295) (xy 148.209 74.295))
+  (wire (pts (xy 153.162 74.422) (xy 148.082 74.422))
     (stroke (width 0) (type default) (color 0 0 0 0))
   )
@@
     (stroke (width 0) (type default) (color 0 0 0 0))
   )
+  (wire (pts (xy 138.938 74.422) (xy 140.462 74.422))
+    (stroke (width 0) (type default) (color 0 0 0 0))
+  )
   (wire (pts (xy 196.85 63.5) (xy 203.2 63.5))
     (stroke (width 0) (type default) (color 0 0 0 0))
@@
     (stroke (width 0) (type default) (color 0 0 0 0))
   )
-  (wire (pts (xy 139.319 69.215) (xy 139.319 74.295))
-    (stroke (width 0) (type default) (color 0 0 0 0))
-  )
   (polyline (pts (xy 65.532 14.986) (xy 41.402 14.986))
     (stroke (width 0) (type default) (color 0 0 0 0))
@@
     (stroke (width 0) (type default) (color 0 0 0 0))
   )
-  (wire (pts (xy 139.319 67.818) (xy 139.319 69.088))
-    (stroke (width 0) (type default) (color 0 0 0 0))
-  )
   (wire (pts (xy 123.317 145.796) (xy 123.317 147.066))
     (stroke (width 0) (type default) (color 0 0 0 0))
@@
     (stroke (width 0) (type default) (color 0 0 0 0))
   )
-  (wire (pts (xy 153.289 69.215) (xy 148.209 69.215))
+  (wire (pts (xy 153.162 70.104) (xy 148.082 70.104))
     (stroke (width 0) (type default) (color 0 0 0 0))
   )
@@
     (stroke (width 0) (type default) (color 0 0 0 0))
   )
-  (wire (pts (xy 139.319 74.295) (xy 140.589 74.295))
-    (stroke (width 0) (type default) (color 0 0 0 0))
-  )
   (polyline (pts (xy 57.404 156.718) (xy 157.226 156.718))
     (stroke (width 0) (type default) (color 0 0 0 0))
@@
     (stroke (width 0) (type default) (color 0 0 0 0))
   )
-  (wire (pts (xy 139.319 69.215) (xy 140.589 69.215))
-    (stroke (width 0) (type default) (color 0 0 0 0))
-  )
   (wire (pts (xy 251.46 127) (xy 266.7 127))
     (stroke (width 0) (type default) (color 0 0 0 0))
@@
     (stroke (width 0) (type default) (color 0 0 0 0))
   )
+  (wire (pts (xy 138.938 68.58) (xy 138.938 70.104))
+    (stroke (width 0) (type default) (color 0 0 0 0))
+  )
   (wire (pts (xy 251.46 144.78) (xy 266.7 144.78))
     (stroke (width 0) (type default) (color 0 0 0 0))
@@
     (stroke (width 0) (type default) (color 0 0 0 0))
   )
+  (wire (pts (xy 138.938 74.422) (xy 138.938 70.104))
+    (stroke (width 0) (type default) (color 0 0 0 0))
+  )
   (polyline (pts (xy 166.37 85.09) (xy 262.89 85.09))
     (stroke (width 0) (type default) (color 0 0 0 0))
@@
     (stroke (width 0) (type default) (color 0 0 0 0))
   )
+  (wire (pts (xy 138.938 70.104) (xy 140.462 70.104))
+    (stroke (width 0) (type default) (color 0 0 0 0))
+  )
   (wire (pts (xy 130.175 186.69) (xy 137.16 186.69))
     (stroke (width 0) (type default) (color 0 0 0 0))
@@
     (effects (font (size 1.27 1.27)) (justify left bottom))
   )
-  (label "SDA" (at 153.289 69.215 180)
+  (label "SDA" (at 153.162 70.104 180)
     (effects (font (size 1.27 1.27)) (justify right bottom))
   )
@@
     (effects (font (size 1.27 1.27)) (justify right bottom))
   )
-  (label "SCL" (at 153.289 74.295 180)
+  (label "SCL" (at 153.162 74.422 180)
     (effects (font (size 1.27 1.27)) (justify right bottom))
   )
@@
     (pin "1")
   )
-  (symbol (lib_id "Connector:TestPoint") (at 148.209 69.215 0) (unit 1)
+  (symbol (lib_id "Connector:TestPoint") (at 148.082 70.104 0) (unit 1)
     (in_bom yes) (on_board yes)
-    (property "Reference" "TP8" (id 0) (at 148.971 65.405 0)
+    (property "Reference" "TP8" (id 0) (at 148.844 66.294 0)
       (effects (font (size 1.27 1.27)) (justify left))
     )
-    (property "Value" "SDA" (id 1) (at 150.749 67.1829 0)
+    (property "Value" "SDA" (id 1) (at 150.622 68.0719 0)
       (effects (font (size 1.27 1.27)) (justify left) hide)
     )
-    (property "Footprint" "TestPoint:TestPoint_Pad_1.0x1.0mm" (id 2) (at 153.289 69.215 0)
+    (property "Footprint" "TestPoint:TestPoint_Pad_1.0x1.0mm" (id 2) (at 153.162 70.104 0)
       (effects (font (size 1.27 1.27)) hide)
     )
-    (property "Datasheet" "~" (id 3) (at 153.289 69.215 0)
+    (property "Datasheet" "~" (id 3) (at 153.162 70.104 0)
       (effects (font (size 1.27 1.27)) hide)
     )
@@
     (pin "1")
   )
-  (symbol (lib_id "Device:R") (at 144.399 69.215 90) (mirror x) (unit 1)
+  (symbol (lib_id "Device:R") (at 144.272 70.104 90) (mirror x) (unit 1)
     (in_bom yes) (on_board yes)
-    (property "Reference" "R12" (id 0) (at 142.494 67.31 90)
+    (property "Reference" "R12" (id 0) (at 142.24 68.072 90)
       (effects (font (size 1.27 1.27)) (justify right))
     )
-    (property "Value" "4.7K" (id 1) (at 141.859 69.215 90)
+    (property "Value" "4.7K" (id 1) (at 141.732 70.104 90)
       (effects (font (size 1.27 1.27)) (justify right))
     )
-    (property "Footprint" "Resistor_SMD:R_0603_1608Metric" (id 2) (at 144.399 67.437 90)
+    (property "Footprint" "Resistor_SMD:R_0603_1608Metric" (id 2) (at 144.272 68.326 90)
       (effects (font (size 1.27 1.27)) hide)
     )
-    (property "Datasheet" "~" (id 3) (at 144.399 69.215 0)
+    (property "Datasheet" "~" (id 3) (at 144.272 70.104 0)
       (effects (font (size 1.27 1.27)) hide)
     )
@@
     (pin "1")
   )
-  (symbol (lib_id "Device:R") (at 144.399 74.295 90) (mirror x) (unit 1)
+  (symbol (lib_id "Device:R") (at 144.272 74.422 90) (mirror x) (unit 1)
     (in_bom yes) (on_board yes)
-    (property "Reference" "R13" (id 0) (at 142.367 72.263 90)
+    (property "Reference" "R13" (id 0) (at 142.494 72.39 90)
       (effects (font (size 1.27 1.27)) (justify right))
     )
-    (property "Value" "4.7K" (id 1) (at 141.859 74.295 90)
+    (property "Value" "4.7K" (id 1) (at 141.732 74.422 90)
       (effects (font (size 1.27 1.27)) (justify right))
     )
-    (property "Footprint" "Resistor_SMD:R_0603_1608Metric" (id 2) (at 144.399 72.517 90)
+    (property "Footprint" "Resistor_SMD:R_0603_1608Metric" (id 2) (at 144.272 72.644 90)
       (effects (font (size 1.27 1.27)) hide)
     )
-    (property "Datasheet" "~" (id 3) (at 144.399 74.295 0)
+    (property "Datasheet" "~" (id 3) (at 144.272 74.422 0)
       (effects (font (size 1.27 1.27)) hide)
     )
@@
     (pin "2")
   )
-  (symbol (lib_id "Connector:TestPoint") (at 148.209 74.295 0) (unit 1)
+  (symbol (lib_id "Connector:TestPoint") (at 148.082 74.422 180) (unit 1)
     (in_bom yes) (on_board yes)
-    (property "Reference" "TP9" (id 0) (at 148.971 70.231 0)
+    (property "Reference" "TP9" (id 0) (at 149.86 79.502 0)
       (effects (font (size 1.27 1.27)) (justify left))
     )
-    (property "Value" "SCL" (id 1) (at 150.749 72.2629 0)
+    (property "Value" "SCL" (id 1) (at 145.542 76.4541 0)
       (effects (font (size 1.27 1.27)) (justify left) hide)
     )
-    (property "Footprint" "TestPoint:TestPoint_Pad_1.0x1.0mm" (id 2) (at 153.289 74.295 0)
+    (property "Footprint" "TestPoint:TestPoint_Pad_1.0x1.0mm" (id 2) (at 143.002 74.422 0)
       (effects (font (size 1.27 1.27)) hide)
     )
-    (property "Datasheet" "~" (id 3) (at 153.289 74.295 0)
+    (property "Datasheet" "~" (id 3) (at 143.002 74.422 0)
       (effects (font (size 1.27 1.27)) hide)
     )
@@
     (pin "1")
   )
-  (symbol (lib_id "power:+3V3") (at 139.319 67.818 0) (mirror y) (unit 1)
+  (symbol (lib_id "power:+3V3") (at 138.938 68.58 0) (mirror y) (unit 1)
     (in_bom yes) (on_board yes)
-    (property "Reference" "#PWR054" (id 0) (at 139.319 71.628 0)
+    (property "Reference" "#PWR054" (id 0) (at 138.938 72.39 0)
       (effects (font (size 1.27 1.27)) hide)
     )
-    (property "Value" "+3V3" (id 1) (at 136.144 65.913 0))
-    (property "Footprint" "" (id 2) (at 139.319 67.818 0)
+    (property "Value" "+3V3" (id 1) (at 138.2776 65.024 0))
+    (property "Footprint" "" (id 2) (at 138.938 68.58 0)
       (effects (font (size 1.27 1.27)) hide)
     )
-    (property "Datasheet" "" (id 3) (at 139.319 67.818 0)
+    (property "Datasheet" "" (id 3) (at 138.938 68.58 0)
       (effects (font (size 1.27 1.27)) hide)
     )
