File: hardware/pi-carrier/eurocard.kicad_sch (KiCad schematic)
At the start: 67 parts, among them J1 DIN41612_C96_male_ra_molliebus, J2 usb, J4 Conn_02x20_Odd_Even, J5 Conn_02x20_raspberry_pi4B, J7 button1, J8 button1, J9 Conn_02x05_Odd_Even, U1 SN74LVC1G07DBVR, U10 Lite-on LTP747KR, U11 TCAN332DR, U12 MCP2518FD, U2 TCAN332DR, U3 LM1117IMPX-3.3, U6 STM32F103C8T6, U8 SN74AHCT125PWR, U9 MAX7219CWG, X1 ASE-40.000MHz-LC, X2 ASE-8.000MHz-LC, Y1 ABS07-32.768KHZ-6-T

Commit message: pi-carrier: tweak test points
Parts:
- added TP18: PB4, TestPoint:TestPoint_Pad_1.0x1.0mm, symbol Connector:TestPoint
- added TP19: PA6, TestPoint:TestPoint_Pad_1.0x1.0mm, symbol Connector:TestPoint
- added TP20: PA7, TestPoint:TestPoint_Pad_1.0x1.0mm, symbol Connector:TestPoint
- added TP21: PA11, TestPoint:TestPoint_Pad_1.0x1.0mm, symbol Connector:TestPoint
- added TP22: PA12, TestPoint:TestPoint_Pad_1.0x1.0mm, symbol Connector:TestPoint
- added TP23: PA15, TestPoint:TestPoint_Pad_1.0x1.0mm, symbol Connector:TestPoint
- F1: footprint Fuse:Fuse_1812_4532Metric_Pad1.30x3.40mm_HandSolder -> Fuse:Fuse_1812_4532Metric
- TP3: value SB -> STBY
Connections:
- net at U6.16 (PA6): now also TP19.1
- net at U6.17 (PA7): now also TP20.1
- net at U6.32 (PA11): now also TP21.1
- net at U6.33 (PA12): now also TP22.1
- net at U6.38 (PA15): now also TP23.1
- net at U6.40 (PB4): now also TP18.1
- no-connect marks 58 -> 52
Other:
- moved on the sheet: C10, C12, C13, C15, C16, C6, D3, R12, R13, R14, R15, R16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

Commit message: pi-carrier: add wired or logic
Parts:
- removed TP23: PA15, TestPoint:TestPoint_Pad_1.0x1.0mm, symbol Connector:TestPoint
- added C3, C8: 100nF 16V, Capacitor_SMD:C_0603_1608Metric, symbol Device:C
- added U4: 74LVC2G04, Package_TO_SOT_SMD:SOT-23-6, symbol 74xGxx:74LVC2G04
- added U5: 74LVC2G38, Package_SO:VSSOP-8_2.3x2mm_P0.5mm, symbol 74xGxx:74LVC2G38
Connections:
- net +3V3: now also C3.1, C8.1, U4.5 (VCC), U4.5 (VCC), U5.8 (VCC), U5.8 (VCC)
- net GND: now also C3.2, C8.2, U4.2 (GND), U4.2 (GND), U5.4 (GND), U5.4 (GND)
- net OR_INA: now reaches J1.a15 (OR_INA)
- net OR_INA: now also U5.7
- net OR_INB: now reaches J1.a16 (OR_INB)
- net OR_INB: now also U5.3
- net OR_OUT: now reaches J1.a17 (OR_OUT)
- net OR_OUT: now also U4.3
- net BARRIER_EN: now reaches U6.38 (PA15)
- net BARRIER_EN: now also U5.1, U5.5
- net GPIO5 renamed BARRIER_OUT
- net BARRIER_OUT: now also U4.1, U5.6
- net GPIO6 renamed BARRIER_IN
- net BARRIER_IN: now also U4.4
- new net: U4.6, U5.2
- no-connect marks 52 -> 49
Other:
- note added: "Wired-OR Barrier"
- note added: "opt power button"
- note removed: "Pi PMIC header"
- note removed: "STM32 SWD"
- note removed: "USB OTG"
- note removed: "boot from user flash"
- note removed: "power button (opt)"
- moved on the sheet: BT1, C14, C20, C9, D1, J1, J2, J7, J8, J9, R1, R14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
