File: hardware/pi-carrier/eurocard.kicad_sch (KiCad schematic)
At the start: 79 parts, among them J1 DIN41612_C96_male_ra_molliebus, J2 Debug, J3 Console, J4 Conn_02x20_Odd_Even, J5 Conn_02x20_raspberry_pi4B, J9 Conn_02x05_Odd_Even, U1 74LVC1G07, U10 Lite-on LTP747KR, U11 TCAN332DR, U12 MCP2518FD, U2 TCAN332DR, U3 LM1117IMPX-3.3, U4 74LVC2G04, U5 74LVC2G38, U6 STM32F103C8T6, U8 SN74AHCT125PWR, U9 MAX7219CWG, X1 ASE-40.000MHz-LC, X2 ASE-8.000MHz-LC, Y1 ABS07-32.768KHZ-6-T

Commit message: pi-carrier: drop 3-pin debug connector
Problem: meh, extra 3-pin debug connector is not too helpful.

Drop it.
Parts:
- removed J2: Debug, Connector_JST:JST_SH_BM03B-SRSS-TB_1x03-1MP_P1.00mm_Vertical, symbol Connector_Generic_MountingPin:Conn_01x03_MountingPin
Changed lines of the file:
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@@
   (junction (at 38.1 17.78) (diameter 0) (color 0 0 0 0)
   )
-  (junction (at 110.49 64.77) (diameter 0) (color 0 0 0 0)
-  )
   (junction (at 82.55 96.52) (diameter 0) (color 0 0 0 0)
   )
@@
     (stroke (width 0) (type default))
   )
+  (wire (pts (xy 86.36 54.61) (xy 93.98 54.61))
+    (stroke (width 0) (type default))
+  )
   (polyline (pts (xy 161.29 86.36) (xy 266.7 86.36))
     (stroke (width 0) (type default))
@@
     (stroke (width 0) (type default))
   )
-  (wire (pts (xy 86.36 54.61) (xy 105.41 54.61))
-    (stroke (width 0) (type default))
-  )
-  (wire (pts (xy 86.36 57.15) (xy 97.79 57.15))
+  (wire (pts (xy 86.36 57.15) (xy 93.98 57.15))
     (stroke (width 0) (type default))
   )
@@
     (stroke (width 0) (type default))
   )
-  (wire (pts (xy 105.41 57.15) (xy 105.41 64.77))
-    (stroke (width 0) (type default))
-  )
   (polyline (pts (xy 124.46 45.72) (xy 124.46 13.97))
     (stroke (width 0) (type default))
@@
     (stroke (width 0) (type default))
   )
-  (wire (pts (xy 105.41 64.77) (xy 110.49 64.77))
-    (stroke (width 0) (type default))
-  )
   (wire (pts (xy 119.38 148.59) (xy 119.38 151.13))
     (stroke (width 0) (type default))
@@
     (stroke (width 0) (type default))
   )
-  (wire (pts (xy 97.79 59.69) (xy 105.41 59.69))
-    (stroke (width 0) (type default))
-  )
   (wire (pts (xy 213.36 114.3) (xy 226.06 114.3))
     (stroke (width 0) (type default))
@@
     (stroke (width 0) (type default))
   )
-  (wire (pts (xy 97.79 57.15) (xy 97.79 59.69))
-    (stroke (width 0) (type default))
-  )
   (wire (pts (xy 223.52 50.8) (xy 237.49 50.8))
     (stroke (width 0) (type default))
@@
     )
   )
-  (symbol (lib_id "power:GND") (at 110.49 64.77 0) (unit 1)
-    (in_bom yes) (on_board yes) (dnp no)
-    (property "Reference" "#PWR014" (at 110.49 71.12 0)
-      (effects (font (size 1.27 1.27)) hide)
-    )
-    (property "Value" "GND" (at 107.95 67.945 0)
-      (effects (font (size 1.27 1.27)))
-    )
-    (property "Footprint" "" (at 110.49 64.77 0)
-      (effects (font (size 1.27 1.27)) hide)
-    )
-    (property "Datasheet" "" (at 110.49 64.77 0)
-      (effects (font (size 1.27 1.27)) hide)
-    )
-    (pin "1")
-    (instances
-      (project "eurocard"
-        (path "/e048be62-6e5d-4330-8748-f1a6c1c5d89d"
-          (reference "#PWR014") (unit 1)
-        )
-      )
-    )
-  )
   (symbol (lib_id "Connector:TestPoint") (at 171.45 58.42 180) (unit 1)
     (in_bom yes) (on_board yes) (dnp no)
@@
         )
       )
-    )
-  )
-  (symbol (lib_id "Connector_Generic_MountingPin:Conn_01x03_MountingPin") (at 110.49 57.15 0) (unit 1)
-    (in_bom yes) (on_board yes) (dnp no)
-    (property "Reference" "J2" (at 109.22 52.07 0)
-      (effects (font (size 1.27 1.27)) (justify left))
-    )
-    (property "Value" "Debug" (at 112.395 57.15 0)
-      (effects (font (size 1.27 1.27)) (justify left))
-    )
-    (property "Footprint" "Connector_JST:JST_SH_BM03B-SRSS-TB_1x03-1MP_P1.00mm_Vertical" (at 110.49 57.15 0)
-      (effects (font (size 1.27 1.27)) hide)
-    )
-    (property "Datasheet" "~" (at 110.49 57.15 0)
-      (effects (font (size 1.27 1.27)) hide)
-    )
-    (pin "1")
-    (pin "3")
-    (pin "MP")
-    (pin "2")
-    (instances
-      (project "eurocard"
-        (path "/e048be62-6e5d-4330-8748-f1a6c1c5d89d"
-          (reference "J2") (unit 1)
-        )
-      )

Commit message: pi-carrier: add 3-pin power connector
Problem: RUN_PG and GLOBAL_EN should be via a connector
rather than solderd in.

Replace the testpoints on the back of the board with a 3-pin
JST connector on the front of the board.
Parts:
- removed TP25, TP26: TestPoint, TestPoint:TestPoint_Pad_1.0x1.0mm, symbol Connector:TestPoint
- added J2: Console, Connector_JST:JST_SH_SM03B-SRSS-TB_1x03-1MP_P1.00mm_Horizontal, symbol Connector_Generic_MountingPin:Conn_01x03_MountingPin
Connections:
- net GLOBAL_EN: now also J2.2 (Pin_2)
- net GND: now also J2.3 (Pin_3), J2.MP (MountPin)
- net RUN_PG: now also J2.1 (Pin_1)
Changed lines of the file:
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@@
   (junction (at 71.12 185.42) (diameter 0) (color 0 0 0 0)
   )
+  (junction (at 236.22 100.33) (diameter 0) (color 0 0 0 0)
+  )
   (junction (at 167.64 106.68) (diameter 0) (color 0 0 0 0)
   )
@@
     (stroke (width 0) (type default))
   )
+  (wire (pts (xy 231.14 95.25) (xy 231.14 100.33))
+    (stroke (width 0) (type default))
+  )
   (wire (pts (xy 63.5 171.45) (xy 58.42 171.45))
     (stroke (width 0) (type default))
@@
     (stroke (width 0) (type default))
   )
+  (wire (pts (xy 218.44 90.17) (xy 231.14 90.17))
+    (stroke (width 0) (type default))
+  )
   (wire (pts (xy 236.22 30.48) (xy 236.22 27.94))
     (stroke (width 0) (type default))
@@
     (stroke (width 0) (type default))
   )
-  (wire (pts (xy 254 92.71) (xy 254 100.33))
-    (stroke (width 0) (type default))
-  )
   (wire (pts (xy 90.17 30.48) (xy 90.17 33.02))
     (stroke (width 0) (type default))
@@
     (stroke (width 0) (type default))
   )
+  (wire (pts (xy 254 92.71) (xy 252.73 92.71))
+    (stroke (width 0) (type default))
+  )
   (wire (pts (xy 194.31 48.26) (xy 196.85 48.26))
     (stroke (width 0) (type default))
@@
     (stroke (width 0) (type default))
   )
-  (wire (pts (xy 170.18 88.9) (xy 180.34 88.9))
-    (stroke (width 0) (type default))
-  )
   (wire (pts (xy 13.97 181.61) (xy 24.13 181.61))
     (stroke (width 0) (type default))
@@
     (stroke (width 0) (type default))
   )
-  (wire (pts (xy 254 100.33) (xy 259.08 100.33))
-    (stroke (width 0) (type default))
-  )
   (wire (pts (xy 48.26 186.69) (xy 50.8 186.69))
     (stroke (width 0) (type default))
@@
     (stroke (width 0) (type default))
   )
+  (wire (pts (xy 252.73 100.33) (xy 259.08 100.33))
+    (stroke (width 0) (type default))
+  )
   (wire (pts (xy 137.16 134.62) (xy 142.24 134.62))
     (stroke (width 0) (type default))
@@
     (stroke (width 0) (type default))
   )
+  (wire (pts (xy 218.44 92.71) (xy 231.14 92.71))
+    (stroke (width 0) (type default))
+  )
   (wire (pts (xy 175.26 63.5) (xy 175.26 71.12))
     (stroke (width 0) (type default))
@@
     (stroke (width 0) (type default))
   )
+  (wire (pts (xy 252.73 92.71) (xy 252.73 100.33))
+    (stroke (width 0) (type default))
+  )
   (wire (pts (xy 196.85 48.26) (xy 196.85 63.5))
     (stroke (width 0) (type default))
@@
     (stroke (width 0) (type default))
   )
-  (wire (pts (xy 168.91 91.44) (xy 180.34 91.44))
-    (stroke (width 0) (type default))
-  )
   (wire (pts (xy 46.99 144.78) (xy 55.88 144.78))
     (stroke (width 0) (type default))
@@
     (stroke (width 0) (type default))
   )
+  (wire (pts (xy 231.14 100.33) (xy 236.22 100.33))
+    (stroke (width 0) (type default))
+  )
   (wire (pts (xy 223.52 35.56) (xy 252.73 35.56))
     (stroke (width 0) (type default))
@@
     (effects (font (size 1.27 1.27)) (justify left bottom))
   )
-  (label "RUN_PG" (at 180.34 88.9 180) (fields_autoplaced)
-    (effects (font (size 1.27 1.27)) (justify right bottom))
-  )
   (label "CAN-" (at 55.88 144.78 180) (fields_autoplaced)
     (effects (font (size 1.27 1.27)) (justify right bottom))
@@
     (effects (font (size 1.27 1.27)) (justify right bottom))
   )
+  (label "GLOBAL_EN" (at 218.44 92.71 0) (fields_autoplaced)
+    (effects (font (size 1.27 1.27)) (justify left bottom))
+  )
   (label "GA3" (at 55.88 129.54 180) (fields_autoplaced)
     (effects (font (size 1.27 1.27)) (justify right bottom))
@@
     (effects (font (size 1.27 1.27)) (justify right bottom))
   )
+  (label "RUN_PG" (at 218.44 90.17 0) (fields_autoplaced)
+    (effects (font (size 1.27 1.27)) (justify left bottom))
+  )
   (label "SWDIO" (at 149.86 137.16 180) (fields_autoplaced)
     (effects (font (size 1.27 1.27)) (justify right bottom))
@@
     (effects (font (size 1.27 1.27)) (justify right bottom))
   )
-  (label "GLOBAL_EN" (at 180.34 91.44 180) (fields_autoplaced)
-    (effects (font (size 1.27 1.27)) (justify right bottom))
-  )
   (symbol (lib_id "power:GND") (at 73.66 111.76 90) (unit 1)
     (in_bom yes) (on_board yes) (dnp no)
@@
     )
   )
+  (symbol (lib_id "power:GND") (at 236.22 100.33 0) (unit 1)
+    (in_bom yes) (on_board yes) (dnp no)
+    (property "Reference" "#PWR010" (at 236.22 106.68 0)
+      (effects (font (size 1.27 1.27)) hide)
+    )
+    (property "Value" "GND" (at 233.68 103.505 0)
+      (effects (font (size 1.27 1.27)))
+    )
+    (property "Footprint" "" (at 236.22 100.33 0)
+      (effects (font (size 1.27 1.27)) hide)
+    )
+    (property "Datasheet" "" (at 236.22 100.33 0)
+      (effects (font (size 1.27 1.27)) hide)
+    )
+    (pin "1")
+    (instances
+      (project "eurocard"
+        (path "/e048be62-6e5d-4330-8748-f1a6c1c5d89d"
+          (reference "#PWR010") (unit 1)
+        )
+      )
+    )
+  )
   (symbol (lib_id "Device:C") (at 73.66 104.14 90) (unit 1)
     (in_bom yes) (on_board yes) (dnp no)
@@
     )
   )
+  (symbol (lib_id "Connector_Generic_MountingPin:Conn_01x03_MountingPin") (at 236.22 92.71 0) (unit 1)
+    (in_bom yes) (on_board yes) (dnp no)
+    (property "Reference" "J2" (at 234.95 87.63 0)
+      (effects (font (size 1.27 1.27)) (justify left))
+    )
+    (property "Value" "Console" (at 238.506 96.774 90)
+      (effects (font (size 1.27 1.27)) (justify left) hide)
+    )
+    (property "Footprint" "Connector_JST:JST_SH_SM03B-SRSS-TB_1x03-1MP_P1.00mm_Horizontal" (at 236.22 92.71 0)
+      (effects (font (size 1.27 1.27)) hide)
+    )
+    (property "Datasheet" "~" (at 236.22 92.71 0)
+      (effects (font (size 1.27 1.27)) hide)
+    )
+    (pin "1")
+    (pin "3")
+    (pin "MP")
+    (pin "2")
+    (instances
+      (project "eurocard"
+        (path "/e048be62-6e5d-4330-8748-f1a6c1c5d89d"
+          (reference "J2") (unit 1)
+        )
+      )
+    )
+  )
   (symbol (lib_id "Connector:TestPoint") (at 142.24 134.62 270) (unit 1)
     (in_bom yes) (on_board yes) (dnp no)
@@
     )
     (property "Value" "Console" (at 261.366 96.774 90)
-      (effects (font (size 1.27 1.27)) (justify left))
+      (effects (font (size 1.27 1.27)) (justify left) hide)
     )
     (property "Footprint" "Connector_JST:JST_SH_SM03B-SRSS-TB_1x03-1MP_P1.00mm_Horizontal" (at 259.08 92.71 0)
@@
     )
   )
-  (symbol (lib_id "Connector:TestPoint") (at 168.91 91.44 90) (unit 1)
-    (in_bom yes) (on_board yes) (dnp no)
-    (property "Reference" "TP26" (at 164.465 91.44 90)
-      (effects (font (size 1.27 1.27)) (justify left))
-    )
-    (property "Value" "TestPoint" (at 166.8779 88.9 0)
-      (effects (font (size 1.27 1.27)) (justify left) hide)
-    )
-    (property "Footprint" "TestPoint:TestPoint_Pad_1.0x1.0mm" (at 168.91 86.36 0)
-      (effects (font (size 1.27 1.27)) hide)
-    )
-    (property "Datasheet" "~" (at 168.91 86.36 0)
-      (effects (font (size 1.27 1.27)) hide)
-    )
-    (pin "1")
-    (instances
-      (project "eurocard"
-        (path "/e048be62-6e5d-4330-8748-f1a6c1c5d89d"
-          (reference "TP26") (unit 1)
-        )
-      )
-    )
-  )
   (symbol (lib_id "power:GND") (at 259.08 100.33 0) (unit 1)
     (in_bom yes) (on_board yes) (dnp no)
@@
         )
       )
-    )
-  )
-  (symbol (lib_id "Connector:TestPoint") (at 170.18 88.9 90) (unit 1)
-    (in_bom yes) (on_board yes) (dnp no)
-    (property "Reference" "TP25" (at 165.735 88.9 90)
-      (effects (font (size 1.27 1.27)) (justify left))
-    )
-    (property "Value" "TestPoint" (at 168.1479 86.36 0)
-      (effects (font (size 1.27 1.27)) (justify left) hide)
-    )
-    (property "Footprint" "TestPoint:TestPoint_Pad_1.0x1.0mm" (at 170.18 83.82 0)
-      (effects (font (size 1.27 1.27)) hide)
-    )
-    (property "Datasheet" "~" (at 170.18 83.82 0)
-      (effects (font (size 1.27 1.27)) hide)
-    )
-    (pin "1")
-    (instances
-      (project "eurocard"
-        (path "/e048be62-6e5d-4330-8748-f1a6c1c5d89d"
-          (reference "TP25") (unit 1)
-        )
-      )

Commit message: pi-carrier: make room for M.2
- remove J4 HAT connector and mounting holes
- relocate components to make space for M.2
- move heartbeat LED and debug J9 near STM32
- drop GPIO console connection, just use JST connector
- reroute traces
Parts:
- removed J4: Conn_02x20_Odd_Even, 00_eurocard:Rasp_pi_hat_socket, symbol Connector_Generic:Conn_02x20_Odd_Even
- removed R4, R6: 0, Resistor_SMD:R_0603_1608Metric, symbol Device:R
Connections:
- net GPIO10: no longer names the net of J5.19 (MOSI0/GPIO10)
- net GPIO11: no longer names the net of J5.23 (SCLK0/GPIO11)
- net GPIO14: no longer names the net of J5.8 (GPIO14/TXD)
- net GPIO15: no longer names the net of J5.10 (GPIO15/RXD)
- net GPIO17: no longer names the net of J5.11 (GPIO17)
- net GPIO22: no longer names the net of J5.15 (GPIO22)
- net GPIO23: no longer names the net of J5.16 (GPIO23)
- net GPIO24: no longer names the net of J5.18 (GPIO24)
- net GPIO25: no longer names the net of J5.22 (GPIO25)
- net GPIO4: no longer names the net of J5.7 (GCLK0/GPIO4)
- net GPIO7: no longer names the net of J5.26 (~{CE1}/GPIO7)
- net GPIO8: no longer names the net of J5.24 (~{CE0}/GPIO8)
- net GPIO9: no longer names the net of J5.21 (MISO0/GPIO9)
- net ID_SC: no longer names the net of J5.28 (ID_SC/GPIO1)
- net ID_SD: no longer names the net of J5.27 (ID_SD/GPIO0)
- no-connect marks 52 -> 67
Other:
- note added: "Raspberry pi"
- note removed: "DNP"
- note removed: "Raspberry pi and HAT header"
- moved on the sheet: J2, J3

Commit message: pi-carrier: drop excessive testpoints
Problem: the test points have not been all that useful and
complicate routing.

Drop them, except the ones that are connected to unused
STM32 GPIO lines, which are useful.

Update board.
Parts:
- removed TP1, TP10, TP12, TP13, TP14, TP15, TP16, TP17, TP2, TP3, TP4, TP5, TP6, TP7, TP8, TP9: TestPoint, TestPoint:TestPoint_Pad_1.0x1.0mm, symbol Connector:TestPoint

Commit message: pi-carrier: reroute BUS5V_2
Problem: The matrix 5V supply is unnecessarily routed to BUS5V_1.

Have it use BUS5V_2 which is closer (but unfused currently).
Connections:
- net +5V: no longer C11.2, C5.1, C7.1, R11.1, U8.14 (VCC), U9.19 (V+)
- net BUS5V_2: now also C11.2, C5.1, C7.1, R11.1, U8.14 (VCC), U9.19 (V+)
Other:
- moved on the sheet: C11, C5

Commit message: pi-carrier: add M.2 interface to schematic
Problem: it would be nice to have an M.2 slot on the pi-carrier
so a compute node could have local nvme storage.

Add a new schematic page for an M.2 connector.

References:

Pi 5 PCIe FFC pinout:
  https://datasheets.raspberrypi.com/pcie/pcie-connector-standard.pdf

3V3 3A power supply and M.2 design hints:
  https://github.com/will127534/CM4-Nvme-NAS

TPS563202 4.3V to 17V input, 3A synchronous buck converter in SOT563
  https://www.ti.com/lit/ds/symlink/tps563202.pdf

KiCad 5 no 17 hierarchical labels & pins - John's Basement
  https://youtu.be/m_HTBurAJn4?si=loStiD6Dr1jY2ZZ0
Other:
- added sheet M.2 Storage (m2.kicad_sch)
Changed lines of the file:
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@@
     (stroke (width 0) (type default))
   )
+  (wire (pts (xy 232.41 148.59) (xy 242.57 148.59))
+    (stroke (width 0) (type default))
+  )
   (polyline (pts (xy 262.89 80.01) (xy 262.89 85.09))
     (stroke (width 0) (type default))
@@
     (effects (font (size 1.27 1.27)) (justify right bottom))
   )
+  (label "BUS5V_2" (at 232.41 148.59 0) (fields_autoplaced)
+    (effects (font (size 1.27 1.27)) (justify left bottom))
+  )
   (label "GA1" (at 55.88 134.62 180) (fields_autoplaced)
     (effects (font (size 1.27 1.27)) (justify right bottom))
@@
       )
     )
+  )
+  (sheet (at 242.57 144.78) (size 12.7 13.97) (fields_autoplaced)
+    (stroke (width 0.1524) (type solid))
+    (fill (color 0 0 0 0.0000))
+    (property "Sheetname" "M.2 Storage" (at 242.57 144.0684 0)
+      (effects (font (size 1.27 1.27)) (justify left bottom))
+    )
+    (property "Sheetfile" "m2.kicad_sch" (at 242.57 159.3346 0)
+      (effects (font (size 1.27 1.27)) (justify left top))
+    )
+    (pin "PCIE_5V" input (at 242.57 148.59 180)
+      (effects (font (size 1.27 1.27)) (justify left))
+    )
+    (instances
+      (project "eurocard"
+        (path "/e048be62-6e5d-4330-8748-f1a6c1c5d89d" (page "2"))
+      )
+    )

Commit message: pi-carrier: use vertical JST connectors
Problem: horizontal JST connectors are inappropriate for the
design now that less board space is available.

Switch to vertical JST connectors.
Add 3d model.
Parts:
- J2, J3: footprint Connector_JST:JST_SH_SM03B-SRSS-TB_1x03-1MP_P1.00mm_Horizontal -> Connector_JST:JST_SH_BM03B-SRSS-TB_1x03-1MP_P1.00mm_Vertical
Changed lines of the file:
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@@
       (effects (font (size 1.27 1.27)) (justify left) hide)
     )
-    (property "Footprint" "Connector_JST:JST_SH_SM03B-SRSS-TB_1x03-1MP_P1.00mm_Horizontal" (at 255.27 116.84 0)
+    (property "Footprint" "Connector_JST:JST_SH_BM03B-SRSS-TB_1x03-1MP_P1.00mm_Vertical" (at 255.27 116.84 0)
       (effects (font (size 1.27 1.27)) hide)
     )
@@
       (effects (font (size 1.27 1.27)) (justify left) hide)
     )
-    (property "Footprint" "Connector_JST:JST_SH_SM03B-SRSS-TB_1x03-1MP_P1.00mm_Horizontal" (at 255.27 95.25 0)
+    (property "Footprint" "Connector_JST:JST_SH_BM03B-SRSS-TB_1x03-1MP_P1.00mm_Vertical" (at 255.27 95.25 0)
       (effects (font (size 1.27 1.27)) hide)
     )

Commit message: pi-carrier: relocate battery, add connectors
Problem: there is no room for an efuse near power entry.

Move the coin battery holder to the other side of the M.2 power
suply and instead of routing, use a JST SH connector that would
allow it to be used either for the STM32 or for a Pi 5 RTC.
Parts:
- added J6, J8: Conn_01x02_MountingPin, Connector_JST:JST_SH_BM02B-SRSS-TB_1x02-1MP_P1.00mm_Vertical, symbol Connector_Generic_MountingPin:Conn_01x02_MountingPin
Connections:
- net GND: now also J6.1 (Pin_1), J6.MP (MountPin), J8.MP (MountPin); no longer BT1.2 (-)
- net at BT1.1 (+): now also J8.2 (Pin_2); no longer D1.1
- new net: BT1.2 (-), J8.1 (Pin_1)
- new net: D1.1, J6.2 (Pin_2)
Other:
- note removed: "STM32 real time clock power"
- moved on the sheet: BT1, C20, D1
