File: hardware/pi-carrier/m2.kicad_sch (KiCad schematic)
At the start: 18 parts, among them J4 Bus_M.2_Socket_M, J7 Conn_01x16_MountingPin, U7 TPS563202S

Commit message: pi-carrier: select inductor footprint
Problem: M.2 switching power supply inductor has no footprint.

The TPS563202 data sheet uses a WE 74437349012 part for the reference
design.  Wrong value for our design but that part has a 7.30 x 6.60
footprint, Z=5mm.  Go with the nearest stock footprint found in the
KiCad library.
Parts:
- L1: footprint (none) -> Inductor_SMD:L_7.3x7.3_H4.5
Changed lines of the file:
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@@
       (effects (font (size 1.27 1.27)))
     )
-    (property "Footprint" "" (at 114.3 135.89 0)
+    (property "Footprint" "Inductor_SMD:L_7.3x7.3_H4.5" (at 114.3 135.89 0)
       (effects (font (size 1.27 1.27)) hide)
     )

Commit message: pi-carrier: add M.2 2280 outline and mounting
Problem: the M.2 connector must be aligned with the mounting
hole and silk board outline.

Add it to the footprint.
Connections:
- net GND: now also J4.MP (GND)
Changed lines of the file:
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@@
   (junction (at 58.42 59.69) (diameter 0) (color 0 0 0 0)
+  )
+  (junction (at 217.17 132.08) (diameter 0) (color 0 0 0 0)
   )
   (junction (at 50.8 82.55) (diameter 0) (color 0 0 0 0)
@@
     (stroke (width 0) (type default))
   )
-  (wire (pts (xy 217.17 130.81) (xy 217.17 133.35))
+  (wire (pts (xy 217.17 130.81) (xy 217.17 132.08))
     (stroke (width 0) (type default))
   )
@@
     (stroke (width 0) (type default))
   )
+  (wire (pts (xy 217.17 132.08) (xy 217.17 133.35))
+    (stroke (width 0) (type default))
+  )
   (wire (pts (xy 217.17 26.67) (xy 217.17 34.29))
     (stroke (width 0) (type default))
@@
     (stroke (width 0) (type default))
   )
+  (wire (pts (xy 217.17 132.08) (xy 226.06 132.08))
+    (stroke (width 0) (type default))
+  )
   (wire (pts (xy 55.88 49.53) (xy 74.93 49.53))
     (stroke (width 0) (type default))
@@
   (label "PCIE_PWR_EN" (at 49.53 140.97 0) (fields_autoplaced)
     (effects (font (size 1.27 1.27)) (justify left bottom))
+  )
+  (label "MP" (at 226.06 132.08 180) (fields_autoplaced)
+    (effects (font (size 1.27 1.27)) (justify right bottom))
   )
   (label "PCIE_CLK_N" (at 173.99 120.65 0) (fields_autoplaced)
@@
     (pin "40")
     (pin "30")
+    (pin "MP")
     (instances
       (project "eurocard"

Commit message: pi-carrier: add M.2 storage
Drop unnecessary DNP 0R resistor in PCIE_DET_WAKE.
Nudge battery towards the DIN connector to make more room.
Place the M.2 outline.
Place activity LED.
Adjust FFC to center of pi card edge.
Route M.2 non-differential signals.
Parts:
- removed R9: 0, Resistor_SMD:R_0603_1608Metric, symbol Device:R
- J4: footprint (none) -> 00_eurocard:Conn_TE-M.2-0.5-67P-doublesided_TypeM
- J7: footprint (none) -> 00_eurocard:FPC16
Connections:
- net ~{PEWAKE} is gone; now on net PCIE_DET_WAKE: J4.54 (~{PEWAKE})
- net PI_5V: now also J7.2 (Pin_2)
- no-connect marks 16 -> 15
Other:
- note removed: "DNP"
- moved on the sheet: C21, C22, R4

Commit message: pi-carrier: update M.2 power circuit
Problem: oops, TI buck converter is obsolete.

Use the pin-compatible replacement, TPS563203.
Adjust recommended component values for 3V3 and add some
more passives per the new spec sheet.
Parts:
- added C26: 10pF, Capacitor_SMD:C_0603_1608Metric, symbol Device:C
- added C27: 100nF, Capacitor_SMD:C_0603_1608Metric, symbol Device:C
- L1: value 3.3uH -> 4.7uH
- R2: value 1.69K -> 135K
- R3: value 1.69K -> 30K
- U7: value TPS563202S -> TPS563203
Connections:
- net GND: now also C27.2
- net M2_3V3: now also C26.2
- net PCIE_5V: now also C27.1
- net at R2.2, R3.1, U7.6 (FB): now also C26.1
Other:
- moved on the sheet: C21, C22, C24, C25, TP23

Commit message: pi-carrier: change FPC footprint to a real product
Problem: FPC footprint doesn't seem to match real connectors.

Use this one:

https://www.digikey.com/en/products/detail/amphenol-cs-fci/F31W-1A7H1-11016/11564570
https://cdn.amphenol-cs.com/media/wysiwyg/files/drawing/f31z-f31w.pdf

Include 3d model.
Parts:
- J7: footprint 00_eurocard:FPC16 -> 00_eurocard:CONN_F31W-1A7H1-11016_AMP
Changed lines of the file:
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@@
       (effects (font (size 1.27 1.27)) (justify left))
     )
-    (property "Footprint" "00_eurocard:FPC16" (at 50.8 57.15 0)
+    (property "Footprint" "00_eurocard:CONN_F31W-1A7H1-11016_AMP" (at 50.8 57.15 0)
       (effects (font (size 1.27 1.27)) hide)
     )

Commit message: pi-carrier: lay out M.2 power supply again
Problem: the M.2 power supply layout sucks.

Do it again.
Parts:
- removed TP23: TestPoint, TestPoint:TestPoint_Pad_1.0x1.0mm, symbol Connector:TestPoint
- added JP1, JP2: SolderJumper_2_Bridged, Jumper:SolderJumper-2_P1.3mm_Bridged_RoundedPad1.0x1.5mm, symbol Jumper:SolderJumper_2_Bridged
- added TP1: TestPoint, TestPoint:TestPoint_Pad_1.0x1.0mm, symbol Connector:TestPoint
Connections:
- net M2_3V3: now also JP2.2 (B); no longer C24.1, C25.1, C26.2, L1.2, R2.1
- net PCIE_5V: now also JP1.1 (A); no longer C21.1, C22.1, C27.1, U7.1 (VIN)
- net PCIE_PWR_EN: now also TP1.1
- new net: C24.1, C25.1, C26.2, JP2.1 (A), L1.2, R2.1
- new net: C21.1, C22.1, C27.1, JP1.2 (B), U7.1 (VIN)
Other:
- moved on the sheet: C21, C22, C23, C24, C25, C26, C27, D4, L1, R2, R3, R4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

Commit message: pi-carrier: more re-routing
- reroute diff clock signal around connector
- move pull-down to M.2 power supply block
- reroute M.2 3V3 rail
Connections:
- net PCIE_DET_WAKE: no longer J4.54 (~{PEWAKE})
- no-connect marks 15 -> 16
Changed lines of the file:
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@@
   (junction (at 58.42 39.37) (diameter 0) (color 0 0 0 0)
   )
+  (junction (at 41.91 144.78) (diameter 0) (color 0 0 0 0)
+  )
   (junction (at 124.46 144.78) (diameter 0) (color 0 0 0 0)
   )
@@
   (junction (at 148.59 144.78) (diameter 0) (color 0 0 0 0)
   )
+  (junction (at 190.5 144.78) (diameter 0) (color 0 0 0 0)
+  )
   (junction (at 135.89 144.78) (diameter 0) (color 0 0 0 0)
   )
@@
   )
   (junction (at 69.85 144.78) (diameter 0) (color 0 0 0 0)
+  )
+  (junction (at 63.5 39.37) (diameter 0) (color 0 0 0 0)
   )
   (no_connect (at 191.77 74.93))
@@
   (no_connect (at 191.77 72.39))
   (no_connect (at 191.77 62.23))
+  (no_connect (at 191.77 44.45))
   (no_connect (at 191.77 80.01))
   (no_connect (at 191.77 87.63))
@@
     (stroke (width 0) (type default))
   )
-  (wire (pts (xy 39.37 144.78) (xy 46.99 144.78))
-    (stroke (width 0) (type default))
-  )
-  (wire (pts (xy 58.42 39.37) (xy 74.93 39.37))
+  (wire (pts (xy 39.37 144.78) (xy 41.91 144.78))
+    (stroke (width 0) (type default))
+  )
+  (wire (pts (xy 58.42 39.37) (xy 63.5 39.37))
     (stroke (width 0) (type default))
   )
@@
     (stroke (width 0) (type default))
   )
-  (wire (pts (xy 185.42 144.78) (xy 194.31 144.78))
+  (wire (pts (xy 190.5 144.78) (xy 201.93 144.78))
     (stroke (width 0) (type default))
   )
@@
     (stroke (width 0) (type default))
   )
+  (wire (pts (xy 63.5 39.37) (xy 74.93 39.37))
+    (stroke (width 0) (type default))
+  )
   (wire (pts (xy 173.99 57.15) (xy 191.77 57.15))
     (stroke (width 0) (type default))
@@
     (stroke (width 0) (type default))
   )
+  (wire (pts (xy 190.5 144.78) (xy 185.42 144.78))
+    (stroke (width 0) (type default))
+  )
   (wire (pts (xy 55.88 49.53) (xy 74.93 49.53))
     (stroke (width 0) (type default))
@@
     (stroke (width 0) (type default))
   )
-  (wire (pts (xy 173.99 44.45) (xy 191.77 44.45))
-    (stroke (width 0) (type default))
-  )
   (wire (pts (xy 101.6 59.69) (xy 119.38 59.69))
     (stroke (width 0) (type default))
@@
     (stroke (width 0) (type default))
   )
+  (wire (pts (xy 41.91 144.78) (xy 46.99 144.78))
+    (stroke (width 0) (type default))
+  )
   (wire (pts (xy 69.85 152.4) (xy 69.85 153.67))
     (stroke (width 0) (type default))
@@
     (effects (font (size 1.27 1.27)) (justify left bottom))
   )
-  (label "M2_3V3" (at 194.31 144.78 180) (fields_autoplaced)
+  (label "M2_3V3" (at 201.93 144.78 180) (fields_autoplaced)
     (effects (font (size 1.27 1.27)) (justify right bottom))
   )
@@
   )
   (label "PCIE_TX_P" (at 173.99 52.07 0) (fields_autoplaced)
-    (effects (font (size 1.27 1.27)) (justify left bottom))
-  )
-  (label "PCIE_DET_WAKE" (at 173.99 44.45 0) (fields_autoplaced)
     (effects (font (size 1.27 1.27)) (justify left bottom))
   )
@@
     )
   )
+  (symbol (lib_id "power:PWR_FLAG") (at 41.91 144.78 0) (unit 1)
+    (in_bom yes) (on_board yes) (dnp no) (fields_autoplaced)
+    (property "Reference" "#FLG05" (at 41.91 142.875 0)
+      (effects (font (size 1.27 1.27)) hide)
+    )
+    (property "Value" "PWR_FLAG" (at 41.91 139.7 0)
+      (effects (font (size 1.27 1.27)))
+    )
+    (property "Footprint" "" (at 41.91 144.78 0)
+      (effects (font (size 1.27 1.27)) hide)
+    )
+    (property "Datasheet" "~" (at 41.91 144.78 0)
+      (effects (font (size 1.27 1.27)) hide)
+    )
+    (pin "1")
+    (instances
+      (project "eurocard"
+        (path "/e048be62-6e5d-4330-8748-f1a6c1c5d89d/78247a58-bd33-4427-a596-05636cd08db2"
+          (reference "#FLG05") (unit 1)
+        )
+      )
+    )
+  )
   (symbol (lib_id "power:GND") (at 69.85 153.67 0) (unit 1)
     (in_bom yes) (on_board yes) (dnp no) (fields_autoplaced)
@@
     )
   )
+  (symbol (lib_id "power:PWR_FLAG") (at 63.5 39.37 0) (unit 1)
+    (in_bom yes) (on_board yes) (dnp no) (fields_autoplaced)
+    (property "Reference" "#FLG04" (at 63.5 37.465 0)
+      (effects (font (size 1.27 1.27)) hide)
+    )
+    (property "Value" "PWR_FLAG" (at 63.5 34.29 0)
+      (effects (font (size 1.27 1.27)))
+    )
+    (property "Footprint" "" (at 63.5 39.37 0)
+      (effects (font (size 1.27 1.27)) hide)
+    )
+    (property "Datasheet" "~" (at 63.5 39.37 0)
+      (effects (font (size 1.27 1.27)) hide)
+    )
+    (pin "1")
+    (instances
+      (project "eurocard"
+        (path "/e048be62-6e5d-4330-8748-f1a6c1c5d89d/78247a58-bd33-4427-a596-05636cd08db2"
+          (reference "#FLG04") (unit 1)
+        )
+      )
+    )
+  )
   (symbol (lib_id "Device:R") (at 135.89 161.29 0) (unit 1)
     (in_bom yes) (on_board yes) (dnp no) (fields_autoplaced)
@@
         )
       )
+    )
+  )
+  (symbol (lib_id "power:PWR_FLAG") (at 190.5 144.78 0) (unit 1)
+    (in_bom yes) (on_board yes) (dnp no)
+    (property "Reference" "#FLG06" (at 190.5 142.875 0)
+      (effects (font (size 1.27 1.27)) hide)
+    )
+    (property "Value" "PWR_FLAG" (at 190.5 139.7 0)
+      (effects (font (size 1.27 1.27)))
+    )
+    (property "Footprint" "" (at 190.5 144.78 0)
+      (effects (font (size 1.27 1.27)) hide)
+    )
+    (property "Datasheet" "~" (at 190.5 144.78 0)
+      (effects (font (size 1.27 1.27)) hide)
+    )
+    (pin "1")
+    (instances
+      (project "eurocard"
+        (path "/e048be62-6e5d-4330-8748-f1a6c1c5d89d/78247a58-bd33-4427-a596-05636cd08db2"
+          (reference "#FLG06") (unit 1)
+        )
+      )

Commit message: pi-carrier: add jumper to M.2 power enable
Problem: the M.2 power block is connected directly to the enable
line on the FFC.

Add a jumper so the whole block can be cut out if necessary.
Drop test point since the jumper can act as one.
Parts:
- removed TP1: TestPoint, TestPoint:TestPoint_Pad_1.0x1.0mm, symbol Connector:TestPoint
- added JP3: SolderJumper_2_Bridged, Jumper:SolderJumper-2_P1.3mm_Bridged_RoundedPad1.0x1.5mm, symbol Jumper:SolderJumper_2_Bridged
Connections:
- net PCIE_PWR_EN: now also JP3.1 (A); no longer R4.1, U7.5 (EN)
- new net: JP3.2 (B), R4.1, U7.5 (EN)
Changed lines of the file:
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@@
 (kicad_sch (version 20230121) (generator eeschema)
   (paper "USLetter")
-  (junction (at 57.15 163.83) (diameter 0) (color 0 0 0 0)
-  )
   (junction (at 135.89 156.21) (diameter 0) (color 0 0 0 0)
   )
@@
     (stroke (width 0) (type default))
   )
-  (wire (pts (xy 57.15 163.83) (xy 80.01 163.83))
+  (wire (pts (xy 67.945 164.465) (xy 80.01 164.465))
     (stroke (width 0) (type default))
   )
@@
     (stroke (width 0) (type default))
   )
-  (wire (pts (xy 41.91 163.83) (xy 57.15 163.83))
-    (stroke (width 0) (type default))
-  )
   (wire (pts (xy 119.38 59.69) (xy 119.38 60.96))
     (stroke (width 0) (type default))
@@
     (stroke (width 0) (type default))
   )
-  (wire (pts (xy 80.01 163.83) (xy 80.01 149.86))
+  (wire (pts (xy 80.01 164.465) (xy 80.01 149.86))
     (stroke (width 0) (type default))
   )
@@
     (stroke (width 0) (type default))
   )
+  (wire (pts (xy 39.37 164.465) (xy 60.325 164.465))
+    (stroke (width 0) (type default))
+  )
   (wire (pts (xy 114.3 151.13) (xy 114.3 147.32))
     (stroke (width 0) (type default))
@@
     (effects (font (size 1.27 1.27)) (justify right bottom))
   )
-  (label "PCIE_PWR_EN" (at 41.91 163.83 0) (fields_autoplaced)
+  (label "PCIE_PWR_EN" (at 39.37 164.465 0) (fields_autoplaced)
     (effects (font (size 1.27 1.27)) (justify left bottom))
   )
@@
   (hierarchical_label "PCIE_5V" (shape input) (at 31.75 144.78 180) (fields_autoplaced)
     (effects (font (size 1.27 1.27)) (justify right))
-  )
-  (symbol (lib_id "Connector:TestPoint") (at 57.15 163.83 180) (unit 1)
-    (in_bom yes) (on_board yes) (dnp no) (fields_autoplaced)
-    (property "Reference" "TP1" (at 59.69 165.862 0)
-      (effects (font (size 1.27 1.27)) (justify right))
-    )
-    (property "Value" "TestPoint" (at 59.69 168.402 0)
-      (effects (font (size 1.27 1.27)) (justify right))
-    )
-    (property "Footprint" "TestPoint:TestPoint_Pad_1.0x1.0mm" (at 52.07 163.83 0)
-      (effects (font (size 1.27 1.27)) hide)
-    )
-    (property "Datasheet" "~" (at 52.07 163.83 0)
-      (effects (font (size 1.27 1.27)) hide)
-    )
-    (pin "1")
-    (instances
-      (project "eurocard"
-        (path "/e048be62-6e5d-4330-8748-f1a6c1c5d89d/78247a58-bd33-4427-a596-05636cd08db2"
-          (reference "TP1") (unit 1)
-        )
-      )
-    )
   )
   (symbol (lib_id "Device:R") (at 135.89 151.13 0) (unit 1)
@@
         )
       )
+    )
+  )
+  (symbol (lib_id "Jumper:SolderJumper_2_Bridged") (at 64.135 164.465 0) (unit 1)
+    (in_bom yes) (on_board yes) (dnp no) (fields_autoplaced)
+    (property "Reference" "JP3" (at 64.135 160.655 0)
+      (effects (font (size 1.27 1.27)))
+    )
+    (property "Value" "SolderJumper_2_Bridged" (at 64.135 160.655 0)
+      (effects (font (size 1.27 1.27)) hide)
+    )
+    (property "Footprint" "Jumper:SolderJumper-2_P1.3mm_Bridged_RoundedPad1.0x1.5mm" (at 64.135 164.465 0)
+      (effects (font (size 1.27 1.27)) hide)
+    )
+    (property "Datasheet" "~" (at 64.135 164.465 0)
+      (effects (font (size 1.27 1.27)) hide)
+    )
+    (pin "2")
+    (pin "1")
+    (instances
+      (project "eurocard"
+        (path "/e048be62-6e5d-4330-8748-f1a6c1c5d89d/78247a58-bd33-4427-a596-05636cd08db2"
+          (reference "JP3") (unit 1)
+        )
+      )
