File: hardware/pi-carrier/m2.kicad_sch (KiCad schematic)
At the start: 21 parts, among them J4 Bus_M.2_Socket_M, J7 Conn_01x16_MountingPin, U7 TPS563203

Commit message: pi-carrier: clean up schematic
Problem: the schematic is still too busy for one page and lacks
room to expand.

Move matrix display and OR network to a hierarchical page.
Tidy up the main schematic.
Changed lines of the file:
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@@
   (junction (at 58.42 59.69) (diameter 0) (color 0 0 0 0)
-  )
-  (junction (at 217.17 132.08) (diameter 0) (color 0 0 0 0)
   )
   (junction (at 50.8 82.55) (diameter 0) (color 0 0 0 0)
@@
     (stroke (width 0) (type default))
   )
-  (wire (pts (xy 217.17 130.81) (xy 217.17 132.08))
+  (wire (pts (xy 217.17 130.81) (xy 217.17 133.35))
     (stroke (width 0) (type default))
   )
@@
     (stroke (width 0) (type default))
   )
-  (wire (pts (xy 217.17 132.08) (xy 217.17 133.35))
-    (stroke (width 0) (type default))
-  )
   (wire (pts (xy 217.17 26.67) (xy 217.17 34.29))
     (stroke (width 0) (type default))
@@
     (stroke (width 0) (type default))
   )
-  (wire (pts (xy 217.17 132.08) (xy 226.06 132.08))
-    (stroke (width 0) (type default))
-  )
   (wire (pts (xy 190.5 144.78) (xy 185.42 144.78))
     (stroke (width 0) (type default))
@@
     (effects (font (size 1.27 1.27)) (justify left bottom))
   )
-  (label "MP" (at 226.06 132.08 180) (fields_autoplaced)
-    (effects (font (size 1.27 1.27)) (justify right bottom))
-  )
   (label "PCIE_CLK_N" (at 173.99 120.65 0) (fields_autoplaced)

Commit message: pi-carrier: adjust pcie diff-pair skew, Z
Problem: pcie pairs are just using the netclass parameters
and have skewed lengths.

Adjust trace width and distance to minimize Zdiff given the
limitations of a 2-layer board, although it is still out of
tolerance.  Add notes to schematic from pcbway's impedance
calculator.

Address intra-pair skew with squiggles close to the end that
introduced the skew, and stitch vias per TI differential pair
routing guide.
Other:
- note added: "Differential routing notes: Goal: 90R +/-10% differential impedance[1] Track height 1oz Cu[2]: 0.0348mm Isolation height for 1.6mm 2 layer board: 1.53mm Dialectric constant FR4[3]: 4.3 Trace Width Trace Spacing Zdiff[3] 0.2mm 0.25mm 163R (default netclass) 0.2mm 0.154mm (6mil) 142R 0.3mm 0.154mm 127R 0.27mm 0.165mm 133R (meets 6mil fab limit + FFC footprint clearances) [1] https://datasheets.rasp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"
Changed lines of the file:
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@@
     (stroke (width 0) (type default))
+  )
+  (text "Differential routing notes:\n\nGoal: 90R +/-10% differential impedance[1]\n\nTrack height 1oz Cu[2]: 0.0348mm\nIsolation height for 1.6mm 2 layer board: 1.53mm\nDialectric constant FR4[3]: 4.3\n\nTrace Width    Trace Spacing     Zdiff[3]\n0.2mm          0.25mm            163R (default netclass)\n0.2mm          0.154mm (6mil)    142R\n0.3mm          0.154mm           127R\n0.27mm         0.165mm           133R (meets 6mil fab limit + FFC footprint clearances)\n\n[1] https://datasheets.raspberrypi.com/pcie/pcie-connector-standard.pdf\n[2] https://pcbprime.com/pcb-tips/how-thick-is-1oz-copper/\n[3] https://www.pcbway.com/pcb_prototype/impedance_calculator.html"
+    (at 15.24 201.93 0)
+    (effects (font (size 1.27 1.27)) (justify left bottom))
   )
   (label "PCIE_TX_N" (at 74.93 64.77 180) (fields_autoplaced)

Commit message: pi-carrier: add enable LED to M.2 power
Problem: it would be nice to know when the pi has enabled
the M.2 power supply.

Add an LED to the power supply block.
Parts:
- added D7: LED, LED_SMD:LED_0805_2012Metric_Pad1.15x1.40mm_HandSolder, symbol Device:LED
- added R18: 220, Resistor_SMD:R_0603_1608Metric, symbol Device:R
Connections:
- net GND: now also D7.1 (K)
- net PCIE_PWR_EN: now also R18.2
- new net: D7.2 (A), R18.1
Changed lines of the file:
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@@
+    (stroke (width 0) (type default))
+  )
+  (wire (pts (xy 102.87 111.76) (xy 102.87 106.68))
     (stroke (width 0) (type default))
   )
@@
     (stroke (width 0) (type default))
   )
+  (wire (pts (xy 116.84 106.68) (xy 119.38 106.68))
+    (stroke (width 0) (type default))
+  )
   (wire (pts (xy 173.99 54.61) (xy 191.77 54.61))
     (stroke (width 0) (type default))
@@
     (stroke (width 0) (type default))
   )
+  (wire (pts (xy 127 106.68) (xy 142.24 106.68))
+    (stroke (width 0) (type default))
+  )
   (wire (pts (xy 58.42 82.55) (xy 50.8 82.55))
     (stroke (width 0) (type default))
@@
     (stroke (width 0) (type default))
   )
-  (wire (pts (xy 127 95.25) (xy 138.43 95.25))
+  (wire (pts (xy 127 95.25) (xy 142.24 95.25))
     (stroke (width 0) (type default))
   )
@@
   )
   (wire (pts (xy 55.88 46.99) (xy 74.93 46.99))
+    (stroke (width 0) (type default))
+  )
+  (wire (pts (xy 102.87 106.68) (xy 109.22 106.68))
     (stroke (width 0) (type default))
   )
@@
     (effects (font (size 1.27 1.27)) (justify right bottom))
   )
-  (label "M2_3V3" (at 138.43 95.25 180) (fields_autoplaced)
+  (label "M2_3V3" (at 142.24 95.25 180) (fields_autoplaced)
     (effects (font (size 1.27 1.27)) (justify right bottom))
   )
@@
   (label "PCIE_DET_WAKE" (at 101.6 59.69 0) (fields_autoplaced)
     (effects (font (size 1.27 1.27)) (justify left bottom))
+  )
+  (label "PCIE_PWR_EN" (at 142.24 106.68 180) (fields_autoplaced)
+    (effects (font (size 1.27 1.27)) (justify right bottom))
   )
   (label "PCIE_RX_P" (at 173.99 57.15 0) (fields_autoplaced)
@@
     )
   )
+  (symbol (lib_id "Device:R") (at 123.19 106.68 90) (unit 1)
+    (in_bom yes) (on_board yes) (dnp no) (fields_autoplaced)
+    (property "Reference" "R18" (at 123.19 100.33 90)
+      (effects (font (size 1.27 1.27)))
+    )
+    (property "Value" "220" (at 123.19 102.87 90)
+      (effects (font (size 1.27 1.27)))
+    )
+    (property "Footprint" "Resistor_SMD:R_0603_1608Metric" (at 123.19 108.458 90)
+      (effects (font (size 1.27 1.27)) hide)
+    )
+    (property "Datasheet" "~" (at 123.19 106.68 0)
+      (effects (font (size 1.27 1.27)) hide)
+    )
+    (pin "1")
+    (pin "2")
+    (instances
+      (project "eurocard"
+        (path "/e048be62-6e5d-4330-8748-f1a6c1c5d89d/78247a58-bd33-4427-a596-05636cd08db2"
+          (reference "R18") (unit 1)
+        )
+      )
+    )
+  )
   (symbol (lib_id "Device:C") (at 148.59 151.13 180) (unit 1)
     (in_bom yes) (on_board yes) (dnp no)
@@
     )
   )
+  (symbol (lib_id "Device:LED") (at 113.03 106.68 0) (unit 1)
+    (in_bom yes) (on_board yes) (dnp no)
+    (property "Reference" "D7" (at 111.4425 100.33 0)
+      (effects (font (size 1.27 1.27)))
+    )
+    (property "Value" "LED" (at 111.4425 102.87 0)
+      (effects (font (size 1.27 1.27)))
+    )
+    (property "Footprint" "LED_SMD:LED_0805_2012Metric_Pad1.15x1.40mm_HandSolder" (at 113.03 106.68 0)
+      (effects (font (size 1.27 1.27)) hide)
+    )
+    (property "Datasheet" "~" (at 113.03 106.68 0)
+      (effects (font (size 1.27 1.27)) hide)
+    )
+    (pin "2")
+    (pin "1")
+    (instances
+      (project "eurocard"
+        (path "/e048be62-6e5d-4330-8748-f1a6c1c5d89d/78247a58-bd33-4427-a596-05636cd08db2"
+          (reference "D7") (unit 1)
+        )
+      )
+    )
+  )
   (symbol (lib_id "power:PWR_FLAG") (at 190.5 144.78 0) (unit 1)
     (in_bom yes) (on_board yes) (dnp no)
@@
         )
       )
+    )
+  )
+  (symbol (lib_id "power:GND") (at 102.87 111.76 0) (unit 1)
+    (in_bom yes) (on_board yes) (dnp no) (fields_autoplaced)
+    (property "Reference" "#PWR051" (at 102.87 118.11 0)
+      (effects (font (size 1.27 1.27)) hide)
+    )
+    (property "Value" "GND" (at 102.87 116.84 0)
+      (effects (font (size 1.27 1.27)))
+    )
+    (property "Footprint" "" (at 102.87 111.76 0)
+      (effects (font (size 1.27 1.27)) hide)
+    )
+    (property "Datasheet" "" (at 102.87 111.76 0)
+      (effects (font (size 1.27 1.27)) hide)
+    )
+    (pin "1")
+    (instances
+      (project "eurocard"
+        (path "/e048be62-6e5d-4330-8748-f1a6c1c5d89d/78247a58-bd33-4427-a596-05636cd08db2"
+          (reference "#PWR051") (unit 1)
+        )
+      )

Commit message: pi-carrier: drive EN LED from within block
Problem the EN LED is connected "outside" the jumper
but it is really part of the power supply block.

Connect it to the other end of the jumper.
Connections:
- net PCIE_PWR_EN: no longer R18.2
- net at JP3.2 (B), R4.1, U7.5 (EN): now also R18.2
Other:
- moved on the sheet: C21, C22, C23, C24, C25, C26, C27, D7, JP1, JP2, JP3, L1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

Commit message: pi-carrier: re-reoute pcie diff pairs
Problem: PCIe diff pair impedance is not correct.

Use keepouts to avoid co-planar ground pour next to diff pairs.

Recalculate for 90R non-coplanar diff pair using JLCPCB calculator:
W = 6.23 mil (0.1583mm), S = 8 mil (0.2032mm).
Update board netclass DP values.
Note values in schematic.

Set project min W and S, which was causing the wrong paramters to be
used before.  Go with 6 mil (0.1524mm) for both.

Re-route diff pairs.

NOTE: the EEWeb calculator for coupled microstrips[1] does not agree:

T = 1.38 mil (L1 thickness in JLC04161H-3313 stackup)
W = 6.23 mil
H = 3.91 mil (prepreg thickness in JLC04161H-3313 stackup)
S = 8 mil
subtrate dielectric = 4.1 (JLCPCB 3313 material)
Calculated differential impedance: 118.2R

[1] https://www.eeweb.com/tools/edge-coupled-microstrip-impedance/
Other:
- note added: "Differential routing notes: Goal: 90R +/-10% differential impedance[1] Stackup: JLC04161H-3313 (low cost from JLCPCB) JLCPCB calculator (non-coplanar diff pair): width: 6.2300 mils (0.1583 mm) spacing: 8 mils (0.2032 mm)"
- note removed: "Differential routing notes: Goal: 90R +/-10% differential impedance[1] Track height 1oz Cu[2]: 0.0348mm Isolation height for 1.6mm 2 layer board: 1.53mm Dialectric constant FR4[3]: 4.3 Trace Width Trace Spacing Zdiff[3] 0.2mm 0.25mm 163R (default netclass) 0.2mm 0.154mm (6mil) 142R 0.3mm 0.154mm 127R 0.27mm 0.165mm 133R (meets 6mil fab limit + FFC footprint clearances) [1] https://datasheets.rasp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"
Changed lines of the file:
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@@
     (stroke (width 0) (type default))
   )
-  (text "Differential routing notes:\n\nGoal: 90R +/-10% differential impedance[1]\n\nTrack height 1oz Cu[2]: 0.0348mm\nIsolation height for 1.6mm 2 layer board: 1.53mm\nDialectric constant FR4[3]: 4.3\n\nTrace Width    Trace Spacing     Zdiff[3]\n0.2mm          0.25mm            163R (default netclass)\n0.2mm          0.154mm (6mil)    142R\n0.3mm          0.154mm           127R\n0.27mm         0.165mm           133R (meets 6mil fab limit + FFC footprint clearances)\n\n[1] https://datasheets.raspberrypi.com/pcie/pcie-connector-standard.pdf\n[2] https://pcbprime.com/pcb-tips/how-thick-is-1oz-copper/\n[3] https://www.pcbway.com/pcb_prototype/impedance_calculator.html"
+  (text "Differential routing notes:\n\nGoal: 90R +/-10% differential impedance[1]\n\nStackup: JLC04161H-3313 (low cost from JLCPCB)\n\nJLCPCB calculator (non-coplanar diff pair):\nwidth: 6.2300 mils (0.1583 mm)\nspacing: 8 mils (0.2032 mm)\n"
     (at 15.24 201.93 0)
     (effects (font (size 1.27 1.27)) (justify left bottom))

Commit message: pi-carrier: relocate M.2 power
Problem: the M.2 power is located in an odd place.

Move it over next to the e-fuse.
Parts:
- removed JP1, JP2, JP3: SolderJumper_2_Bridged, Jumper:SolderJumper-2_P1.3mm_Bridged_RoundedPad1.0x1.5mm, symbol Jumper:SolderJumper_2_Bridged
Connections:
- net M2_3V3: now also C24.1, C25.1, C26.2, L1.2, R2.1
- net PCIE_5V: now also C21.1, C22.1, C27.1, U7.1 (VIN)
- net PCIE_PWR_EN: now also R18.2, R4.1, U7.5 (EN)
Changed lines of the file:
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@@
   (junction (at 148.59 135.89) (diameter 0) (color 0 0 0 0)
-  )
-  (junction (at 190.5 135.89) (diameter 0) (color 0 0 0 0)
   )
   (junction (at 135.89 135.89) (diameter 0) (color 0 0 0 0)
@@
     (stroke (width 0) (type default))
   )
-  (wire (pts (xy 68.58 163.83) (xy 80.645 163.83))
+  (wire (pts (xy 47.625 163.83) (xy 80.645 163.83))
     (stroke (width 0) (type default))
   )
@@
     (stroke (width 0) (type default))
   )
-  (wire (pts (xy 175.26 135.89) (xy 177.8 135.89))
+  (wire (pts (xy 175.26 135.89) (xy 194.31 135.89))
     (stroke (width 0) (type default))
   )
@@
     (stroke (width 0) (type default))
   )
-  (wire (pts (xy 40.005 163.83) (xy 60.96 163.83))
-    (stroke (width 0) (type default))
-  )
   (wire (pts (xy 114.3 142.24) (xy 114.3 138.43))
     (stroke (width 0) (type default))
@@
     (stroke (width 0) (type default))
   )
-  (wire (pts (xy 190.5 135.89) (xy 201.93 135.89))
-    (stroke (width 0) (type default))
-  )
   (wire (pts (xy 86.36 140.97) (xy 86.36 143.51))
     (stroke (width 0) (type default))
@@
   )
   (wire (pts (xy 58.42 44.45) (xy 58.42 52.07))
-    (stroke (width 0) (type default))
-  )
-  (wire (pts (xy 190.5 135.89) (xy 185.42 135.89))
     (stroke (width 0) (type default))
   )
@@
     (effects (font (size 1.27 1.27)) (justify left bottom))
   )
-  (label "M2_3V3" (at 201.93 135.89 180) (fields_autoplaced)
+  (label "M2_3V3" (at 194.31 135.89 180) (fields_autoplaced)
     (effects (font (size 1.27 1.27)) (justify right bottom))
   )
@@
     (effects (font (size 1.27 1.27)) (justify right bottom))
   )
-  (label "PCIE_PWR_EN" (at 40.005 163.83 0) (fields_autoplaced)
+  (label "PCIE_PWR_EN" (at 47.625 163.83 0) (fields_autoplaced)
     (effects (font (size 1.27 1.27)) (justify left bottom))
   )
@@
     (effects (font (size 1.27 1.27)) (justify left bottom))
   )
-  (hierarchical_label "PCIE_5V" (shape input) (at 31.75 135.89 180) (fields_autoplaced)
+  (hierarchical_label "PCIE_5V" (shape input) (at 39.37 135.89 180) (fields_autoplaced)
     (effects (font (size 1.27 1.27)) (justify right))
   )
@@
     )
   )
-  (symbol (lib_id "Jumper:SolderJumper_2_Bridged") (at 181.61 135.89 0) (unit 1)
-    (in_bom yes) (on_board yes) (dnp no) (fields_autoplaced)
-    (property "Reference" "JP2" (at 181.61 132.08 0)
-      (effects (font (size 1.27 1.27)))
-    )
-    (property "Value" "SolderJumper_2_Bridged" (at 181.61 132.08 0)
-      (effects (font (size 1.27 1.27)) hide)
-    )
-    (property "Footprint" "Jumper:SolderJumper-2_P1.3mm_Bridged_RoundedPad1.0x1.5mm" (at 181.61 135.89 0)
-      (effects (font (size 1.27 1.27)) hide)
-    )
-    (property "Datasheet" "~" (at 181.61 135.89 0)
-      (effects (font (size 1.27 1.27)) hide)
-    )
-    (pin "2")
-    (pin "1")
-    (instances
-      (project "eurocard"
-        (path "/e048be62-6e5d-4330-8748-f1a6c1c5d89d/78247a58-bd33-4427-a596-05636cd08db2"
-          (reference "JP2") (unit 1)
-        )
-      )
-    )
-  )
   (symbol (lib_id "Regulator_Switching:TPS563202S") (at 101.6 138.43 0) (unit 1)
     (in_bom yes) (on_board yes) (dnp no) (fields_autoplaced)
@@
     )
   )
-  (symbol (lib_id "Jumper:SolderJumper_2_Bridged") (at 64.77 163.83 0) (unit 1)
-    (in_bom yes) (on_board yes) (dnp no) (fields_autoplaced)
-    (property "Reference" "JP3" (at 64.77 160.02 0)
-      (effects (font (size 1.27 1.27)))
-    )
-    (property "Value" "SolderJumper_2_Bridged" (at 64.77 160.02 0)
-      (effects (font (size 1.27 1.27)) hide)
-    )
-    (property "Footprint" "Jumper:SolderJumper-2_P1.3mm_Bridged_RoundedPad1.0x1.5mm" (at 64.77 163.83 0)
-      (effects (font (size 1.27 1.27)) hide)
-    )
-    (property "Datasheet" "~" (at 64.77 163.83 0)
-      (effects (font (size 1.27 1.27)) hide)
-    )
-    (pin "2")
-    (pin "1")
-    (instances
-      (project "eurocard"
-        (path "/e048be62-6e5d-4330-8748-f1a6c1c5d89d/78247a58-bd33-4427-a596-05636cd08db2"
-          (reference "JP3") (unit 1)
-        )
-      )
-    )
-  )
   (symbol (lib_id "Device:C") (at 69.85 139.7 0) (unit 1)
     (in_bom yes) (on_board yes) (dnp no)
@@
     )
     (property "Value" "PWR_FLAG" (at 41.91 130.81 0)
-      (effects (font (size 1.27 1.27)))
+      (effects (font (size 1.27 1.27)) hide)
     )
     (property "Footprint" "" (at 41.91 135.89 0)
@@
     )
   )
-  (symbol (lib_id "power:PWR_FLAG") (at 190.5 135.89 0) (unit 1)
-    (in_bom yes) (on_board yes) (dnp no)
-    (property "Reference" "#FLG06" (at 190.5 133.985 0)
-      (effects (font (size 1.27 1.27)) hide)
-    )
-    (property "Value" "PWR_FLAG" (at 190.5 130.81 0)
-      (effects (font (size 1.27 1.27)))
-    )
-    (property "Footprint" "" (at 190.5 135.89 0)
-      (effects (font (size 1.27 1.27)) hide)
-    )
-    (property "Datasheet" "~" (at 190.5 135.89 0)
-      (effects (font (size 1.27 1.27)) hide)
-    )
-    (pin "1")
-    (instances
-      (project "eurocard"
-        (path "/e048be62-6e5d-4330-8748-f1a6c1c5d89d/78247a58-bd33-4427-a596-05636cd08db2"
-          (reference "#FLG06") (unit 1)
-        )
-      )
-    )
-  )
   (symbol (lib_id "power:GND") (at 101.6 147.32 0) (unit 1)
     (in_bom yes) (on_board yes) (dnp no) (fields_autoplaced)
@@
         )
       )
-    )
-  )
-  (symbol (lib_id "Jumper:SolderJumper_2_Bridged") (at 35.56 135.89 0) (unit 1)
-    (in_bom yes) (on_board yes) (dnp no) (fields_autoplaced)
-    (property "Reference" "JP1" (at 35.56 132.08 0)
-      (effects (font (size 1.27 1.27)))
-    )
-    (property "Value" "SolderJumper_2_Bridged" (at 35.56 132.08 0)
-      (effects (font (size 1.27 1.27)) hide)
-    )
-    (property "Footprint" "Jumper:SolderJumper-2_P1.3mm_Bridged_RoundedPad1.0x1.5mm" (at 35.56 135.89 0)
-      (effects (font (size 1.27 1.27)) hide)
-    )
-    (property "Datasheet" "~" (at 35.56 135.89 0)
-      (effects (font (size 1.27 1.27)) hide)
-    )
-    (pin "2")
-    (pin "1")
-    (instances
-      (project "eurocard"
-        (path "/e048be62-6e5d-4330-8748-f1a6c1c5d89d/78247a58-bd33-4427-a596-05636cd08db2"
-          (reference "JP1") (unit 1)
-        )
-      )

Commit message: pi-carrier: update to version 4
Problem: design files and board skil still says v3.2.

Bump to v4.

Also change some schematic page sizes from A4 to US letter.
Other:
- company: (none) -> WorlickWerx
- title: (none) -> Molliebus Pi Carrier
Changed lines of the file:
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@@
 (kicad_sch (version 20230121) (generator eeschema)
   (paper "USLetter")
+  (title_block
+    (title "Molliebus Pi Carrier")
+    (date "2024-04-20")
+    (rev "4")
+    (company "WorlickWerx")
+    (comment 1 "SPDX-License-Identifier: CERN-OHL-1.2")
+  )
   (junction (at 80.645 163.83) (diameter 0) (color 0 0 0 0)
   )
