File: hardware/pi-carrier/m2.kicad_sch (KiCad schematic)
At the start: 20 parts, among them J4 Bus_M.2_Socket_M, J7 Conn_01x16_MountingPin, U7 TPS563203

Commit message: pi-carrier: fix kicad ERC errors
Problem: kicad 8 has some new ERC failures.

Set power output pin of eFuse to correct type.
Remove extra power flags.
Changed lines of the file:
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@@
-	)
-	(junction
-		(at 41.91 135.89)
-		(diameter 0)
-		(color 0 0 0 0)
 	)
 	(junction
@@
 	(wire
 		(pts
-			(xy 39.37 135.89) (xy 41.91 135.89)
+			(xy 39.37 135.89) (xy 46.99 135.89)
 		)
 		(stroke
@@
 		(pts
 			(xy 173.99 39.37) (xy 191.77 39.37)
-		)
-		(stroke
-			(width 0)
-			(type default)
-		)
-	)
-	(wire
-		(pts
-			(xy 41.91 135.89) (xy 46.99 135.89)
 		)
 		(stroke
@@
 					(unit 1)
 				)
-			)
-		)
-	)
-	(symbol
-		(lib_id "power:PWR_FLAG")
-		(at 41.91 135.89 0)
-		(unit 1)
-		(exclude_from_sim no)
-		(in_bom yes)
-		(on_board yes)
-		(dnp no)
-		(fields_autoplaced yes)
-		(property "Reference" "#FLG05"
-			(at 41.91 133.985 0)
-			(effects
-				(font
-					(size 1.27 1.27)
-				)
-				(hide yes)
-			)
-		)
-		(property "Value" "PWR_FLAG"
-			(at 41.91 130.81 0)
-			(effects
-				(font
-					(size 1.27 1.27)
-				)
-				(hide yes)
-			)
-		)
-		(property "Footprint" ""
-			(at 41.91 135.89 0)
-			(effects
-				(font
-					(size 1.27 1.27)
-				)
-				(hide yes)
-			)
-		)
-		(property "Datasheet" "~"
-			(at 41.91 135.89 0)
-			(effects
-				(font
-					(size 1.27 1.27)
-				)
-				(hide yes)
-			)
-		)
-		(property "Description" ""
-			(at 41.91 135.89 0)
-			(effects
-				(font
-					(size 1.27 1.27)
-				)
-				(hide yes)
-			)
-		)
-		(pin "1"
-		)
-		(instances
-			(project "eurocard"
-				(path "/e048be62-6e5d-4330-8748-f1a6c1c5d89d/78247a58-bd33-4427-a596-05636cd08db2"
-					(reference "#FLG05")
-					(unit 1)
-				)
