File: hardware/pi-carrier/efuse.kicad_sch (KiCad schematic)
At the start: 9 parts, among them U13 TPS2421-1DDAR

Commit message: pi-carrier: fix efuse powerpad signal type
Problem: the efuse has a "powerpad" on the bottom that is
labeled as a bidirectional pin but should be grounded.

Fix the symbol to make that a power pin.
Also drop the symbol's implicit connection to a nonexistent footprint.
Parts:
- U13: footprint 00_eurocard:VREG_LM5017MR_NOPB -> TPS2421-1DDAR:VREG_LM5017MR_NOPB
Changed lines of the file:
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@@
       (effects (font (size 1.27 1.27)))
     )
-    (property "Footprint" "00_eurocard:VREG_LM5017MR_NOPB" (at 158.75 90.17 0)
+    (property "Footprint" "TPS2421-1DDAR:VREG_LM5017MR_NOPB" (at 158.75 90.17 0)
       (effects (font (size 1.27 1.27)) (justify bottom) hide)
     )

Commit message: pi-carrier: put 3V3 reg behind efuse
Problem: the efuse *might* allow for hot swapping, at least from
a current control point of view, but the linear 3V3 supply, which
is low current but has a large electrolytic capacitor, is still
directly connected to the bus.

Put it behind the efuse and relocate to the bottom of the board.
Parts:
- U13: footprint TPS2421-1DDAR:VREG_LM5017MR_NOPB -> 00_eurocard:VREG_LM5017MR_NOPB
Changed lines of the file:
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@@
       (effects (font (size 1.27 1.27)))
     )
-    (property "Footprint" "TPS2421-1DDAR:VREG_LM5017MR_NOPB" (at 158.75 90.17 0)
+    (property "Footprint" "00_eurocard:VREG_LM5017MR_NOPB" (at 158.75 90.17 0)
       (effects (font (size 1.27 1.27)) (justify bottom) hide)
     )

Commit message: pi-carrier: add some efuse calculations to notes
Problem: the calculations for efuse config may require change
based on prototype evaluation but the data sheet is not super
clear on how to calculate them.

Add some notes to the schematic.
Parts:
- R10: value 66.5K -> 49.9K
Other:
- note added: "Notes: R10 determines current limit: I_{SET} = fault current (fault timer started) I_{LIM} = 1.5 * I_{SET} R_{RSET} = 200KΩ / I_{SET} (recommended range of 49.9K to 200K) For maximum current within recommendations, R{RSET} = 49.9K. I_{SET} = 200K / 49.9K = 4.0A I_{LIM} = 1.5 * 4.0A = 6.0A C28 determines the fault timer period: C_{CT} = T_{FAULT} / (40 x 10^{3}) (farads and seconds) C_{CT} T_{FAUL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"
Changed lines of the file:
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@@
     (stroke (width 0) (type default))
+  )
+  (text "Notes:\n\nR10 determines current limit:\n\nI_{SET} = fault current (fault timer started)\nI_{LIM} = 1.5 * I_{SET}\nR_{RSET} = 200KΩ / I_{SET} (recommended range of 49.9K to 200K)\n\nFor maximum current within recommendations, R{RSET} = 49.9K.\nI_{SET} = 200K / 49.9K = 4.0A\nI_{LIM} = 1.5 * 4.0A = 6.0A\n\nC28 determines the fault timer period:\n\nC_{CT} = T_{FAULT} / (40 x 10^{3}) (farads and seconds)\n\nC_{CT}                  T_{FAULT}\n47 x 10^{-9} (47nF)   1880 x 10^{-6} = 1.8msec\n"
+    (at 20.32 191.77 0)
+    (effects (font (size 1.27 1.27)) (justify left bottom))
   )
   (hierarchical_label "VOUT" (shape input) (at 220.98 85.09 0) (fields_autoplaced)
@@
       (effects (font (size 1.27 1.27)))
     )
-    (property "Value" "66.5K" (at 132.08 82.55 90)
+    (property "Value" "49.9K" (at 132.08 82.55 90)
       (effects (font (size 1.27 1.27)))
     )
