File: hardware/pi-carrier/efuse.kicad_sch (KiCad schematic)
At the start: 7 parts, among them U13 TPS2421-1DDAR

Commit message: pi-carrier: fix kicad ERC errors
Problem: kicad 8 has some new ERC failures.

Set power output pin of eFuse to correct type.
Remove extra power flags.
Changed lines of the file:
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@@
 	)
 	(hierarchical_label "VOUT"
-		(shape input)
+		(shape output)
 		(at 213.36 85.09 0)
 		(fields_autoplaced yes)
