File: hardware/pi-carrier/ornet.kicad_sch (KiCad schematic)
At the start: 4 parts, among them U4 74LVC2G04, U5 74LVC2G38

Commit message: pi-carrier: update to version 4
Problem: design files and board skil still says v3.2.

Bump to v4.

Also change some schematic page sizes from A4 to US letter.
Other:
- company: (none) -> WorlickWerx
- title: (none) -> Molliebus Pi Carrier
Changed lines of the file:
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@@
 (kicad_sch (version 20230121) (generator eeschema)
-  (paper "A4")
+  (paper "USLetter")
+  (title_block
+    (title "Molliebus Pi Carrier")
+    (date "2024-04-20")
+    (rev "4")
+    (company "WorlickWerx")
+    (comment 1 "SPDX-License-Identifier: CERN-OHL-1.2")
+  )
   (junction (at 99.06 140.97) (diameter 0) (color 0 0 0 0)
   )
