File: hardware/40pin-adapter/40pin-adapter.kicad_pcb (KiCad board)
At the start: 2 copper layers, 16.1 x 51.5 mm, 3 parts, among them J1 Conn_02x20_Odd_Even, J2 Conn_02x20_Odd_Even

Commit message: hardware/40pin-adapter: use stackable connector
Rework this to use Samtec HLE-120-02-xxx-DV-BE-A
connector.  It is a low profile SMD connector with
holes to allow header pins to go through the board.

Call this version 2.0 on the silk screen.

Ordered from oshpark on 14 July 2020.
Parts:
- J1, J2: footprint Connector_PinSocket_2.54mm:PinSocket_2x20_P2.54mm_Vertical -> Connector_Samtec_HLE_SMD:Samtec_HLE-120-02-xxx-DV-BE-A_2x20_P2.54mm_Horizontal
- REF**: moved to B.Cu
- moved J2 27.1 mm to (165.1, 91.4), turned to 270 degrees
- moved J1 27.0 mm to (154.9, 91.4), turned to 270 degrees
- moved REF** 25.5 mm to (159.9, 91.4), turned to 90 degrees
Routing:
- net /PI38: track 11.0 -> 26.2 mm, vias 0 -> 2
- net /PI1: track 11.0 -> 15.7 mm, vias 0 -> 2
- net /PI3: track 11.0 -> 14.9 mm, vias 0 -> 2
- net /PI40: track 11.0 -> 14.9 mm, vias 0 -> 2
- net /PI2: track 11.0 -> 14.3 mm, vias 0 -> 2
- net /PI37: track 11.0 -> 14.3 mm, vias 0 -> 2
- net /PI39: track 11.0 -> 14.0 mm, vias 0 -> 2
- net /PI4: track 11.0 -> 14.0 mm, vias 0 -> 2
Other:
- board size 16.1 x 51.5 mm -> 20.3 x 50.8 mm
- board text added: "(c) WorlickWerx CERN-OHL-1.2"
- board text added: "1"
- board text added: "20pin-adapter v2.0"
- board text removed: "40pin-adapter v1.0 (c) 2020 WorlickWerx"
- board text removed: "CERN-OHL-1.2"

Commit message: hardware/40pin-adapter: reduce footprint, add LED,term
The pcb is larger than it needs to be.  Reduce the footprint
to just outside of the header pads, and move vias inward.

Also, may as well add a power LED here where it's more visible
than on the main board next to the connector.

I2C is perhaps better terminated here than the main board too,
since it's closer to the end of the bus, so add two 4.7K resistors.

We can always skip populating if the main board works out better.
Parts:
- removed REF**: OSHW-Logo_5.7x6mm_SilkScreen, Symbol:OSHW-Logo_5.7x6mm_SilkScreen
- added D1: LED, LED_SMD:LED_0805_2012Metric_Pad1.15x1.40mm_HandSolder, B.Cu at (160.0, 105.4)
- added R1: 330, Resistor_SMD:R_0805_2012Metric_Pad1.15x1.40mm_HandSolder, B.Cu at (160.0, 108.0)
- added R2: 4.7K, Resistor_SMD:R_0805_2012Metric_Pad1.15x1.40mm_HandSolder, B.Cu at (160.0, 74.9)
- added R3: 4.7K, Resistor_SMD:R_0805_2012Metric_Pad1.15x1.40mm_HandSolder, B.Cu at (160.0, 77.5)
Connections:
- net /PI1 renamed +3V3
- net /PI25 renamed GND
- net /PI4 renamed +5V
Routing:
- net +5V: track 14.0 -> 52.7 mm
- net +3V3: track 15.7 -> 32.5 mm
- net /PI38: track 26.2 -> 11.2 mm, vias 2 -> 0
- net /PI3: track 14.9 -> 25.9 mm
- net GND: track 11.0 -> 18.2 mm, vias 0 -> 1
- net /PI5: track 11.0 -> 15.6 mm, vias 0 -> 1
- net /PI40: track 14.9 -> 11.8 mm
- net /PI39: track 14.0 -> 11.3 mm
- net Net-(D1-Pad2): track 0.00 -> 2.54 mm
- net /PI37: track 14.3 -> 12.0 mm
- net /PI2: track 14.3 -> 12.2 mm
- net /PI17: vias 0 -> 1
Other:
- board size 20.3 x 50.8 mm -> 17.8 x 50.8 mm
- board text added: "(c) 2020 WorlickWerx"
- board text added: "40pin-adapter v3"
- board text added: "CERN-OHL-1.2"
- board text added: "i2c term"
- board text added: "on"
- board text removed: "(c) WorlickWerx CERN-OHL-1.2"
- board text removed: "1"
- board text removed: "20pin-adapter v2.0"

Commit message: 40pin-adapter: drop LED and term, update footprint
Problem: The LED and i2c terminators need to be on the
main board, not the adapter, leaving open the possibility of
using an IDC ribbon cable instead.

Drop them from the adapter and update the version to v4.

Adjust schematic to letter size and fill in title, etc..
Update PCB.
Parts:
- removed D1: LED, LED_SMD:LED_0805_2012Metric_Pad1.15x1.40mm_HandSolder
- removed R1: 330, Resistor_SMD:R_0805_2012Metric_Pad1.15x1.40mm_HandSolder
- removed R2, R3: 4.7K, Resistor_SMD:R_0805_2012Metric_Pad1.15x1.40mm_HandSolder
- J1, J2: footprint Connector_Samtec_HLE_SMD:Samtec_HLE-120-02-xxx-DV-BE-A_2x20_P2.54mm_Horizontal -> 00_40pin-adapter:Samtec_HLE-120-02-xxx-DV-BE-A_2x20_P2.54mm_Horizontal
Connections:
- net +3V3 renamed /PI1
- net +5V renamed /PI4
- net GND renamed /PI25
Routing:
- net /PI4: track 52.7 -> 11.0 mm, vias 2 -> 0
- net /PI1: track 32.5 -> 13.4 mm
- net /PI3: track 25.9 -> 12.4 mm
- net /PI25: track 18.2 -> 11.0 mm, vias 1 -> 0
- net /PI5: track 15.6 -> 11.0 mm, vias 1 -> 0
- net Net-(D1-Pad2): track 2.54 -> 0.00 mm
Other:
- board text added: "40pin-adapter v4"
- board text removed: "40pin-adapter v3"
- board text removed: "i2c term"
- board text removed: "on"
