File: hardware/40pin-adapter/40pin-adapter.sch (KiCad schematic (older format))
At the start: 2 parts, among them J1 Conn_02x20_Odd_Even, J2 Conn_02x20_Odd_Even

Commit message: hardware/40pin-adapter: use stackable connector
Rework this to use Samtec HLE-120-02-xxx-DV-BE-A
connector.  It is a low profile SMD connector with
holes to allow header pins to go through the board.

Call this version 2.0 on the silk screen.

Ordered from oshpark on 14 July 2020.
Parts:
- J1, J2: footprint Connector_PinSocket_2.54mm:PinSocket_2x20_P2.54mm_Vertical -> Connector_Samtec_HLE_SMD:Samtec_HLE-120-02-xxx-DV-BE-A_2x20_P2.54mm_Horizontal
Changed lines of the file:
@@
 F 0 "J2" H 4400 4475 50  0000 C CNN
 F 1 "Conn_02x20_Odd_Even" H 4400 4476 50  0001 C CNN
-F 2 "Connector_PinSocket_2.54mm:PinSocket_2x20_P2.54mm_Vertical" H 4350 3450 50  0001 C CNN
+F 2 "Connector_Samtec_HLE_SMD:Samtec_HLE-120-02-xxx-DV-BE-A_2x20_P2.54mm_Horizontal" H 4350 3450 50  0001 C CNN
 F 3 "~" H 4350 3450 50  0001 C CNN
 	1    4350 3450
@@
 F 0 "J1" H 2750 4475 50  0000 C CNN
 F 1 "Conn_02x20_Odd_Even" H 2750 4476 50  0001 C CNN
-F 2 "Connector_PinSocket_2.54mm:PinSocket_2x20_P2.54mm_Vertical" H 2700 3450 50  0001 C CNN
+F 2 "Connector_Samtec_HLE_SMD:Samtec_HLE-120-02-xxx-DV-BE-A_2x20_P2.54mm_Horizontal" H 2700 3450 50  0001 C CNN
 F 3 "~" H 2700 3450 50  0001 C CNN
 	1    2700 3450

Commit message: hardware/40pin-adapter: reduce footprint, add LED,term
The pcb is larger than it needs to be.  Reduce the footprint
to just outside of the header pads, and move vias inward.

Also, may as well add a power LED here where it's more visible
than on the main board next to the connector.

I2C is perhaps better terminated here than the main board too,
since it's closer to the end of the bus, so add two 4.7K resistors.

We can always skip populating if the main board works out better.
Parts:
- added D1: LED, LED_SMD:LED_0805_2012Metric_Pad1.15x1.40mm_HandSolder, symbol Device:LED
- added R1: 330, Resistor_SMD:R_0805_2012Metric_Pad1.15x1.40mm_HandSolder, symbol Device:R
- added R2, R3: 4.7K, Resistor_SMD:R_0805_2012Metric_Pad1.15x1.40mm_HandSolder, symbol Device:R
Connections:
- net PI3: now also R3.1
- net PI5: now also R2.1
- net PI1 renamed +3V3
- net +3V3: now also R2.2, R3.2
- net PI25 renamed GND
- net GND: now also D1.1 (K)
- net PI4 renamed +5V
- net +5V: now also R1.2
- new net: D1.2 (A), R1.1
Changed lines of the file:
@@
 PI40
-Wire Wire Line
-	4150 2550 3800 2550
-Text Label 3800 2550 0    50   ~ 0
-PI1
 Wire Wire Line
 	4150 2650 3800 2650
@@
 Text Label 2150 4450 0    50   ~ 0
 PI39
+$Comp
+L Device:LED D1
+U 1 1 5F399C28
+P 6350 3800
+F 0 "D1" V 6389 3682 50  0000 R CNN
+F 1 "LED" V 6298 3682 50  0000 R CNN
+F 2 "LED_SMD:LED_0805_2012Metric_Pad1.15x1.40mm_HandSolder" H 6350 3800 50  0001 C CNN
+F 3 "~" H 6350 3800 50  0001 C CNN
+	1    6350 3800
+	0    -1   -1   0
+$EndComp
+$Comp
+L Device:R R1
+U 1 1 5F39A021
+P 6350 3200
+F 0 "R1" H 6280 3154 50  0000 R CNN
+F 1 "330" H 6280 3245 50  0000 R CNN
+F 2 "Resistor_SMD:R_0805_2012Metric_Pad1.15x1.40mm_HandSolder" V 6280 3200 50  0001 C CNN
+F 3 "~" H 6350 3200 50  0001 C CNN
+	1    6350 3200
+	-1   0    0    1
+$EndComp
+$Comp
+L power:GND #PWR0101
+U 1 1 5F3A67F0
+P 6350 4300
+F 0 "#PWR0101" H 6350 4050 50  0001 C CNN
+F 1 "GND" H 6355 4127 50  0000 C CNN
+F 2 "" H 6350 4300 50  0001 C CNN
+F 3 "" H 6350 4300 50  0001 C CNN
+	1    6350 4300
+	1    0    0    -1
+$EndComp
+Wire Wire Line
+	6350 3950 6350 4300
+Wire Wire Line
+	6350 3350 6350 3650
+$Comp
+L power:+5V #PWR0102
+U 1 1 5F3B4D8D
+P 6350 2700
+F 0 "#PWR0102" H 6350 2550 50  0001 C CNN
+F 1 "+5V" H 6365 2873 50  0000 C CNN
+F 2 "" H 6350 2700 50  0001 C CNN
+F 3 "" H 6350 2700 50  0001 C CNN
+	1    6350 2700
+	1    0    0    -1
+$EndComp
+Wire Wire Line
+	6350 2700 6350 3050
+$Comp
+L Device:R R2
+U 1 1 5F3B966D
+P 6950 3200
+F 0 "R2" H 6880 3154 50  0000 R CNN
+F 1 "4.7K" H 6880 3245 50  0000 R CNN
+F 2 "Resistor_SMD:R_0805_2012Metric_Pad1.15x1.40mm_HandSolder" V 6880 3200 50  0001 C CNN
+F 3 "~" H 6950 3200 50  0001 C CNN
+	1    6950 3200
+	-1   0    0    1
+$EndComp
+$Comp
+L Device:R R3
+U 1 1 5F3B9B80
+P 7250 3200
+F 0 "R3" H 7180 3154 50  0000 R CNN
+F 1 "4.7K" H 7180 3245 50  0000 R CNN
+F 2 "Resistor_SMD:R_0805_2012Metric_Pad1.15x1.40mm_HandSolder" V 7180 3200 50  0001 C CNN
+F 3 "~" H 7250 3200 50  0001 C CNN
+	1    7250 3200
+	-1   0    0    1
+$EndComp
+$Comp
+L power:+3.3V #PWR0103
+U 1 1 5F3BA388
+P 6950 2700
+F 0 "#PWR0103" H 6950 2550 50  0001 C CNN
+F 1 "+3.3V" H 6965 2873 50  0000 C CNN
+F 2 "" H 6950 2700 50  0001 C CNN
+F 3 "" H 6950 2700 50  0001 C CNN
+	1    6950 2700
+	1    0    0    -1
+$EndComp
+Wire Wire Line
+	6950 2700 6950 2900
+Wire Wire Line
+	7250 3050 7250 2900
+Wire Wire Line
+	7250 2900 6950 2900
+Connection ~ 6950 2900
+Wire Wire Line
+	6950 2900 6950 3050
+Wire Wire Line
+	7250 3350 7250 3500
+Wire Wire Line
+	7250 3500 7550 3500
+Text Label 7550 3500 2    50   ~ 0
+SDA
+Wire Wire Line
+	6950 3350 6950 3600
+Wire Wire Line
+	6950 3600 7550 3600
+Text Label 7550 3600 2    50   ~ 0
+SCL
+$Comp
+L power:+5V #PWR0104
+U 1 1 5F3CCC53
+P 5800 2700
+F 0 "#PWR0104" H 5800 2550 50  0001 C CNN
+F 1 "+5V" H 5815 2873 50  0000 C CNN
+F 2 "" H 5800 2700 50  0001 C CNN
+F 3 "" H 5800 2700 50  0001 C CNN
+	1    5800 2700
+	1    0    0    -1
+$EndComp
+$Comp
+L power:GND #PWR0105
+U 1 1 5F3D1EE2
+P 5800 4300
+F 0 "#PWR0105" H 5800 4050 50  0001 C CNN
+F 1 "GND" H 5805 4127 50  0000 C CNN
+F 2 "" H 5800 4300 50  0001 C CNN
+F 3 "" H 5800 4300 50  0001 C CNN
+	1    5800 4300
+	1    0    0    -1
+$EndComp
+Wire Wire Line
+	5500 3200 6000 3200
+Text Label 6000 3200 2    50   ~ 0
+SDA
+Text Label 5500 3200 0    50   ~ 0
+PI3
+Wire Wire Line
+	5500 3300 6000 3300
+Text Label 6000 3300 2    50   ~ 0
+SCL
+Text Label 5500 3300 0    50   ~ 0
+PI5
+Wire Wire Line
+	5500 3900 5800 3900
+Text Label 5500 3900 0    50   ~ 0
+PI1
+$Comp
+L power:+3.3V #PWR0106
+U 1 1 5F3EB655
+P 5800 3650
+F 0 "#PWR0106" H 5800 3500 50  0001 C CNN
+F 1 "+3.3V" H 5815 3823 50  0000 C CNN
+F 2 "" H 5800 3650 50  0001 C CNN
+F 3 "" H 5800 3650 50  0001 C CNN
+	1    5800 3650
+	1    0    0    -1
+$EndComp
+$Comp
+L power:PWR_FLAG #FLG0101
+U 1 1 5F405B4B
+P 5800 2900
+F 0 "#FLG0101" H 5800 2975 50  0001 C CNN
+F 1 "PWR_FLAG" V 5800 3028 50  0001 L CNN
+F 2 "" H 5800 2900 50  0001 C CNN
+F 3 "~" H 5800 2900 50  0001 C CNN
+	1    5800 2900
+	0    1    1    0
+$EndComp
+Wire Wire Line
+	5800 2700 5800 2900
+$Comp
+L power:PWR_FLAG #FLG0102
+U 1 1 5F40B84E
+P 5800 3900
+F 0 "#FLG0102" H 5800 3975 50  0001 C CNN
+F 1 "PWR_FLAG" V 5800 4028 50  0001 L CNN
+F 2 "" H 5800 3900 50  0001 C CNN
+F 3 "~" H 5800 3900 50  0001 C CNN
+	1    5800 3900
+	0    1    1    0
+$EndComp
+Connection ~ 5800 3900
+$Comp
+L power:PWR_FLAG #FLG0103
+U 1 1 5F40C409
+P 5800 4100
+F 0 "#FLG0103" H 5800 4175 50  0001 C CNN
+F 1 "PWR_FLAG" V 5800 4228 50  0001 L CNN
+F 2 "" H 5800 4100 50  0001 C CNN
+F 3 "~" H 5800 4100 50  0001 C CNN
+	1    5800 4100
+	0    1    1    0
+$EndComp
+Wire Wire Line
+	4150 2550 3800 2550
+Text Label 3800 2550 0    50   ~ 0
+PI1
+Wire Wire Line
+	5500 2900 5800 2900
+Connection ~ 5800 2900
+Text Label 5500 2900 0    50   ~ 0
+PI4
+Wire Wire Line
+	5500 4100 5800 4100
+Wire Wire Line
+	5800 4100 5800 4300
+Connection ~ 5800 4100
+Text Label 5500 4100 0    50   ~ 0
+PI25
+Wire Wire Line
+	5800 3650 5800 3900
 $EndSCHEMATC

Commit message: 40pin-connector: copy footprint to local lib
Copy the one footprint used in this project to lib.pretty,
and update footprint mapping in schematic.

Drop fp-info-cache from git - this file should not be tracked.
Parts:
- J1, J2: footprint Connector_Samtec_HLE_SMD:Samtec_HLE-120-02-xxx-DV-BE-A_2x20_P2.54mm_Horizontal -> 00_40pin-connector:Samtec_HLE-120-02-xxx-DV-BE-A_2x20_P2.54mm_Horizontal
Changed lines of the file:
@@
 F 0 "J2" H 4400 4475 50  0000 C CNN
 F 1 "Conn_02x20_Odd_Even" H 4400 4476 50  0001 C CNN
-F 2 "Connector_Samtec_HLE_SMD:Samtec_HLE-120-02-xxx-DV-BE-A_2x20_P2.54mm_Horizontal" H 4350 3450 50  0001 C CNN
+F 2 "00_40pin-connector:Samtec_HLE-120-02-xxx-DV-BE-A_2x20_P2.54mm_Horizontal" H 4350 3450 50  0001 C CNN
 F 3 "~" H 4350 3450 50  0001 C CNN
 	1    4350 3450
@@
 F 0 "J1" H 2750 4475 50  0000 C CNN
 F 1 "Conn_02x20_Odd_Even" H 2750 4476 50  0001 C CNN
-F 2 "Connector_Samtec_HLE_SMD:Samtec_HLE-120-02-xxx-DV-BE-A_2x20_P2.54mm_Horizontal" H 2700 3450 50  0001 C CNN
+F 2 "00_40pin-connector:Samtec_HLE-120-02-xxx-DV-BE-A_2x20_P2.54mm_Horizontal" H 2700 3450 50  0001 C CNN
 F 3 "~" H 2700 3450 50  0001 C CNN
 	1    2700 3450

Commit message: 40pin-adapter: drop LED and term, update footprint
Problem: The LED and i2c terminators need to be on the
main board, not the adapter, leaving open the possibility of
using an IDC ribbon cable instead.

Drop them from the adapter and update the version to v4.

Adjust schematic to letter size and fill in title, etc..
Update PCB.
Parts:
- removed D1: LED, LED_SMD:LED_0805_2012Metric_Pad1.15x1.40mm_HandSolder, symbol Device:LED
- removed R1: 330, Resistor_SMD:R_0805_2012Metric_Pad1.15x1.40mm_HandSolder, symbol Device:R
- removed R2, R3: 4.7K, Resistor_SMD:R_0805_2012Metric_Pad1.15x1.40mm_HandSolder, symbol Device:R
- J1, J2: footprint 00_40pin-connector:Samtec_HLE-120-02-xxx-DV-BE-A_2x20_P2.54mm_Horizontal -> 00_40pin-adapter:Samtec_HLE-120-02-xxx-DV-BE-A_2x20_P2.54mm_Horizontal
Connections:
- net +3V3 renamed PI1
- net +5V renamed PI4
- net GND renamed PI25
Other:
- moved on the sheet: J1, J2
