File: hardware/bus-8/bus-8.kicad_pcb (KiCad board)
At the start: 2 copper layers, 198.9 x 128.6 mm, 108 parts, among them J1 C96ABC, J10 Conn_01x04, J11 Conn_01x04, J12 Conn_01x04, J13 Conn_01x04, J14 Conn_01x04, J15 Conn_01x04, J16 Conn_01x04, J17 Conn_01x04, J18 Conn_01x04, J19 Conn_01x04, J2 C96ABC, J20 Conn_01x04, J21 Conn_01x04, J22 Conn_01x04, J23 Conn_01x04, J24 Conn_01x04, J25 Conn_01x04, J26 Conn_01x04, J27 Conn_01x04, J28 Conn_01x04, J29 Conn_01x04, J3 C96ABC, J30 Conn_01x04, J31 Conn_01x04, J32 Conn_01x04, J33 Conn_01x04, J34 Conn_01x04, J35 Conn_01x04, J36 Conn_01x04, J37 Conn_01x04, J38 Conn_01x04, J39 Conn_01x04, J4 C96ABC, J40 Conn_01x04, J41 Conn_01x04, J42 Conn_01x04, J43 Conn_01x04, J44 Conn_01x04, J45 Conn_01x04, J46 Conn_01x04, J47 Conn_01x04, J48 Conn_01x04, J49 Conn_01x04, J5 C96ABC, J50 Conn_01x04, J51 Conn_01x04, J52 Conn_01x04, J53 Conn_01x04, J54 Conn_01x04, J55 Conn_01x04, J56 Conn_01x04, J57 Conn_01x04, J58 Conn_01x04, J59 Conn_01x04, J6 C96ABC, J60 Conn_01x04, J61 Conn_01x04, J62 Conn_01x04, J63 Conn_01x04, J64 Conn_01x04, J65 ATX-20, J66 Conn_02x07_Odd_Even, J67 Conn_02x07_Odd_Even, J7 C96ABC, J8 C96ABC, J9 Conn_01x04

Commit message: bus-8: make CAN term 0.25 W
Problem: CAN requires a 0.25 W terminator but we specified an
0605 package.

Specify the wattage and increase the package size to 1210.
Reroute PCB.
Parts:
- R1, R2: value 120 -> 120 0.25W; footprint Resistor_SMD:R_0603_1608Metric_Pad0.98x0.95mm_HandSolder -> Resistor_SMD:R_1210_3225Metric_Pad1.30x2.65mm_HandSolder
- moved J67 1.90 mm to (245.1, 61.6)
- moved R2 1.73 mm to (251.2, 67.1)
- moved JP17 1.65 mm to (59.4, 59.1)
- moved JP18 0.81 mm to (251.2, 61.6)
- moved R1 0.59 mm to (59.4, 64.3)
Routing:
- net /~RESET~: track 206.2 -> 210.8 mm
- net /OR_INA: track 207.8 -> 209.5 mm
- net /OR_INB: track 209.4 -> 211.0 mm
- net Net-(JP18-Pad1): track 2.12 -> 3.30 mm
- net /OR_OUT: track 213.8 -> 213.2 mm
Other:
- board text added: "supervisor in"
- board text added: "supervisor out"
- board text removed: "Crate supervisor IN"
- board text removed: "Crate supervisor OUT"

Commit message: bus-8: change resistors to TH
Problem: pcbwap PCBA online form thinks we need a stencil if there
are any SMT parts.  Since there are only two, make them TH.
Parts:
- R1, R2: footprint Resistor_SMD:R_1210_3225Metric_Pad1.30x2.65mm_HandSolder -> Resistor_THT:R_Axial_DIN0204_L3.6mm_D1.6mm_P7.62mm_Horizontal
- moved R1 7.09 mm to (59.7, 71.4)
- moved R2 4.55 mm to (251.2, 71.6)
- moved JP18 1.38 mm to (251.2, 60.2)
- moved JP17 1.24 mm to (59.4, 60.3)
Routing:
- net /CAN+: track 204.1 -> 210.6 mm
