File: hardware/supervisor/supervisor.kicad_pcb (KiCad board)
At the start: 2 copper layers, 40 x 100.1 mm, 53 parts, among them J1 Conn_02x05_Odd_Even, J2 Conn_02x10_Odd_Even, J3 Conn_02x07_Odd_Even, J4 RJ12, M1 Fan_4pin, M2 Fan_4pin, M3 Fan_4pin, SW1 SW_Push, SW3 SW_Push, U1 SN74LVC07ADB, U2 TCAN332DR, U3 LM1117-IMPX3.3, U4 SN74LVC1G86DBV, U5 SN74LVC2G74DCUR, U6 STM32F103C8T6, U7 CAT811TTBI-GT3, U8 SN74LVC07ADB, Y1 8Mhz

Commit message: supervisor: connect Vbat to Vdd
Problem: Vbat is floating, but AN2586 strongly recommends
to connect it to Vdd (3V3) when unused.

Connect Vbat to Vdd.
Connections:
- U6 pad 1: Net-(U6-Pad1) -> +3V3
Routing:
- net +3V3: track 342.7 -> 345.1 mm

Commit message: supervisor: add bypass cap for Vbat
Problem: it is suggested that Vbat should have a separate
100nF bypass cap.

Add cap.
Parts:
- added C16: 100nF 16V, Capacitor_SMD:C_0805_2012Metric_Pad1.18x1.45mm_HandSolder, B.Cu at (110.2, 65.6)
Routing:
- net +3V3: track 345.1 -> 344.4 mm
- net GND: vias 15 -> 16
Changed lines of the file:
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@@
   (general
     (thickness 1.6)
-    (drawings 78)
-    (tracks 818)
+    (drawings 76)
+    (tracks 822)
     (zones 0)
-    (modules 53)
+    (modules 54)
     (nets 80)
   )
@@
     (add_net "Net-(U6-Pad43)")
   )
+  (module Capacitor_SMD:C_0805_2012Metric_Pad1.18x1.45mm_HandSolder (layer B.Cu)
+    (at 110.236 65.5535 270)
+    (descr "Capacitor SMD 0805 (2012 Metric), square (rectangular) end terminal, IPC_7351 nominal with elongated pad for handsoldering. (Body size source: IPC-SM-782 page 76, https://www.pcb-3d.com/wordpress/wp-content/uploads/ipc-sm-782a_amendment_1_and_2.pdf, https://docs.google.com/spreadsheets/d/1BsfQQcO9C6DZCsRaXUlFlo91Tg2WpOkGARC1WS5S8t0/edit?usp=sharing), generated with kicad-footprint-generator")
+    (tags "capacitor handsolder")
+    (attr smd)
+    (fp_text reference C16 (at 0 1.68 90) (layer B.SilkS)
+      (effects (font (size 1 1) (thickness 0.15)) (justify mirror))
+    )
+    (fp_text value "100nF 16V" (at 0 -1.68 90) (layer B.Fab)
+      (effects (font (size 1 1) (thickness 0.15)) (justify mirror))
+    )
+    (fp_line (start 1.88 -0.98) (end -1.88 -0.98) (layer B.CrtYd) (width 0.05))
+    (fp_line (start 1.88 0.98) (end 1.88 -0.98) (layer B.CrtYd) (width 0.05))
+    (fp_line (start -1.88 0.98) (end 1.88 0.98) (layer B.CrtYd) (width 0.05))
+    (fp_line (start -1.88 -0.98) (end -1.88 0.98) (layer B.CrtYd) (width 0.05))
+    (fp_line (start -0.261252 -0.735) (end 0.261252 -0.735) (layer B.SilkS) (width 0.12))
+    (fp_line (start -0.261252 0.735) (end 0.261252 0.735) (layer B.SilkS) (width 0.12))
+    (fp_line (start 1 -0.625) (end -1 -0.625) (layer B.Fab) (width 0.1))
+    (fp_line (start 1 0.625) (end 1 -0.625) (layer B.Fab) (width 0.1))
+    (fp_line (start -1 0.625) (end 1 0.625) (layer B.Fab) (width 0.1))
+    (fp_line (start -1 -0.625) (end -1 0.625) (layer B.Fab) (width 0.1))
+    (fp_text user %R (at 0 0 90) (layer B.Fab)
+      (effects (font (size 0.5 0.5) (thickness 0.08)) (justify mirror))
+    )
+    (pad 2 smd roundrect (at 1.0375 0 270) (size 1.175 1.45) (layers B.Cu B.Paste B.Mask) (roundrect_rratio 0.212766)
+      (net 1 GND))
+    (pad 1 smd roundrect (at -1.0375 0 270) (size 1.175 1.45) (layers B.Cu B.Paste B.Mask) (roundrect_rratio 0.212766)
+      (net 3 +3V3))
+    (model ${KISYS3DMOD}/Capacitor_SMD.3dshapes/C_0805_2012Metric.wrl
+      (at (xyz 0 0 0))
+      (scale (xyz 1 1 1))
+      (rotate (xyz 0 0 0))
+    )
+  )
   (module Symbol:OSHW-Logo2_7.3x6mm_SilkScreen (layer B.Cu)
     (at 102.3112 144.78 180)
@@
     (tags "capacitor handsolder")
     (attr smd)
-    (fp_text reference C7 (at 0 1.68 90) (layer B.SilkS)
+    (fp_text reference C7 (at 0 -1.524 90) (layer B.SilkS)
       (effects (font (size 1 1) (thickness 0.15)) (justify mirror))
     )
@@
     (arrow2b (pts (xy 131.445 48.26) (xy 132.031421 49.386504)))
   )
-  (gr_line (start 130.556 50.546) (end 130.556 50.8) (layer F.SilkS) (width 0.12))
-  (gr_line (start 130.556 50.8) (end 130.556 50.546) (layer F.SilkS) (width 0.12))
   (gr_text SWD (at 102.362 58.674) (layer F.SilkS)
     (effects (font (size 1 1) (thickness 0.15)))
@@
   (via (at 94.3356 68.1228) (size 0.8) (drill 0.4) (layers F.Cu B.Cu) (net 1))
   (via (at 98.1456 57.404) (size 0.8) (drill 0.4) (layers F.Cu B.Cu) (net 1))
+  (via (at 115.57 58.166) (size 0.8) (drill 0.4) (layers F.Cu B.Cu) (net 1))
   (via (at 126.4158 140.8938) (size 0.8) (drill 0.4) (layers F.Cu B.Cu) (net 2))
   (segment (start 126.3904 142.4686) (end 126.3904 140.9192) (width 0.25) (layer B.Cu) (net 2))
@@
   (segment (start 126.478401 101.613599) (end 126.478401 96.292299) (width 0.5) (layer B.Cu) (net 3))
   (segment (start 107.8012 107.4892) (end 107.3912 107.8992) (width 0.25) (layer B.Cu) (net 3))
-  (via (at 108.91012 65.33388) (size 0.8) (drill 0.4) (layers F.Cu B.Cu) (net 3))
-  (segment (start 112.522 63.5) (end 110.744 63.5) (width 0.25) (layer F.Cu) (net 3))
-  (segment (start 110.744 63.5) (end 108.91012 65.33388) (width 0.25) (layer F.Cu) (net 3))
-  (segment (start 108.91012 70.15988) (end 108.839 70.231) (width 0.25) (layer B.Cu) (net 3))
-  (segment (start 108.91012 65.33388) (end 108.91012 70.15988) (width 0.25) (layer B.Cu) (net 3))
   (via (at 108.27004 107.2642) (size 0.8) (drill 0.4) (layers F.Cu B.Cu) (net 3))
   (segment (start 107.3912 107.2642) (end 108.27004 107.2642) (width 0.25) (layer F.Cu) (net 3))
@@
   (segment (start 100.711 58.8645) (end 100.9015 59.055) (width 0.25) (layer F.Cu) (net 3))
   (segment (start 95.3516 58.8645) (end 100.711 58.8645) (width 0.25) (layer F.Cu) (net 3))
-  (segment (start 110.04124 66.465) (end 108.91012 65.33388) (width 0.25) (layer F.Cu) (net 3))
-  (segment (start 110.8995 66.465) (end 110.04124 66.465) (width 0.25) (layer F.Cu) (net 3))
+  (segment (start 110.8995 66.465) (end 111.843 66.465) (width 0.25) (layer F.Cu) (net 3))
+  (segment (start 112.312 65.996) (end 112.312 65.0525) (width 0.25) (layer F.Cu) (net 3))
+  (segment (start 111.843 66.465) (end 112.312 65.996) (width 0.25) (layer F.Cu) (net 3))
+  (segment (start 108.91012 70.15988) (end 108.839 70.231) (width 0.25) (layer B.Cu) (net 3))
+  (segment (start 108.91012 66.04) (end 108.91012 70.15988) (width 0.25) (layer B.Cu) (net 3))
+  (via (at 108.91012 66.04) (size 0.8) (drill 0.4) (layers F.Cu B.Cu) (net 3))
+  (segment (start 109.33512 66.465) (end 108.91012 66.04) (width 0.25) (layer F.Cu) (net 3))
+  (segment (start 110.8995 66.465) (end 109.33512 66.465) (width 0.25) (layer F.Cu) (net 3))
+  (segment (start 108.91012 65.84188) (end 110.236 64.516) (width 0.25) (layer B.Cu) (net 3))
+  (segment (start 108.91012 66.04) (end 108.91012 65.84188) (width 0.25) (layer B.Cu) (net 3))
   (via (at 96.6089 63.5762) (size 0.8) (drill 0.4) (layers F.Cu B.Cu) (net 4))
   (segment (start 97.8863 63.5508) (end 96.6343 63.5508) (width 0.25) (layer F.Cu) (net 4))

Commit message: supervisor: add 1uF bypass on Vdda
Problem: AN2576 recomends a 1uF decoupling cap on Vdda, in
addition to the 100nF.

Add cap.
Parts:
- added C17: 1uF 16V, Capacitor_SMD:C_0805_2012Metric_Pad1.18x1.45mm_HandSolder, B.Cu at (112.5, 70.9)
Routing:
- net GND: track 48.1 -> 51.0 mm
- net +3V3: track 344.4 -> 347.3 mm

Commit message: supervisor: add cap to RESET~
Problem: AN2576 suggests 100nF cap on ~RESET to protect against
parasitic resets.

Add cap.
Parts:
- added C18: 100nF 16V, Capacitor_SMD:C_0805_2012Metric_Pad1.18x1.45mm_HandSolder, B.Cu at (106.7, 67.1)
Routing:
- net GND: track 51.0 -> 61.8 mm
- net /~RESET~: track 66.8 -> 68.8 mm

Commit message: supervisor: change fill clearance to 0.2mm
Problem: the 0.5mm fill clearance setting is way too conservative,
resulting in many extra tracks and vias needing to be manually added.

Reduce from 0.5mm to 0.2mm and remove redundant tracks and vias.

Pcbway's least expensive track spacing is 6 mils = 0.1524mm.

N.B. this causes groudn fill between pads of 0805 resistors, but
that should be OK AFAICT.
Routing:
- net GND: track 61.8 -> 7.96 mm, vias 16 -> 5

Commit message: supervisor: add HSE series resistor
Problem: AN2576 suggests that the HSE xtal should have a
series resistor with a value 5-6 times the xtal series resistance.

Add resistor, with typical value of 390 ohms for now.
Parts:
- added R9: 390, Resistor_SMD:R_0805_2012Metric_Pad1.20x1.40mm_HandSolder, B.Cu at (106.7, 71.1)
Connections:
- U6 pad 6: Net-(C12-Pad1) -> Net-(R9-Pad1)
Routing:
- net Net-(R9-Pad1): track 0.00 -> 8.25 mm, vias 0 -> 1
- net Net-(C12-Pad1): track 9.75 -> 5.43 mm
- net /~RESET~: track 68.8 -> 71.4 mm, vias 6 -> 5
- net /FAN3_PWM: track 14.2 -> 13.4 mm
Changed lines of the file:
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@@
     (thickness 1.6)
     (drawings 76)
-    (tracks 781)
+    (tracks 786)
     (zones 0)
-    (modules 56)
-    (nets 80)
+    (modules 57)
+    (nets 81)
   )
   (page A4)
@@
   (net 78 "Net-(J4-Pad1)")
   (net 79 "Net-(J4-Pad6)")
+  (net 80 "Net-(R9-Pad1)")
   (net_class Default "This is the default net class."
     (clearance 0.2)
@@
     (add_net "Net-(M3-Pad4)")
     (add_net "Net-(R10-Pad2)")
+    (add_net "Net-(R9-Pad1)")
     (add_net "Net-(SW3-Pad2)")
     (add_net "Net-(U1-Pad10)")
@@
     (add_net "Net-(U6-Pad43)")
   )
+  (module Resistor_SMD:R_0805_2012Metric_Pad1.20x1.40mm_HandSolder (layer B.Cu)
+    (at 106.68 71.136 270)
+    (descr "Resistor SMD 0805 (2012 Metric), square (rectangular) end terminal, IPC_7351 nominal with elongated pad for handsoldering. (Body size source: IPC-SM-782 page 72, https://www.pcb-3d.com/wordpress/wp-content/uploads/ipc-sm-782a_amendment_1_and_2.pdf), generated with kicad-footprint-generator")
+    (tags "resistor handsolder")
+    (attr smd)
+    (fp_text reference R9 (at 2.651 0 90) (layer B.SilkS)
+      (effects (font (size 1 1) (thickness 0.15)) (justify mirror))
+    )
+    (fp_text value 390 (at 0 -1.65 90) (layer B.Fab)
+      (effects (font (size 1 1) (thickness 0.15)) (justify mirror))
+    )
+    (fp_line (start 1.85 -0.95) (end -1.85 -0.95) (layer B.CrtYd) (width 0.05))
+    (fp_line (start 1.85 0.95) (end 1.85 -0.95) (layer B.CrtYd) (width 0.05))
+    (fp_line (start -1.85 0.95) (end 1.85 0.95) (layer B.CrtYd) (width 0.05))
+    (fp_line (start -1.85 -0.95) (end -1.85 0.95) (layer B.CrtYd) (width 0.05))
+    (fp_line (start -0.227064 -0.735) (end 0.227064 -0.735) (layer B.SilkS) (width 0.12))
+    (fp_line (start -0.227064 0.735) (end 0.227064 0.735) (layer B.SilkS) (width 0.12))
+    (fp_line (start 1 -0.625) (end -1 -0.625) (layer B.Fab) (width 0.1))
+    (fp_line (start 1 0.625) (end 1 -0.625) (layer B.Fab) (width 0.1))
+    (fp_line (start -1 0.625) (end 1 0.625) (layer B.Fab) (width 0.1))
+    (fp_line (start -1 -0.625) (end -1 0.625) (layer B.Fab) (width 0.1))
+    (fp_text user %R (at 0 0 90) (layer B.Fab)
+      (effects (font (size 0.5 0.5) (thickness 0.08)) (justify mirror))
+    )
+    (pad 2 smd roundrect (at 1 0 270) (size 1.2 1.4) (layers B.Cu B.Paste B.Mask) (roundrect_rratio 0.208333)
+      (net 68 "Net-(C12-Pad1)"))
+    (pad 1 smd roundrect (at -1 0 270) (size 1.2 1.4) (layers B.Cu B.Paste B.Mask) (roundrect_rratio 0.208333)
+      (net 80 "Net-(R9-Pad1)"))
+    (model ${KISYS3DMOD}/Resistor_SMD.3dshapes/R_0805_2012Metric.wrl
+      (at (xyz 0 0 0))
+      (scale (xyz 1 1 1))
+      (rotate (xyz 0 0 0))
+    )
+  )
   (module Capacitor_SMD:C_0805_2012Metric_Pad1.18x1.45mm_HandSolder (layer B.Cu)
     (at 106.68 67.056 270)
@@
       (net 25 /~RESET~))
     (pad 6 smd roundrect (at -4.1625 -0.25) (size 1.475 0.3) (layers F.Cu F.Paste F.Mask) (roundrect_rratio 0.25)
-      (net 68 "Net-(C12-Pad1)"))
+      (net 80 "Net-(R9-Pad1)"))
     (pad 5 smd roundrect (at -4.1625 -0.75) (size 1.475 0.3) (layers F.Cu F.Paste F.Mask) (roundrect_rratio 0.25)
       (net 67 "Net-(C11-Pad1)"))
@@
   (segment (start 97.605 69.215) (end 97.79 69.03) (width 0.25) (layer F.Cu) (net 25))
   (segment (start 96.52 69.215) (end 97.605 69.215) (width 0.25) (layer F.Cu) (net 25))
-  (via (at 105.886153 69.818153) (size 0.8) (drill 0.4) (layers F.Cu B.Cu) (net 25))
-  (segment (start 106.261807 69.442499) (end 105.886153 69.818153) (width 0.25) (layer F.Cu) (net 25))
   (segment (start 110.8995 69.465) (end 110.876999 69.442499) (width 0.25) (layer F.Cu) (net 25))
-  (segment (start 110.876999 69.442499) (end 106.261807 69.442499) (width 0.25) (layer F.Cu) (net 25))
-  (via (at 103.632 69.342) (size 0.8) (drill 0.4) (layers F.Cu B.Cu) (net 25))
-  (segment (start 105.886153 69.818153) (end 105.41 69.342) (width 0.25) (layer B.Cu) (net 25))
-  (segment (start 105.41 69.342) (end 103.632 69.342) (width 0.25) (layer B.Cu) (net 25))
-  (segment (start 103.632 69.342) (end 102.743 70.231) (width 0.25) (layer F.Cu) (net 25))
-  (segment (start 98.991 70.231) (end 97.79 69.03) (width 0.25) (layer F.Cu) (net 25))
-  (segment (start 102.743 70.231) (end 98.991 70.231) (width 0.25) (layer F.Cu) (net 25))
   (via (at 96.0374 72.4916) (size 0.8) (drill 0.4) (layers F.Cu B.Cu) (net 25))
   (segment (start 96.0374 69.6976) (end 96.52 69.215) (width 0.25) (layer F.Cu) (net 25))
@@
   (segment (start 105.649198 104.521) (end 107.214598 102.9556) (width 0.25) (layer F.Cu) (net 25))
   (segment (start 98.602801 104.521) (end 105.649198 104.521) (width 0.25) (layer F.Cu) (net 25))
-  (segment (start 105.886153 68.887347) (end 106.68 68.0935) (width 0.25) (layer B.Cu) (net 25))
-  (segment (start 105.886153 69.818153) (end 105.886153 68.887347) (width 0.25) (layer B.Cu) (net 25))
+  (via (at 104.532682 67.624864) (size 0.8) (drill 0.4) (layers F.Cu B.Cu) (net 25))
+  (segment (start 106.211364 67.624864) (end 104.532682 67.624864) (width 0.25) (layer B.Cu) (net 25))
+  (segment (start 106.68 68.0935) (end 106.211364 67.624864) (width 0.25) (layer B.Cu) (net 25))
+  (segment (start 98.615001 69.855001) (end 97.79 69.03) (width 0.25) (layer F.Cu) (net 25))
+  (segment (start 102.507363 69.855001) (end 98.615001 69.855001) (width 0.25) (layer F.Cu) (net 25))
+  (segment (start 104.532682 67.624864) (end 104.532682 67.829682) (width 0.25) (layer F.Cu) (net 25))
+  (segment (start 102.897364 69.465) (end 102.564182 69.798182) (width 0.25) (layer F.Cu) (net 25))
+  (segment (start 110.8995 69.465) (end 102.897364 69.465) (width 0.25) (layer F.Cu) (net 25))
+  (segment (start 102.564182 69.798182) (end 102.507363 69.855001) (width 0.25) (layer F.Cu) (net 25))
+  (segment (start 104.532682 67.829682) (end 102.564182 69.798182) (width 0.25) (layer F.Cu) (net 25))
   (via (at 122.428 94.869) (size 0.8) (drill 0.4) (layers F.Cu B.Cu) (net 26))
   (segment (start 122.395999 94.836999) (end 122.428 94.869) (width 0.25) (layer F.Cu) (net 26))
@@
   (segment (start 100.6184 82.1436) (end 100.6392 82.1228) (width 0.25) (layer F.Cu) (net 63))
   (segment (start 97.9424 82.1436) (end 100.6184 82.1436) (width 0.25) (layer F.Cu) (net 63))
-  (via (at 107.927435 72.139562) (size 0.8) (drill 0.4) (layers F.Cu B.Cu) (net 64))
-  (segment (start 108.496474 72.708601) (end 107.927435 72.139562) (width 0.25) (layer F.Cu) (net 64))
-  (segment (start 110.8995 71.965) (end 110.155899 72.708601) (width 0.25) (layer F.Cu) (net 64))
-  (segment (start 110.155899 72.708601) (end 108.496474 72.708601) (width 0.25) (layer F.Cu) (net 64))
-  (segment (start 107.927435 72.139562) (end 108.46519 72.677317) (width 0.25) (layer B.Cu) (net 64))
-  (segment (start 108.46519 72.677317) (end 108.46519 77.10721) (width 0.25) (layer B.Cu) (net 64))
   (via (at 105.9688 79.6036) (size 0.8) (drill 0.4) (layers F.Cu B.Cu) (net 64))
   (segment (start 108.46519 77.10721) (end 105.9688 79.6036) (width 0.25) (layer B.Cu) (net 64))
   (segment (start 105.9688 79.6036) (end 107.905801 79.6036) (width 0.25) (layer F.Cu) (net 64))
+  (via (at 108.077 72.644) (size 0.8) (drill 0.4) (layers F.Cu B.Cu) (net 64))
+  (segment (start 108.014601 72.708601) (end 107.95 72.644) (width 0.25) (layer F.Cu) (net 64))
+  (segment (start 110.155899 72.708601) (end 108.014601 72.708601) (width 0.25) (layer F.Cu) (net 64))
+  (segment (start 110.8995 71.965) (end 110.155899 72.708601) (width 0.25) (layer F.Cu) (net 64))
+  (segment (start 108.46519 73.15919) (end 108.46519 73.39881) (width 0.25) (layer B.Cu) (net 64))
+  (segment (start 107.95 72.644) (end 108.46519 73.15919) (width 0.25) (layer B.Cu) (net 64))
+  (segment (start 108.46519 73.39881) (end 108.46519 77.10721) (width 0.25) (layer B.Cu) (net 64))
   (via (at 108.9152 71.9836) (size 0.8) (drill 0.4) (layers F.Cu B.Cu) (net 65))
   (segment (start 110.8995 71.465) (end 109.4338 71.465) (width 0.25) (layer F.Cu) (net 65))
@@
   (segment (start 110.8995 68.465) (end 106.692 68.465) (width 0.25) (layer F.Cu) (net 67))
   (segment (start 104.013 70.666) (end 104.013 72.8218) (width 0.25) (layer B.Cu) (net 68))
-  (segment (start 105.714 68.965) (end 104.013 70.666) (width 0.25) (layer F.Cu) (net 68))
-  (segment (start 110.8995 68.965) (end 105.714 68.965) (width 0.25) (layer F.Cu) (net 68))
+  (segment (start 105.483 72.136) (end 104.013 70.666) (width 0.25) (layer B.Cu) (net 68))
+  (segment (start 106.68 72.136) (end 105.483 72.136) (width 0.25) (layer B.Cu) (net 68))
   (via (at 102.88524 101.79812) (size 0.8) (drill 0.4) (layers F.Cu B.Cu) (net 71))
   (segment (start 102.944761 101.738599) (end 102.88524 101.79812) (width 0.25) (layer F.Cu) (net 71))
@@
   (segment (start 94.264599 60.990599) (end 94.264599 62.311399) (width 0.25) (layer B.Cu) (net 77))
   (segment (start 90.678 59.071) (end 91.558501 59.951501) (width 0.25) (layer B.Cu) (net 77))
+  (segment (start 105.261421 68.965) (end 105.011908 68.715487) (width 0.25) (layer F.Cu) (net 80))
+  (via (at 105.011908 68.715487) (size 0.8) (drill 0.4) (layers F.Cu B.Cu) (net 80))
+  (segment (start 110.8995 68.965) (end 105.261421 68.965) (width 0.25) (layer F.Cu) (net 80))
+  (segment (start 105.259487 68.715487) (end 106.68 70.136) (width 0.25) (layer B.Cu) (net 80))
+  (segment (start 105.011908 68.715487) (end 105.259487 68.715487) (width 0.25) (layer B.Cu) (net 80))
   (zone (net 1) (net_name GND) (layer F.Cu) (hatch edge 0.508)
     (connect_pads (clearance 0.2))

Commit message: supervisor: insert open drain driver in ~reset
Problem: ~RESET is pulled up within the STM32, so driving it with
push-pull CAT811 output is inappropriate.

Route ~RESET through an unused SN74LVC07 gate so that the STM32
input (and the D flip flop clear input which is attached) has an
open drain driver.
Connections:
- R11 pad 2: /~RESET~ -> Net-(R11-Pad2)
- U1 pad 3: /~RESET~ -> Net-(R11-Pad2)
- U1 pad 8: Net-(U1-Pad8) -> /~RESET~
- U1 pad 9: GND -> Net-(R11-Pad2)
- U7 pad 2: /~RESET~ -> Net-(R11-Pad2)
Routing:
- net Net-(R11-Pad2): track 0.00 -> 37.8 mm, vias 0 -> 3
- net /~RESET~: track 71.4 -> 54.9 mm, vias 5 -> 4
- net GND: track 7.96 -> 3.76 mm, vias 5 -> 4
- net +3V3: track 347.3 -> 345.0 mm
- net /SCL: track 41.2 -> 40.4 mm
- net Net-(M2-Pad3): track 53.1 -> 52.9 mm, vias 5 -> 4

Commit message: supervisor: use pick and place footprints
Problem: hand solder footprints may not be optimal for
pick and place assembly.

Switch to non-hand-solder variants.

Also, tweak silk for better readability in some areas.
Parts:
- C10, C11, C12, C13, C14, C15, C16, C17, C18, C2, C3, C4, C5, C6, C7, C8, C9: footprint Capacitor_SMD:C_0805_2012Metric_Pad1.18x1.45mm_HandSolder -> Capacitor_SMD:C_0805_2012Metric
- D1: footprint LED_SMD:LED_0805_2012Metric_Pad1.15x1.40mm_HandSolder -> LED_SMD:LED_0805_2012Metric
- R1, R10, R11, R13, R14, R15, R16, R2, R3, R4, R5, R6, R7, R8, R9: footprint Resistor_SMD:R_0805_2012Metric_Pad1.20x1.40mm_HandSolder -> Resistor_SMD:R_0805_2012Metric
- U2: footprint Package_TO_SOT_SMD:SOT-23-8_Handsoldering -> Package_TO_SOT_SMD:SOT-23-8
