File: hardware/cm4-compute/cm4-compute.kicad_pcb (KiCad board)
At the start: 2 copper layers, 160 x 100 mm, 1 part

Commit message: cm4-compute: add M.2 to board
Parts:
- added H1: MountingHole_Pad, MountingHole:MountingHole_2.2mm_M2_DIN965_Pad_TopBottom, F.Cu at (106.3, 134.6)
- added H2: MountingHole_Pad, MountingHole:MountingHole_2.2mm_M2_DIN965_Pad_TopBottom, F.Cu at (106.3, 114.6)
- added H3: MountingHole_Pad, MountingHole:MountingHole_2.2mm_M2_DIN965_Pad_TopBottom, F.Cu at (106.3, 96.6)
- added J1: M.2_Key_M_Socket_3_PCIe, 00_cm4-compute:Conn_TE-M.2-0.5-67P-doublesided, F.Cu at (106.3, 54.6)
- added R1: 10K, Resistor_SMD:R_0805_2012Metric_Pad1.20x1.40mm_HandSolder, F.Cu at (120.1, 49.3)
- moved Module1 42.9 mm to (124.4, 113.9)
Connections:
- net Net-(Module1-Pad101) renamed /cm4_highspeed/USB_OTG_ID
- net Net-(Module1-Pad103) renamed /cm4_highspeed/USB-
- net Net-(Module1-Pad105) renamed /cm4_highspeed/USB+
- net Net-(Module1-Pad78) renamed /cm4_gpio/GPIO_VREF
- Module1 pad 102: Net-(Module1-Pad102) -> /M.2 expansion/~PCIE_CLK_REQ~
- Module1 pad 107: Net-(Module1-Pad107) -> GND
- Module1 pad 108: Net-(Module1-Pad108) -> GND
- Module1 pad 109: Net-(Module1-Pad109) -> /M.2 expansion/~PCIE_RST~
- Module1 pad 110: Net-(Module1-Pad110) -> /M.2 expansion/PCIE_CLK+
- Module1 pad 112: Net-(Module1-Pad112) -> /M.2 expansion/PCIE_CLK-
- Module1 pad 113: Net-(Module1-Pad113) -> GND
- Module1 pad 114: Net-(Module1-Pad114) -> GND
- Module1 pad 116: Net-(Module1-Pad116) -> /M.2 expansion/PCIE_RX+
- Module1 pad 118: (no net) -> /M.2 expansion/PCIE_RX-
- Module1 pad 119: Net-(Module1-Pad119) -> GND
- Module1 pad 120: Net-(Module1-Pad120) -> GND
- Module1 pad 122: Net-(Module1-Pad122) -> /M.2 expansion/PCIE_TX+
- Module1 pad 124: Net-(Module1-Pad124) -> /M.2 expansion/PCIE_TX-
- Module1 pad 125: Net-(Module1-Pad125) -> GND
- Module1 pad 126: Net-(Module1-Pad126) -> GND
- Module1 pad 131: Net-(Module1-Pad131) -> GND
- Module1 pad 132: Net-(Module1-Pad132) -> GND
- Module1 pad 137: Net-(Module1-Pad137) -> GND
- Module1 pad 138: Net-(Module1-Pad138) -> GND
- Module1 pad 144: Net-(Module1-Pad144) -> GND
- Module1 pad 150: Net-(Module1-Pad150) -> GND
- Module1 pad 155: Net-(Module1-Pad155) -> GND
- Module1 pad 156: Net-(Module1-Pad156) -> GND
- Module1 pad 161: Net-(Module1-Pad161) -> GND
- Module1 pad 162: Net-(Module1-Pad162) -> GND
- Module1 pad 167: Net-(Module1-Pad167) -> GND
- Module1 pad 168: Net-(Module1-Pad168) -> GND
- Module1 pad 173: Net-(Module1-Pad173) -> GND
- Module1 pad 174: Net-(Module1-Pad174) -> GND
- Module1 pad 179: Net-(Module1-Pad179) -> GND
- Module1 pad 180: Net-(Module1-Pad180) -> GND
- Module1 pad 185: Net-(Module1-Pad185) -> GND
- Module1 pad 186: Net-(Module1-Pad186) -> GND
- Module1 pad 191: Net-(Module1-Pad191) -> GND
- Module1 pad 192: Net-(Module1-Pad192) -> GND
- Module1 pad 197: Net-(Module1-Pad197) -> GND
- Module1 pad 198: Net-(Module1-Pad198) -> GND
