File: hardware/kludge_panel_4hp/frontpanel_3u_4hp_holes.kicad_pcb (KiCad board)
At the start: 2 copper layers, 20 x 128.4 mm, 6 parts

Commit message: hardware: change kludge panel holes for Elma
Problem: kludge front panel starting point is for the Reichelt
BGT VS1, but we have Elma S-216-13 eurocard hardware on hand.

Adjust position of two mounting holes in vertical direction so
that they are 13.25mm from the top and bottom edge.  Adjust the
horizontal position of one hole so that it matches the lever
mounting bracket.  Replace the handle hole with a slot for the
lever, which also serves as a handle.

Goal will be to replace Elma hardware with cheap DIY 3D printed
alternative but use the same hole pattern.

Add a README referencing Marten's work.
Parts:
- removed G***: LOGO, logo:marten-logo_5x5_Fcu
Routing:
- net GND: vias 3 -> 0
- added copper zone on F.Cu, net (none)
- removed copper zone on B.Cu, net GND
- removed copper zone on F.Cu, net GND
Other:
- outline, holes or cut-outs redrawn
- board text removed: "4HP"
