File: hardware/kludge/kludge.kicad_pcb (KiCad board)
At the start: 2 copper layers, 160 x 100 mm, 2056 parts

Commit message: hardware/kludge: fix missing 5V connection
Problem: PTC output is not connected to filter cap (+).

Add missing trace.

Also, change the disjoint 5V net to VCC, matching silk label.
Connections:
- REF** pad : 5V -> VCC (x20)
Routing:
- net VCC: track 0.00 -> 243.8 mm
- net 5V: track 249.4 -> 11.1 mm
Changed lines of the file:
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@@
   (net 2 "5V")
   (net 3 "BUS5V")
+  (net 4 "VCC")
   (footprint "lib:pingrid1x1_2.54" (layer "F.Cu")
     (at 191.81 81.03)
@@
     )
     (pad "" thru_hole circle (at 0 0) (size 1.7 1.7) (drill 1) (layers *.Cu *.Mask)
-      (net 2 "5V"))
+      (net 4 "VCC"))
   )
   (footprint "lib:pingrid1x1_2.54" (layer "F.Cu")
@@
     )
     (pad "" thru_hole circle (at 0 0) (size 1.7 1.7) (drill 1) (layers *.Cu *.Mask)
-      (net 2 "5V"))
+      (net 4 "VCC"))
   )
   (footprint "lib:pingrid1x1_2.54" (layer "F.Cu")
@@
     )
     (pad "" thru_hole circle (at 0 0) (size 1.7 1.7) (drill 1) (layers *.Cu *.Mask)
-      (net 2 "5V"))
+      (net 4 "VCC"))
   )
   (footprint "lib:pingrid1x1_2.54" (layer "F.Cu")
@@
     )
     (pad "" thru_hole circle (at 0 0) (size 1.7 1.7) (drill 1) (layers *.Cu *.Mask)
-      (net 2 "5V"))
+      (net 4 "VCC"))
   )
   (footprint "lib:pingrid1x1_2.54" (layer "F.Cu")
@@
     )
     (pad "" thru_hole circle (at 0 0) (size 1.7 1.7) (drill 1) (layers *.Cu *.Mask)
-      (net 2 "5V"))
+      (net 4 "VCC"))
   )
   (footprint "lib:pingrid1x1_2.54" (layer "F.Cu")
@@
     )
     (pad "" thru_hole circle (at 0 0) (size 1.7 1.7) (drill 1) (layers *.Cu *.Mask)
-      (net 2 "5V"))
+      (net 4 "VCC"))
   )
   (footprint "lib:pingrid1x1_2.54" (layer "F.Cu")
@@
     )
     (pad "" thru_hole circle (at 0 0) (size 1.7 1.7) (drill 1) (layers *.Cu *.Mask)
-      (net 2 "5V"))
+      (net 4 "VCC"))
   )
   (footprint "lib:pingrid1x1_2.54" (layer "F.Cu")
@@
     )
     (pad "" thru_hole circle (at 0 0) (size 1.7 1.7) (drill 1) (layers *.Cu *.Mask)
-      (net 2 "5V"))
+      (net 4 "VCC"))
   )
   (footprint "lib:pingrid1x1_2.54" (layer "F.Cu")
@@
     )
     (pad "" thru_hole circle (at 0 0) (size 1.7 1.7) (drill 1) (layers *.Cu *.Mask)
-      (net 2 "5V"))
+      (net 4 "VCC"))
   )
   (footprint "lib:pingrid1x1_2.54" (layer "F.Cu")
@@
     )
     (pad "" thru_hole circle (at 0 0) (size 1.7 1.7) (drill 1) (layers *.Cu *.Mask)
-      (net 2 "5V"))
+      (net 4 "VCC"))
   )
   (footprint "lib:pingrid1x1_2.54" (layer "F.Cu")
@@
     )
     (pad "" thru_hole circle (at 0 0) (size 1.7 1.7) (drill 1) (layers *.Cu *.Mask)
-      (net 2 "5V"))
+      (net 4 "VCC"))
   )
   (footprint "lib:pingrid1x1_2.54" (layer "F.Cu")
@@
     (fp_line (start 1 -1) (end -1 -1) (layer "B.CrtYd") (width 0.05))
     (pad "" smd rect (at 0 0 180) (size 1 1) (layers "B.Cu" "B.Mask")
-      (net 2 "5V"))
+      (net 4 "VCC"))
   )
   (footprint "TestPoint:TestPoint_Pad_1.0x1.0mm" (layer "B.Cu")
@@
     (fp_line (start -1 1) (end 1 1) (layer "B.CrtYd") (width 0.05))
     (pad "" smd rect (at 0 0 180) (size 1 1) (layers "B.Cu" "B.Mask")
-      (net 2 "5V"))
+      (net 4 "VCC"))
   )
   (footprint "TestPoint:TestPoint_Pad_1.0x1.0mm" (layer "B.Cu")
@@
     (fp_line (start -1 1) (end 1 1) (layer "B.CrtYd") (width 0.05))
     (pad "" smd rect (at 0 0 180) (size 1 1) (layers "B.Cu" "B.Mask")
-      (net 2 "5V"))
+      (net 4 "VCC"))
   )
   (footprint "TestPoint:TestPoint_Pad_1.0x1.0mm" (layer "B.Cu")
@@
     (fp_line (start 1 -1) (end -1 -1) (layer "B.CrtYd") (width 0.05))
     (pad "" smd rect (at 0 0 180) (size 1 1) (layers "B.Cu" "B.Mask")
-      (net 2 "5V"))
+      (net 4 "VCC"))
   )
   (footprint "TestPoint:TestPoint_Pad_1.0x1.0mm" (layer "B.Cu")
@@
     (fp_line (start 1 -1) (end -1 -1) (layer "B.CrtYd") (width 0.05))
     (pad "" smd rect (at 0 0 180) (size 1 1) (layers "B.Cu" "B.Mask")
-      (net 2 "5V"))
+      (net 4 "VCC"))
   )
   (footprint "TestPoint:TestPoint_Pad_1.0x1.0mm" (layer "B.Cu")
@@
     (fp_line (start 1 -1) (end -1 -1) (layer "B.CrtYd") (width 0.05))
     (pad "" smd rect (at 0 0 180) (size 1 1) (layers "B.Cu" "B.Mask")
-      (net 2 "5V"))
+      (net 4 "VCC"))
   )
   (footprint "TestPoint:TestPoint_Pad_1.0x1.0mm" (layer "B.Cu")
@@
     (fp_line (start -1 1) (end -1 -1) (layer "B.CrtYd") (width 0.05))
     (pad "" smd rect (at 0 0 180) (size 1 1) (layers "B.Cu" "B.Mask")
-      (net 2 "5V"))
+      (net 4 "VCC"))
   )
   (footprint "TestPoint:TestPoint_Pad_1.0x1.0mm" (layer "B.Cu")
@@
     (fp_line (start -1 1) (end -1 -1) (layer "B.CrtYd") (width 0.05))
     (pad "" smd rect (at 0 0 180) (size 1 1) (layers "B.Cu" "B.Mask")
-      (net 2 "5V"))
+      (net 4 "VCC"))
   )
   (footprint "TestPoint:TestPoint_Pad_1.0x1.0mm" (layer "B.Cu")
@@
     (fp_line (start -1 1) (end 1 1) (layer "B.CrtYd") (width 0.05))
     (pad "" smd rect (at 0 0 180) (size 1 1) (layers "B.Cu" "B.Mask")
-      (net 2 "5V"))
+      (net 4 "VCC"))
   )
   (footprint "TestPoint:TestPoint_Pad_1.0x1.0mm" (layer "B.Cu")
@@
   (segment (start 204.51 58.17) (end 212.13 58.17) (width 2) (layer "B.Cu") (net 1))
   (segment (start 204.51 131.83) (end 212.13 131.83) (width 2) (layer "B.Cu") (net 1))
+  (segment (start 199.43 50.55) (end 201.97 50.55) (width 2) (layer "F.Cu") (net 2))
   (segment (start 191.81 50.55) (end 195.78 50.55) (width 2) (layer "F.Cu") (net 2))
-  (segment (start 189.27 50.55) (end 67.35 50.55) (width 2) (layer "F.Cu") (net 2))
+  (segment (start 198.32 51.66) (end 199.43 50.55) (width 2) (layer "F.Cu") (net 2))
   (segment (start 195.78 50.55) (end 196.89 51.66) (width 2) (layer "F.Cu") (net 2))
-  (segment (start 181.65 50.55) (end 189.27 50.55) (width 2) (layer "B.Cu") (net 2))
-  (segment (start 181.65 50.55) (end 67.35 50.55) (width 2) (layer "B.Cu") (net 2))
+  (segment (start 196.89 51.66) (end 198.32 51.66) (width 2) (layer "F.Cu") (net 2))
   (segment (start 204.51 55.63) (end 209.59 55.63) (width 2) (layer "F.Cu") (net 3))
   (segment (start 201.97 55.63) (end 204.51 55.63) (width 2) (layer "F.Cu") (net 3))
@@
   (segment (start 201.97 134.37) (end 201.97 55.63) (width 2) (layer "F.Cu") (net 3))
   (segment (start 204.51 134.37) (end 209.59 134.37) (width 2) (layer "B.Cu") (net 3))
+  (segment (start 189.27 50.55) (end 67.35 50.55) (width 2) (layer "F.Cu") (net 4))
+  (segment (start 181.65 50.55) (end 189.27 50.55) (width 2) (layer "B.Cu") (net 4))
+  (segment (start 181.65 50.55) (end 67.35 50.55) (width 2) (layer "B.Cu") (net 4))
   (zone (net 0) (net_name "") (layer "F.Cu") (hatch edge 0.508)
     (connect_pads (clearance 0))
     (min_thickness 0.254)
-    (keepout (tracks allowed) (vias allowed) (pads allowed ) (copperpour not_allowed) (footprints allowed))
+    (keepout (tracks allowed) (vias allowed) (pads allowed) (copperpour not_allowed) (footprints allowed))
     (fill (thermal_gap 0.508) (thermal_bridge_width 0.508))
     (polygon
@@
     (connect_pads (clearance 0))
     (min_thickness 0.254)
-    (keepout (tracks not_allowed) (vias not_allowed) (pads not_allowed ) (copperpour allowed) (footprints not_allowed))
+    (keepout (tracks not_allowed) (vias not_allowed) (pads not_allowed) (copperpour allowed) (footprints not_allowed))
     (fill (thermal_gap 0.508) (thermal_bridge_width 0.508))
     (polygon
@@
     (connect_pads (clearance 0))
     (min_thickness 0.254)
-    (keepout (tracks allowed) (vias allowed) (pads allowed ) (copperpour not_allowed) (footprints allowed))
+    (keepout (tracks allowed) (vias allowed) (pads allowed) (copperpour not_allowed) (footprints allowed))
     (fill (thermal_gap 0.508) (thermal_bridge_width 0.508))
     (polygon
@@
     (connect_pads (clearance 0))
     (min_thickness 0.254)
-    (keepout (tracks not_allowed) (vias not_allowed) (pads not_allowed ) (copperpour allowed) (footprints not_allowed))
+    (keepout (tracks not_allowed) (vias not_allowed) (pads not_allowed) (copperpour allowed) (footprints not_allowed))
     (fill (thermal_gap 0.508) (thermal_bridge_width 0.508))
     (polygon
@@
     (connect_pads (clearance 0))
     (min_thickness 0.254)
-    (keepout (tracks allowed) (vias allowed) (pads allowed ) (copperpour not_allowed) (footprints allowed))
+    (keepout (tracks allowed) (vias allowed) (pads allowed) (copperpour not_allowed) (footprints allowed))
     (fill (thermal_gap 0.508) (thermal_bridge_width 0.508))
     (polygon
