File: hardware/pi5_panel_4hp/panel.kicad_pcb (KiCad board)
At the start: 2 copper layers, 20 x 128.4 mm, 5 parts

Commit message: pi5_panel_4hp: finalize layout
Add pi5face footprint and position it on the panel.
This is going to pcbway.
Parts:
- added REF**: piface, Library:pi5face, B.Cu at (97.5, 144.3)
Other:
- board text added: "Notes: 4 HP 20.32mm, nominal 20.0mm, this 19.98mm"
Changed lines of the file:
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@@
     (thickness 1.6)
   )
-  (paper "A4")
+  (paper "USLetter")
   (title_block
     (title "Eurocard faceplate for Raspberry Pi 5 and Elma extractor")
@@
       (plot_on_all_layers_selection 0x0000000_00000000)
       (disableapertmacros false)
-      (usegerberextensions true)
+      (usegerberextensions false)
       (usegerberattributes false)
       (usegerberadvancedattributes false)
@@
       (psa4output false)
       (plotreference true)
-      (plotvalue true)
+      (plotvalue false)
       (plotinvisibletext false)
       (sketchpadsonfab false)
-      (subtractmaskfromsilk false)
+      (subtractmaskfromsilk true)
       (outputformat 1)
       (mirror false)
@@
     (pad "" np_thru_hole oval (at 0 0 180) (size 5.9 3.3) (drill oval 5.9 3.3) (layers "F.Cu"))
   )
+  (footprint "Library:pi5face" (layer "B.Cu")
+    (at 97.4512 144.3416 90)
+    (fp_text reference "REF**" (at -6.75 7.08 270 unlocked) (layer "Cmts.User") hide
+        (effects (font (size 1 1) (thickness 0.15)))
+    )
+    (fp_text value "piface" (at -6.94 2.13 270 unlocked) (layer "Cmts.User") hide
+        (effects (font (size 1 1) (thickness 0.15)))
+    )
+    (fp_text user "${REFERENCE}" (at -6.92 8.35 270 unlocked) (layer "Cmts.User") hide
+        (effects (font (size 1 1) (thickness 0.15)))
+    )
+    (fp_rect (start 14.05 12.85) (end 14.05 12.96)
+      (stroke (width 0.12) (type solid)) (fill none) (layer "B.SilkS"))
+    (fp_rect (start 6.75 13) (end 24.5 0)
+      (stroke (width 0.12) (type solid)) (fill none) (layer "Edge.Cuts"))
+    (fp_rect (start 27.75 0) (end 41.5 8)
+      (stroke (width 0.12) (type solid)) (fill none) (layer "Edge.Cuts"))
+    (fp_rect (start 45.5 0) (end 59.25 8)
+      (stroke (width 0.12) (type solid)) (fill none) (layer "Edge.Cuts"))
+    (fp_rect (start 63.25 0) (end 79.25 13.5)
+      (stroke (width 0.12) (type solid)) (fill none) (layer "Edge.Cuts"))
+    (fp_circle (center 3.75 2.54) (end 5.25 2.54)
+      (stroke (width 0.12) (type solid)) (fill none) (layer "Edge.Cuts"))
+    (fp_circle (center 3.75 7.62) (end 5.25 7.62)
+      (stroke (width 0.12) (type solid)) (fill none) (layer "Edge.Cuts"))
+  )
   (gr_line (start 93.5812 167.3696) (end 93.5812 38.9696)
     (stroke (width 0.05) (type solid)) (layer "Edge.Cuts"))
@@
   (gr_circle (center 106.1112 154.1196) (end 104.6112 154.1196)
     (stroke (width 0.2) (type solid)) (fill none) (layer "Edge.Cuts"))
+  (gr_text "Notes:\n4 HP 20.32mm, nominal 20.0mm, this 19.98mm\n" (at 147.14 35.566) (layer "Dwgs.User")
+    (effects (font (size 1.5 1.5) (thickness 0.3) bold) (justify left bottom))
+  )
   (zone (net 0) (net_name "") (layer "F.Cu") (hatch edge 0.508)
     (connect_pads (clearance 0.508))
