File: hardware/pi5_adapter/pi5_adapter.kicad_sch (KiCad schematic)
At the start: 17 parts, among them J1 GPIO, J2 GPIO, J3 Conn_01x05, J5 Conn_02x05_Odd_Even, U1 CAT24C256, U2 TPS27081ADDCR

Commit message: pi5_adapter: update for kicad 8.0.2
Problem: got an ERC/DRC errors on out of date symbols and
footprints after upgrading to kicad 8.0.2.

Update symbols and footprints.
Parts:
- C1, C2: footprint Capacitor_SMD:C_0603_1608Metric -> (none)
- J1, J2: footprint Connector_PinSocket_2.54mm:PinSocket_2x20_P2.54mm_Vertical -> (none)
- J3: footprint lib:PinSocket_1x05_P2.54mm_Vertical -> (none)
- J5: footprint Connector_PinSocket_2.54mm:PinSocket_2x05_P2.54mm_Vertical -> (none)
- JP1, JP2: footprint Jumper:SolderJumper-2_P1.3mm_Open_RoundedPad1.0x1.5mm -> (none); now left out of the parts list
- R1, R2, R3, R4, R5, R6, R7: footprint Resistor_SMD:R_0603_1608Metric -> (none)
- U1: footprint Package_SO:SOIC-8_3.9x4.9mm_P1.27mm -> (none)
Changed lines of the file:
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@@
 			)
 		)
-		(property "Footprint" "Connector_PinSocket_2.54mm:PinSocket_2x20_P2.54mm_Vertical"
-			(at -58.42 86.36 0)
+		(property "Footprint" ""
+			(at 64.77 62.23 0)
 			(effects
 				(font
@@
 		)
 		(property "Datasheet" "~"
-			(at -58.42 86.36 0)
+			(at 64.77 62.23 0)
 			(effects
 				(font
@@
 		(at 171.45 134.62 0)
 		(unit 1)
-		(exclude_from_sim no)
-		(in_bom yes)
+		(exclude_from_sim yes)
+		(in_bom no)
 		(on_board yes)
 		(dnp no)
@@
 			)
 		)
-		(property "Footprint" "Jumper:SolderJumper-2_P1.3mm_Open_RoundedPad1.0x1.5mm"
+		(property "Footprint" ""
 			(at 171.45 134.62 0)
 			(effects
@@
 			)
 		)
-		(property "Footprint" "Capacitor_SMD:C_0603_1608Metric"
+		(property "Footprint" ""
 			(at 67.31 177.8 0)
 			(effects
@@
 			)
 		)
-		(property "Footprint" "Capacitor_SMD:C_0603_1608Metric"
+		(property "Footprint" ""
 			(at 168.6052 147.32 0)
 			(effects
@@
 			)
 		)
-		(property "Footprint" "Resistor_SMD:R_0603_1608Metric"
+		(property "Footprint" ""
 			(at 146.558 140.97 90)
 			(effects
@@
 		(fields_autoplaced yes)
 		(property "Reference" "J3"
-			(at 69.85 105.41 0)
+			(at 69.85 105.4099 0)
 			(effects
 				(font
@@
 			)
 		)
-		(property "Footprint" "lib:PinSocket_1x05_P2.54mm_Vertical"
+		(property "Footprint" ""
 			(at 67.31 105.41 0)
 			(effects
@@
 			)
 		)
-		(property "Footprint" "Resistor_SMD:R_0603_1608Metric"
+		(property "Footprint" ""
 			(at 93.98 170.18 0)
 			(effects
@@
 			)
 		)
-		(property "Footprint" "Resistor_SMD:R_0603_1608Metric"
+		(property "Footprint" ""
 			(at 135.382 140.97 90)
 			(effects
@@
 		(at 96.52 180.34 0)
 		(unit 1)
-		(exclude_from_sim no)
-		(in_bom yes)
+		(exclude_from_sim yes)
+		(in_bom no)
 		(on_board yes)
 		(dnp no)
@@
 			)
 		)
-		(property "Footprint" "Jumper:SolderJumper-2_P1.3mm_Open_RoundedPad1.0x1.5mm"
+		(property "Footprint" ""
 			(at 96.52 180.34 0)
 			(effects
@@
 			)
 		)
-		(property "Footprint" "Resistor_SMD:R_0603_1608Metric"
+		(property "Footprint" ""
 			(at 131.318 140.97 90)
 			(effects
@@
 			)
 		)
-		(property "Footprint" "Connector_PinSocket_2.54mm:PinSocket_2x20_P2.54mm_Vertical"
-			(at 22.86 86.36 0)
+		(property "Footprint" ""
+			(at 146.05 62.23 0)
 			(effects
 				(font
@@
 		)
 		(property "Datasheet" "~"
-			(at 22.86 86.36 0)
+			(at 146.05 62.23 0)
 			(effects
 				(font
@@
 			)
 		)
-		(property "Footprint" "Resistor_SMD:R_0603_1608Metric"
+		(property "Footprint" ""
 			(at 101.6 170.18 0)
 			(effects
@@
 			)
 		)
-		(property "Footprint" "Resistor_SMD:R_0603_1608Metric"
+		(property "Footprint" ""
 			(at 67.31 126.238 90)
 			(effects
@@
 			)
 		)
-		(property "Footprint" "Package_SO:SOIC-8_3.9x4.9mm_P1.27mm"
+		(property "Footprint" ""
 			(at 81.28 177.8 0)
 			(effects
@@
 		)
 		(property "Description" "IC LOAD SW HIGH SIDE 6SOT"
-			(at 160.02 124.46 0)
-			(effects
-				(font
-					(size 1.524 1.524)
-				)
-				(justify left)
+			(at 154.94 149.86 0)
+			(effects
+				(font
+					(size 1.27 1.27)
+				)
 				(hide yes)
 			)
@@
 		)
 		(property "Value" "PWR_FLAG"
-			(at 160.02 88.9 90)
+			(at 160.02 88.8999 90)
 			(effects
 				(font
@@
 		)
 		(property "Value" "PWR_FLAG"
-			(at 50.546 39.37 90)
+			(at 50.8 39.3699 90)
 			(effects
 				(font
@@
 		)
 		(property "Value" "PWR_FLAG"
-			(at 162.56 34.925 0)
+			(at 162.56 34.29 0)
 			(effects
 				(font
@@
 			)
 		)
-		(property "Footprint" "Connector_PinSocket_2.54mm:PinSocket_2x05_P2.54mm_Vertical"
+		(property "Footprint" ""
 			(at 146.05 105.41 0)
 			(effects
@@
 			)
 		)
-		(property "Footprint" "Resistor_SMD:R_0603_1608Metric"
+		(property "Footprint" ""
 			(at 67.31 132.588 90)
 			(effects
