File: hardware/pi5_adapter/pi5_adapter.kicad_pcb (KiCad board)
At the start: 2 copper layers, 65 x 74 mm, 15 parts, among them J1 GPIO, J2 GPIO, U1 CAT24C256

Commit message: pi5_adapter: add power switch
Problem: the Pi 5 and Pi 3B (not plus) do not expose PMIC
GLOBAL_EN line, thus cannot be controlled with the pi-carrier.
Also, on Pi4 and Pi 3B+ that do expose the PMIC, bodge wires
direct from pi to pi-carrier are inconvenient as it prevents
removal of the pi.

Add the 3A high side load switch that was eliminated from the
pi-carrier.  The power circuit emulates the pi PMIC lines on a
JST SH (1mm) 3-pin connector.  That is,

- GLOBAL_EN (pulled to 5V on the board) turns the switch on when
  floating, off when grounded.

- RUN_PG is pulled high by the pi 3V3 power output

The new components can optionally be left unpopulated and the
Pi GLOBAL_EN and RUN_PG can be soldered to pads on the baord
and brought out on the JST connector.  A bypass jumper must also
be bridged in this mode.
Parts:
- removed C1: 100n, Capacitor_SMD:C_0603_1608Metric
- removed the MH1 at (103.5, 40.5)
- added C2: 1uF, Capacitor_SMD:C_0603_1608Metric, F.Cu at (101.6, 39.2)
- added J3: Conn_01x03_MountingPin, Connector_JST:JST_SH_BM03B-SRSS-TB_1x03-1MP_P1.00mm_Vertical, B.Cu at (102.8, 89.1)
- added J4: Conn_01x02_Pin, Connector_Wire:SolderWire-0.25sqmm_1x02_P4.2mm_D0.65mm_OD1.7mm, F.Cu at (113.4, 94.7)
- added JP2: BYPASS, Jumper:SolderJumper-2_P1.3mm_Open_RoundedPad1.0x1.5mm, F.Cu at (104.9, 37.6)
- added R3: 10K, Resistor_SMD:R_0603_1608Metric, F.Cu at (101.6, 43.5)
- added R4: 10K, Resistor_SMD:R_0603_1608Metric, F.Cu at (101.6, 41.8)
- added R5: 10K, Resistor_SMD:R_0603_1608Metric, F.Cu at (122.2, 93.9)
- added U2: TPS27081ADDCR, Package_TO_SOT_SMD:TSOT-23-6, F.Cu at (105.3, 42.4)
Connections:
- J2 pad 2: +5V -> /5V_EXTERNAL
- J2 pad 4: +5V -> /5V_EXTERNAL
Routing:
- net /GLOBAL_EN: track 0.00 -> 64.5 mm, vias 0 -> 1
- net /RUN_PG: track 0.00 -> 25.3 mm
- net /5V_EXTERNAL: track 0.00 -> 20.1 mm
- net GND: track 36.9 -> 40.0 mm, vias 0 -> 1
- net +3.3V: track 147.8 -> 145.8 mm
- net Net-(U2-R1/C1): track 0.00 -> 1.83 mm
- net +5V: track 17.2 -> 15.5 mm
Other:
- board text added: "Bypass"
- board text added: "GLOBAL_EN"
- board text added: "ID_WP"
- board text added: "RUN_PG"

Commit message: pi5_adapter: move J3
Problem: J3 interferes with heatsink on Pi 5 cooler.

Relocate to other side of the same board edge where it should
not interfere.
Parts:
- moved J3 34.7 mm to (102.6, 54.4)
Routing:
- net /RUN_PG: track 25.3 -> 59.9 mm
- net GND: track 40.0 -> 38.4 mm
Changed lines of the file:
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@@
   )
   (footprint "Connector_JST:JST_SH_BM03B-SRSS-TB_1x03-1MP_P1.00mm_Vertical" (layer "B.Cu")
-    (at 102.8448 89.078 -90)
+    (at 102.5716 54.3702 -90)
     (descr "JST SH series connector, BM03B-SRSS-TB (http://www.jst-mfg.com/product/pdf/eng/eSH.pdf), generated with kicad-footprint-generator")
     (tags "connector JST SH side entry")
@@
     (property "ki_keywords" "connector")
     (attr smd)
-    (fp_text reference "J3" (at -4.1656 -0.1016 -180) (layer "B.SilkS")
+    (fp_text reference "J3" (at 4.304 0.0316 -180) (layer "B.SilkS")
         (effects (font (size 1 1) (thickness 0.15)) (justify mirror))
     )
@@
   (segment (start 123.61 36.07) (end 124.704 34.976) (width 0.5) (layer "F.Cu") (net 1))
   (segment (start 131.23 36.07) (end 132.324 34.976) (width 0.5) (layer "F.Cu") (net 1))
-  (via (at 104.9784 91.3386) (size 0.9) (drill 0.6) (layers "F.Cu" "B.Cu") (net 1))
+  (via (at 104.5466 57.074) (size 0.9) (drill 0.6) (layers "F.Cu" "B.Cu") (free) (net 1))
   (segment (start 130.099 34.939) (end 130.099 34.595) (width 0.5) (layer "B.Cu") (net 1))
   (segment (start 138.85 38.61) (end 140.071 37.389) (width 0.5) (layer "B.Cu") (net 1))
@@
   (segment (start 131.23 46.23) (end 130.136 45.136) (width 0.5) (layer "B.Cu") (net 1))
   (segment (start 114.478 35.042) (end 114.478 34.849) (width 0.5) (layer "B.Cu") (net 1))
-  (segment (start 104.1698 90.078) (end 104.1698 90.53) (width 0.2) (layer "B.Cu") (net 1))
   (segment (start 118.53 48.77) (end 119.878 47.422) (width 0.5) (layer "B.Cu") (net 1))
   (segment (start 143.93 36.07) (end 145.085 34.915) (width 0.5) (layer "B.Cu") (net 1))
@@
   (segment (start 148.006 35.066) (end 148.006 34.849) (width 0.5) (layer "B.Cu") (net 1))
   (segment (start 123.61 45.529) (end 124.257 44.882) (width 0.5) (layer "B.Cu") (net 1))
-  (segment (start 104.1698 90.53) (end 104.9784 91.3386) (width 0.2) (layer "B.Cu") (net 1))
   (segment (start 147.752 44.972) (end 147.752 44.882) (width 0.5) (layer "B.Cu") (net 1))
   (segment (start 145.085 34.915) (end 145.085 34.849) (width 0.5) (layer "B.Cu") (net 1))
@@
   (segment (start 122.1986 94.7168) (end 122.225 94.6904) (width 0.2) (layer "F.Cu") (net 37))
   (segment (start 117.653 94.6914) (end 117.6276 94.7168) (width 0.2) (layer "F.Cu") (net 37))
-  (segment (start 116.383 95.9614) (end 117.6276 94.7168) (width 0.2) (layer "B.Cu") (net 37))
-  (segment (start 108.4836 95.9614) (end 116.383 95.9614) (width 0.2) (layer "B.Cu") (net 37))
-  (segment (start 104.1698 88.078) (end 103.394801 88.078) (width 0.2) (layer "B.Cu") (net 37))
-  (segment (start 103.0948 90.5726) (end 108.4836 95.9614) (width 0.2) (layer "B.Cu") (net 37))
-  (segment (start 103.0948 88.378001) (end 103.0948 90.5726) (width 0.2) (layer "B.Cu") (net 37))
-  (segment (start 103.394801 88.078) (end 103.0948 88.378001) (width 0.2) (layer "B.Cu") (net 37))
+  (segment (start 102.8216 57.292) (end 102.8216 53.670201) (width 0.2) (layer "B.Cu") (net 37))
+  (segment (start 106.628229 93.688) (end 105.3976 92.457371) (width 0.2) (layer "B.Cu") (net 37))
+  (segment (start 110.264056 93.688) (end 106.628229 93.688) (width 0.2) (layer "B.Cu") (net 37))
+  (segment (start 117.6276 94.7168) (end 116.383 95.9614) (width 0.2) (layer "B.Cu") (net 37))
+  (segment (start 116.383 95.9614) (end 112.537456 95.9614) (width 0.2) (layer "B.Cu") (net 37))
+  (segment (start 105.3976 92.457371) (end 105.3976 59.868) (width 0.2) (layer "B.Cu") (net 37))
+  (segment (start 102.8216 53.670201) (end 103.121601 53.3702) (width 0.2) (layer "B.Cu") (net 37))
+  (segment (start 105.3976 59.868) (end 102.8216 57.292) (width 0.2) (layer "B.Cu") (net 37))
+  (segment (start 103.121601 53.3702) (end 103.8966 53.3702) (width 0.2) (layer "B.Cu") (net 37))
+  (segment (start 112.537456 95.9614) (end 110.264056 93.688) (width 0.2) (layer "B.Cu") (net 37))
   (segment (start 104.0192 43.485) (end 104.1258 43.3784) (width 0.2) (layer "F.Cu") (net 38))
   (segment (start 102.4374 43.485) (end 104.0192 43.485) (width 0.2) (layer "F.Cu") (net 38))
@@
   (segment (start 105.3086 42.948701) (end 105.3086 44.501) (width 0.2) (layer "F.Cu") (net 39))
   (via (at 105.3086 44.501) (size 0.9) (drill 0.6) (layers "F.Cu" "B.Cu") (net 39))
-  (segment (start 104.1698 89.078) (end 104.944799 89.078) (width 0.2) (layer "B.Cu") (net 39))
+  (segment (start 106.52 49.004314) (end 106.52 45.7124) (width 0.2) (layer "B.Cu") (net 39))
+  (segment (start 106.793915 93.288) (end 105.7976 92.291686) (width 0.2) (layer "B.Cu") (net 39))
+  (segment (start 105.7976 53.4926) (end 105.7976 49.726714) (width 0.2) (layer "B.Cu") (net 39))
+  (segment (start 113.4276 94.7168) (end 111.9988 93.288) (width 0.2) (layer "B.Cu") (net 39))
+  (segment (start 104.92 54.3702) (end 105.7976 53.4926) (width 0.2) (layer "B.Cu") (net 39))
+  (segment (start 111.9988 93.288) (end 106.793915 93.288) (width 0.2) (layer "B.Cu") (net 39))
+  (segment (start 105.7976 92.291686) (end 105.7976 53.4926) (width 0.2) (layer "B.Cu") (net 39))
   (segment (start 106.52 45.7124) (end 105.3086 44.501) (width 0.2) (layer "B.Cu") (net 39))
-  (segment (start 106.793915 93.288) (end 111.9988 93.288) (width 0.2) (layer "B.Cu") (net 39))
-  (segment (start 104.944799 89.078) (end 105.7976 89.930801) (width 0.2) (layer "B.Cu") (net 39))
-  (segment (start 106.52 49.004314) (end 106.52 45.7124) (width 0.2) (layer "B.Cu") (net 39))
-  (segment (start 111.9988 93.288) (end 113.4276 94.7168) (width 0.2) (layer "B.Cu") (net 39))
+  (segment (start 103.8966 54.3702) (end 104.92 54.3702) (width 0.2) (layer "B.Cu") (net 39))
   (segment (start 105.7976 49.726714) (end 106.52 49.004314) (width 0.2) (layer "B.Cu") (net 39))
-  (segment (start 105.7976 89.930801) (end 105.7976 92.291686) (width 0.2) (layer "B.Cu") (net 39))
-  (segment (start 105.7976 92.291686) (end 106.793915 93.288) (width 0.2) (layer "B.Cu") (net 39))
-  (segment (start 104.1698 89.078) (end 105.1562 89.078) (width 0.2) (layer "B.Cu") (net 39))
-  (segment (start 105.7976 88.4366) (end 105.7976 49.726714) (width 0.2) (layer "B.Cu") (net 39))
-  (segment (start 105.1562 89.078) (end 105.7976 88.4366) (width 0.2) (layer "B.Cu") (net 39))
   (zone (net 1) (net_name "GND") (layer "F.Cu") (hatch edge 0.5)
     (connect_pads (clearance 0))

Commit message: pi5_adapter: add 10-pin board to board connector
Problem: the JST jumpers for power are lame.

Add a board to board connector.
Parts:
- removed J4: Conn_01x02_Pin, Connector_Wire:SolderWire-0.25sqmm_1x02_P4.2mm_D0.65mm_OD1.7mm
- added C1: 100n, Capacitor_SMD:C_0603_1608Metric, F.Cu at (162.5, 57.1)
- added J5: Conn_02x05_Odd_Even, Connector_PinSocket_2.54mm:PinSocket_2x05_P2.54mm_Vertical, B.Cu at (146.5, 105.7)
- added R6: 0R, Resistor_SMD:R_0603_1608Metric, F.Cu at (154.2, 94.7)
- added R7: 0R, Resistor_SMD:R_0603_1608Metric, F.Cu at (156.6, 94.7)
- added REF**: OSHW-Logo2_7.3x6mm_SilkScreen, Symbol:OSHW-Logo2_7.3x6mm_SilkScreen, F.Cu at (161.7, 80.7)
- J3: value Conn_01x03_MountingPin -> Conn_01x05; footprint Connector_JST:JST_SH_BM03B-SRSS-TB_1x03-1MP_P1.00mm_Vertical -> lib:PinSocket_1x05_P2.54mm_Vertical
- moved J3 62.0 mm to (146.5, 98.1)
- moved U1 43.9 mm to (161.7, 62.3), turned to -90 degrees
- moved JP1 35.6 mm to (163.0, 68.2), turned to 0 degrees
- moved R2 28.9 mm to (162.5, 74.2), turned to 180 degrees
- moved R1 26.3 mm to (162.5, 76.4), turned to 180 degrees
- moved R5 24.2 mm to (146.4, 94.7)
Routing:
- net /GPIO15/RXD0: track 11.1 -> 141.6 mm, vias 0 -> 1
- net /GPIO14/TXD0: track 11.3 -> 114.8 mm, vias 0 -> 1
- net /RUN_PG: track 59.9 -> 11.6 mm
- net /GLOBAL_EN: track 64.4 -> 111.0 mm, vias 1 -> 2
- net /ID_SDA: track 101.7 -> 56.6 mm
- net /ID_SCL: track 94.9 -> 56.7 mm
- net /CONSOLE_TX: track 0.00 -> 11.2 mm
- net /CONSOLE_RX: track 0.00 -> 11.2 mm
- net +3.3V: track 145.8 -> 135.9 mm, vias 1 -> 0
- net GND: track 38.4 -> 43.8 mm, vias 1 -> 21
Other:
- outline, holes or cut-outs redrawn
- board text added: "CONSOLE_RX"
- board text added: "CONSOLE_TX"
- board text added: "GND"
- board text added: "GPIO14"
- board text added: "GPIO15"
- board text added: "pi5 carrier v3"

Commit message: pi5_adapter: add notch for pcie
Problem: pcie ffc cable bend radius gets squashed under the board.

Add a slot so it can have some room to bend.
Parts:
- moved REF** 53.7 mm to (113.3, 104.2), turned to 0 degrees
Routing:
- net GND: track 43.8 -> 51.8 mm, vias 21 -> 39
- net /GPIO10/SPI0.MOSI: track 11.1 -> 12.6 mm
- net /GPIO8/SPI0.CE0: track 11.1 -> 12.3 mm
- net /GPIO5: track 11.1 -> 12.0 mm
- net /GPIO18/PCM.CLK: track 11.1 -> 11.9 mm
- net /GPIO25: track 11.1 -> 11.8 mm
- net /GPIO12/PWM0: track 11.1 -> 11.8 mm
- net /GPIO23: track 11.1 -> 11.7 mm
Other:
- outline, holes or cut-outs redrawn
- board text added: "pi5 adapter v3"
- board text removed: "pi5 carrier v3"
